File: board/pic_k42.brd (EAGLE design)
At the start: 100 x 80 mm, 10 parts, among them IC1 PIC18F57K42-E_PT, Q1 ASF1

Commit message: update
Routing:
- net N$6: track 34.5 -> 37.4 mm
- net VSS: track 0.00 -> 2.30 mm
- net N$1: track 22.1 -> 23.2 mm
- net VDD: track 82.6 -> 82.1 mm
- net N$4: track 14.1 -> 14.6 mm
Other:
- board size 100 x 80 mm -> 55.6 x 58.4 mm

Commit message: update
Parts:
- added C10, C12, C5, C6, C7, C8, C9: 0.1, rcl:C1206
- added C11: 15uf, rcl:C1206
- added PORTA, PORTB, PORTC, PORTD, PORTE, PORTF: 332-10, con-garry:332-10
- added POWER: 5VDC, con-amp-quick:02P
- added RS-232-2: serial2, con-amp-quick:04P
- added RS232-1: serial1, con-amp-quick:04P
Connections:
- net VDD: now also C10.1, C11.1, C12.1, C5.1, C6.1, C7.1, C8.1, C9.1, PORTA.9, PORTB.9, PORTC.9, PORTD.9, PORTE.9, PORTF.9, POWER.2
- net VSS: now also C10.2, C11.2, C12.2, C5.2, C6.2, C7.2, C8.2, C9.2, PORTA.10, PORTB.10, PORTC.10, PORTD.10, PORTE.10, PORTF.10, POWER.1, RS-232-2.1, RS232-1.1
Routing:
- net VDD: track 82.1 -> 167.9 mm, vias 1 -> 0
- net N$4: track 14.6 -> 13.9 mm, vias 0 -> 2

Commit message: update
Parts:
- added C13, C14: 0.1, rcl:C1206
- added C15, C16: 15uf, rcl:C1206
- added C17, C18, C19, C20, C21: 1uf, rcl:C0805
- added IC2: REF3440IDBVR, SamacSys_Parts:SOP95P280X145-6N
- added IC3: MAX232, maxim:DIL16
- added X1: 332-02, con-garry:332-02
- moved SV1 10.2 mm to (40.6, 3.81)
- moved R2 6.84 mm to (45.7, 14.0)
- moved R1 6.48 mm to (45.7, 16.5)
- moved C1 3.81 mm to (45.7, 11.4)
- moved RS-232-2 2.54 mm to (66.0, 11.4)
- moved R3 2.54 mm to (45.7, 8.89)
Connections:
- new net N$10: C19.1, IC3.1
- new net N$11: C20.1, IC3.4
- new net N$12: C20.2, IC3.5
- new net N$13: C19.2, IC3.3
- new net N$14: IC3.14, RS232-1.2
- new net N$15: IC3.7, RS-232-2.2
- new net N$16: IC3.13, RS232-1.3
- new net N$17: IC3.8, RS-232-2.3
- new net N$18: IC1.1, IC3.12
- new net N$19: IC3.9, X1.1
- new net N$5: C17.1, IC3.6
- new net N$8: C13.1, C16.1, IC1.24, IC2.5, IC2.6
- new net N$9: C18.1, IC3.2
- net N$6: now also X1.2
- net VDD: now also C14.1, C15.1, C21.1, IC2.3, IC2.4, IC3.16
- net VSS: now also C13.2, C14.2, C15.2, C16.2, C17.2, C18.2, C21.2, IC2.1, IC2.2, IC3.15
Routing:
- net N$18: track 0.00 -> 34.3 mm, vias 0 -> 1
- net N$10: track 0.00 -> 31.8 mm
- net N$14: track 0.00 -> 25.6 mm
- net N$5: track 0.00 -> 21.1 mm
- net N$16: track 0.00 -> 20.5 mm
- net N$13: track 0.00 -> 20.3 mm
- net VDD: track 167.9 -> 185.4 mm
- net N$8: track 0.00 -> 15.3 mm
- net N$12: track 0.00 -> 14.4 mm, vias 0 -> 1
- net N$11: track 0.00 -> 13.6 mm
- net N$17: track 0.00 -> 13.5 mm
- net VSS: track 2.40 -> 15.4 mm
- net N$9: track 0.00 -> 9.05 mm
- net N$15: track 0.00 -> 8.45 mm
- net N$19: track 0.00 -> 6.93 mm
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
Commit message: update
Parts:
- added X2: 332-02, con-garry:332-02
- moved C5 16.9 mm to (74.9, 33.0)
- moved PORTC 16.9 mm to (68.6, 33.0)
- moved C6 15.3 mm to (39.4, 33.0)
- moved PORTD 15.3 mm to (33.0, 33.0)
- moved SV1 5.39 mm to (44.5, 0.00)
- moved C21 5.08 mm to (49.5, 10.2)
- moved C10 3.81 mm to (74.9, 27.9)
- moved C7 3.81 mm to (39.4, 27.9)
- moved PORTA 3.81 mm to (68.6, 27.9)
- moved PORTB 3.81 mm to (33.0, 27.9)
- moved C1 1.27 mm to (44.5, 11.4)
- moved R1 1.27 mm to (44.5, 16.5)
- moved R2 1.27 mm to (44.5, 14.0)
- moved R3 1.27 mm to (44.5, 8.89)
Connections:
- new net N$20: IC1.48, IC3.11
- new net N$22: IC3.10, X2.1
- net N$7: now also X2.2
Routing:
- net N$20: track 0.00 -> 32.7 mm, vias 0 -> 1
- net N$6: track 40.8 -> 60.8 mm, vias 1 -> 0
- net VDD: track 185.4 -> 197.0 mm
- net N$22: track 0.00 -> 3.99 mm
- net N$7: track 36.9 -> 39.3 mm, vias 0 -> 1
- net N$18: track 34.3 -> 35.1 mm
- net N$2: track 23.5 -> 24.1 mm
- net N$1: track 18.3 -> 18.8 mm
Other:
- board size 55.6 x 58.4 mm -> 55.6 x 67.3 mm

Commit message: updates
Parts:
- added LED1: RUN, led:CHIPLED_1206
- added R4: 220, rcl:R1206
Connections:
- new net N$21: LED1.A, R4.1
- new net N$23: IC1.27, R4.2
- net VSS: now also LED1.C
Routing:
- net N$23: track 0.00 -> 18.9 mm
- net N$21: track 0.00 -> 4.20 mm
- net N$6: track 60.8 -> 57.1 mm
- net VDD: track 197.0 -> 195.0 mm
- net N$18: track 35.1 -> 36.3 mm

Commit message: update
Parts:
- added SV2: DEBUG, con-lstb:MA04-1
Connections:
- new net N$24: IC1.28, SV2.3
- new net N$25: IC1.29, SV2.4
- net N$23: now also SV2.2
- net VSS: now also SV2.1
Routing:
- net N$25: track 0.00 -> 25.1 mm
- net N$24: track 0.00 -> 21.2 mm
- net N$23: track 18.9 -> 39.1 mm
- net VDD: track 195.0 -> 210.7 mm
- net N$18: track 36.3 -> 35.1 mm

Commit message: update
Parts:
- added X3: 332-02, con-garry:332-02
Connections:
- net N$1: now also X3.2
- net VSS: now also X3.1
Routing:
- net N$1: track 18.8 -> 21.8 mm
Changed lines of the file:
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@@
 <attribute name="VALUE" x="73.279" y="43.815" size="1.27" layer="27" ratio="10" rot="R90"/>
+</element>
+<element name="X3" library="con-garry" library_urn="urn:adsk.eagle:library:147" package="332-02" package3d_urn="urn:adsk.eagle:package:6810/1" value="332-02" x="40.64" y="15.24" smashed="yes" rot="R180">
+<attribute name="NAME" x="41.26" y="19.05" size="1.27" layer="25" rot="R180"/>
+<attribute name="VALUE" x="41.26" y="12.7" size="1.27" layer="27" rot="R180"/>
 </element>
 </elements>
@@
 <wire x1="43.1292" y1="11.43" x2="43.05" y2="11.43" width="0.1524" layer="1"/>
 <wire x1="43.1292" y1="13.8684" x2="43.028" y2="13.97" width="0.1524" layer="1"/>
-<wire x1="43.1292" y1="14.0208" x2="43.1292" y2="16.4592" width="0.1524" layer="1"/>
+<wire x1="43.1292" y1="14.0208" x2="43.1292" y2="14.3256" width="0.1524" layer="1"/>
+<wire x1="43.1292" y1="14.3256" x2="43.1292" y2="16.4592" width="0.1524" layer="1"/>
 <wire x1="43.1292" y1="16.4592" x2="43.028" y2="16.51" width="0.1524" layer="1"/>
 <wire x1="43.1292" y1="14.0208" x2="43.028" y2="13.97" width="0.1524" layer="1"/>
@@
 <wire x1="42.9768" y1="11.43" x2="38.1" y2="6.5532" width="0.1524" layer="1"/>
 <wire x1="42.9768" y1="11.43" x2="43.05" y2="11.43" width="0.1524" layer="1"/>
+<contactref element="X3" pad="2"/>
+<wire x1="43.1292" y1="14.3256" x2="40.6908" y2="14.3256" width="0.1524" layer="1"/>
+<wire x1="40.6908" y1="14.3256" x2="40.64" y2="14.24" width="0.1524" layer="1"/>
+<wire x1="43.1292" y1="14.3256" x2="43.028" y2="13.97" width="0.1524" layer="1"/>
 </signal>
 <signal name="N$2">
@@
 <wire x1="56.388" y1="42.2148" x2="56.308" y2="42.16" width="0.1524" layer="1"/>
 <wire x1="62.1792" y1="43.2816" x2="62.23" y2="43.31" width="0.1524" layer="1"/>
+<contactref element="X3" pad="1"/>
+<wire x1="57.15" y1="32.6136" x2="57.082" y2="32.7" width="0.1524" layer="1"/>
 <wire x1="57.15" y1="31.8516" x2="57.082" y2="31.75" width="0.1524" layer="1"/>
 <wire x1="39.37" y1="24.26" x2="37.02" y2="23.86" width="0" layer="19" extent="1-1"/>
