File: board/pic_k42.sch (EAGLE design)
At the start: 10 parts, among them IC1 PIC18F57K42-E_PT, Q1 ASF1

Commit message: update
Parts:
- added C10, C12, C5, C6, C7, C8, C9: 0.1, rcl:C-USC1206
- added C11: 15uf, rcl:C-USC1206
- added PORTA, PORTB, PORTC, PORTD, PORTE, PORTF: 332-10, con-garry:332-10
- added POWER: 5VDC, con-amp-quick:M02
- added RS-232-2: serial2, con-amp-quick:M04
- added RS232-1: serial1, con-amp-quick:M04
Connections:
- net VDD: now also C10.1, C11.1, C12.1, C5.1, C6.1, C7.1, C8.1, C9.1, PORTA-9.S, PORTB-9.S, PORTC-9.S, PORTD-9.S, PORTE-9.S, PORTF-9.S, POWER.2
- net VSS: now also C10.2, C11.2, C12.2, C5.2, C6.2, C7.2, C8.2, C9.2, PORTA-10.S, PORTB-10.S, PORTC-10.S, PORTD-10.S, PORTE-10.S, PORTF-10.S, POWER.1, RS-232-2.1, RS232-1.1

Commit message: update
Parts:
- added C13, C14: 0.1, rcl:C-USC1206
- added C15, C16: 15uf, rcl:C-USC1206
- added C17, C18, C19, C20, C21: 1uf, rcl:C-USC0805
- added IC2: REF3440IDBVR, SamacSys_Parts:REF3440IDBVR
- added IC3: MAX232, maxim:MAX232
- added X1: 332-02, con-garry:332-02
Connections:
- new net N$10: C19.1, IC3G$1.C1+
- new net N$11: C20.1, IC3G$1.C2+
- new net N$12: C20.2, IC3G$1.C2-
- new net N$13: C19.2, IC3G$1.C1-
- new net N$14: IC3G$1.T1OUT, RS232-1.2
- new net N$15: IC3G$1.T2OUT, RS-232-2.2
- new net N$16: IC3G$1.R1IN, RS232-1.3
- new net N$17: IC3G$1.R2IN, RS-232-2.3
- new net N$18: IC1.RC7, IC3G$1.R1OUT
- new net N$19: IC3G$1.R2OUT, X1-1.S
- new net N$5: C17.1, IC3G$1.V-
- new net N$8: C13.1, C16.1, IC1.RA3, IC2.5, IC2.6
- new net N$9: C18.1, IC3G$1.V+
- net N$6: now also X1-2.S
- net VDD: now also C14.1, C15.1, C21.1, IC2.3, IC2.4, IC3P.VCC
- net VSS: now also C13.2, C14.2, C15.2, C16.2, C17.2, C18.2, C21.2, IC2.1, IC2.2, IC3P.GND
Other:
- moved on the sheet: RS-232-2, RS232-1

Commit message: update
Parts:
- added X2: 332-02, con-garry:332-02
Connections:
- new net N$20: IC1.RC6, IC3G$1.T1IN
- new net N$22: IC3G$1.T2IN, X2-1.S
- net N$7: now also X2-2.S
Changed lines of the file:
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@@
 <part name="VSS34" library="supply1" library_urn="urn:adsk.eagle:library:371" deviceset="VSS" device=""/>
 <part name="X1" library="con-garry" library_urn="urn:adsk.eagle:library:147" deviceset="332-02" device="" package3d_urn="urn:adsk.eagle:package:6810/1"/>
+<part name="X2" library="con-garry" library_urn="urn:adsk.eagle:library:147" deviceset="332-02" device="" package3d_urn="urn:adsk.eagle:package:6810/1"/>
 </parts>
 <sheets>
@@
 <attribute name="NAME" x="22.86" y="-38.862" size="1.524" layer="95"/>
 <attribute name="VALUE" x="19.558" y="-36.703" size="1.778" layer="96"/>
+</instance>
+<instance part="X2" gate="-1" x="0" y="-30.48" smashed="yes">
+<attribute name="NAME" x="2.54" y="-31.242" size="1.524" layer="95"/>
+<attribute name="VALUE" x="-0.762" y="-29.083" size="1.778" layer="96"/>
+</instance>
+<instance part="X2" gate="-2" x="20.32" y="-30.48" smashed="yes">
+<attribute name="NAME" x="22.86" y="-31.242" size="1.524" layer="95"/>
+<attribute name="VALUE" x="19.558" y="-29.083" size="1.778" layer="96"/>
 </instance>
 </instances>
@@
 <wire x1="53.34" y1="17.78" x2="53.34" y2="10.16" width="0.1524" layer="91"/>
 <wire x1="53.34" y1="10.16" x2="40.64" y2="10.16" width="0.1524" layer="91"/>
-<wire x1="40.64" y1="10.16" x2="40.64" y2="2.54" width="0.1524" layer="91"/>
 <pinref part="SV1" gate="1" pin="5"/>
-<wire x1="40.64" y1="2.54" x2="40.64" y2="0" width="0.1524" layer="91"/>
 <wire x1="53.34" y1="-50.8" x2="53.34" y2="-35.56" width="0.1524" layer="91"/>
 <wire x1="53.34" y1="-35.56" x2="40.64" y2="-35.56" width="0.1524" layer="91"/>
-<wire x1="40.64" y1="-35.56" x2="40.64" y2="0" width="0.1524" layer="91"/>
+<wire x1="40.64" y1="-35.56" x2="40.64" y2="-25.4" width="0.1524" layer="91"/>
 <junction x="53.34" y="-50.8"/>
 <junction x="53.34" y="17.78"/>
+<pinref part="X2" gate="-2" pin="S"/>
+<wire x1="40.64" y1="-25.4" x2="40.64" y2="10.16" width="0.1524" layer="91"/>
+<wire x1="17.78" y1="-30.48" x2="17.78" y2="-25.4" width="0.1524" layer="91"/>
+<wire x1="17.78" y1="-25.4" x2="40.64" y2="-25.4" width="0.1524" layer="91"/>
+<junction x="17.78" y="-30.48"/>
+<junction x="40.64" y="-25.4"/>
 </segment>
 </net>
@@
 <wire x1="-7.62" y1="22.86" x2="0" y2="22.86" width="0.1524" layer="91"/>
 <wire x1="0" y1="22.86" x2="0" y2="10.16" width="0.1524" layer="91"/>
-<wire x1="0" y1="10.16" x2="-45.72" y2="10.16" width="0.1524" layer="91"/>
-<wire x1="-45.72" y1="10.16" x2="-45.72" y2="20.32" width="0.1524" layer="91"/>
+<wire x1="0" y1="10.16" x2="-63.5" y2="10.16" width="0.1524" layer="91"/>
+<junction x="-7.62" y="22.86"/>
 <pinref part="RS-232-2" gate="G$1" pin="2"/>
-<wire x1="-45.72" y1="20.32" x2="-68.58" y2="20.32" width="0.1524" layer="91"/>
+<wire x1="-68.58" y1="20.32" x2="-63.5" y2="20.32" width="0.1524" layer="91"/>
+<wire x1="-63.5" y1="20.32" x2="-63.5" y2="10.16" width="0.1524" layer="91"/>
 <junction x="-68.58" y="20.32"/>
-<junction x="-7.62" y="22.86"/>
 </segment>
 </net>
@@
 <wire x1="-53.34" y1="50.8" x2="-53.34" y2="25.4" width="0.1524" layer="91"/>
 <wire x1="-53.34" y1="25.4" x2="-45.72" y2="25.4" width="0.1524" layer="91"/>
-<wire x1="-45.72" y1="25.4" x2="-45.72" y2="22.86" width="0.1524" layer="91"/>
-<wire x1="-45.72" y1="22.86" x2="-40.64" y2="22.86" width="0.1524" layer="91"/>
-<wire x1="-40.64" y1="22.86" x2="-40.64" y2="20.32" width="0.1524" layer="91"/>
-<wire x1="-40.64" y1="20.32" x2="-38.1" y2="20.32" width="0.1524" layer="91"/>
+<wire x1="-45.72" y1="25.4" x2="-45.72" y2="20.32" width="0.1524" layer="91"/>
+<wire x1="-45.72" y1="20.32" x2="-38.1" y2="20.32" width="0.1524" layer="91"/>
 <junction x="33.02" y="73.66"/>
 <pinref part="IC3" gate="G$1" pin="R1OUT"/>
@@
 </segment>
 </net>
+<net name="N$20" class="0">
+<segment>
+<pinref part="IC3" gate="G$1" pin="T1IN"/>
+<wire x1="-38.1" y1="25.4" x2="-38.1" y2="27.94" width="0.1524" layer="91"/>
+<wire x1="-38.1" y1="27.94" x2="-63.5" y2="27.94" width="0.1524" layer="91"/>
+<wire x1="-63.5" y1="27.94" x2="-63.5" y2="93.98" width="0.1524" layer="91"/>
+<wire x1="-63.5" y1="93.98" x2="40.64" y2="93.98" width="0.1524" layer="91"/>
+<pinref part="IC1" gate="G$1" pin="RC6"/>
+<wire x1="40.64" y1="93.98" x2="40.64" y2="88.9" width="0.1524" layer="91"/>
+<junction x="-38.1" y="25.4"/>
+<junction x="40.64" y="88.9"/>
+</segment>
+</net>
+<net name="N$22" class="0">
+<segment>
+<pinref part="X2" gate="-1" pin="S"/>
+<wire x1="-2.54" y1="-30.48" x2="-40.64" y2="-30.48" width="0.1524" layer="91"/>
+<wire x1="-40.64" y1="-30.48" x2="-40.64" y2="22.86" width="0.1524" layer="91"/>
+<pinref part="IC3" gate="G$1" pin="T2IN"/>
+<wire x1="-40.64" y1="22.86" x2="-38.1" y2="22.86" width="0.1524" layer="91"/>
+<junction x="-38.1" y="22.86"/>
+<junction x="-2.54" y="-30.48"/>
+</segment>
+</net>

Commit message: updates
Parts:
- added LED1: RUN, led:LEDCHIPLED_1206
- added R4: 220, rcl:R-US_R1206
Connections:
- new net N$21: LED1.A, R4.1
- new net N$23: IC1.RE0, R4.2
- net VSS: now also LED1.C
Changed lines of the file:
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@@
 <part name="X1" library="con-garry" library_urn="urn:adsk.eagle:library:147" deviceset="332-02" device="" package3d_urn="urn:adsk.eagle:package:6810/1"/>
 <part name="X2" library="con-garry" library_urn="urn:adsk.eagle:library:147" deviceset="332-02" device="" package3d_urn="urn:adsk.eagle:package:6810/1"/>
+<part name="LED1" library="led" library_urn="urn:adsk.eagle:library:259" deviceset="LED" device="CHIPLED_1206" package3d_urn="urn:adsk.eagle:package:15823/2" value="RUN"/>
+<part name="R4" library="rcl" library_urn="urn:adsk.eagle:library:334" deviceset="R-US_" device="R1206" package3d_urn="urn:adsk.eagle:package:23540/2" value="220"/>
+<part name="VSS35" library="supply1" library_urn="urn:adsk.eagle:library:371" deviceset="VSS" device=""/>
 </parts>
 <sheets>
@@
 <attribute name="NAME" x="22.86" y="-31.242" size="1.524" layer="95"/>
 <attribute name="VALUE" x="19.558" y="-29.083" size="1.778" layer="96"/>
+</instance>
+<instance part="LED1" gate="G$1" x="162.56" y="12.7" smashed="yes">
+<attribute name="NAME" x="166.116" y="8.128" size="1.778" layer="95" rot="R90"/>
+<attribute name="VALUE" x="168.275" y="8.128" size="1.778" layer="96" rot="R90"/>
+</instance>
+<instance part="R4" gate="G$1" x="162.56" y="20.32" smashed="yes" rot="R90">
+<attribute name="NAME" x="161.0614" y="16.51" size="1.778" layer="95" rot="R90"/>
+<attribute name="VALUE" x="165.862" y="16.51" size="1.778" layer="96" rot="R90"/>
+</instance>
+<instance part="VSS35" gate="G$1" x="162.56" y="5.08" smashed="yes">
+<attribute name="VALUE" x="160.02" y="0" size="1.778" layer="96" rot="R90"/>
 </instance>
 </instances>
@@
 <junction x="-22.86" y="50.8"/>
 <junction x="-17.78" y="53.34"/>
+</segment>
+<segment>
+<pinref part="LED1" gate="G$1" pin="C"/>
+<pinref part="VSS35" gate="G$1" pin="VSS"/>
+<junction x="162.56" y="7.62"/>
 </segment>
 </net>
@@
 </segment>
 </net>
+<net name="N$21" class="0">
+<segment>
+<pinref part="LED1" gate="G$1" pin="A"/>
+<pinref part="R4" gate="G$1" pin="1"/>
+<junction x="162.56" y="15.24"/>
+</segment>
+</net>
+<net name="N$23" class="0">
+<segment>
+<wire x1="116.84" y1="50.8" x2="116.84" y2="27.94" width="0.1524" layer="91"/>
+<pinref part="IC1" gate="G$1" pin="RE0"/>
+<wire x1="76.2" y1="50.8" x2="116.84" y2="50.8" width="0.1524" layer="91"/>
+<pinref part="R4" gate="G$1" pin="2"/>
+<wire x1="162.56" y1="25.4" x2="162.56" y2="27.94" width="0.1524" layer="91"/>
+<wire x1="162.56" y1="27.94" x2="116.84" y2="27.94" width="0.1524" layer="91"/>
+</segment>
+</net>

Commit message: update
Parts:
- added SV2: DEBUG, con-lstb:MA04-1
Connections:
- new net N$24: IC1.RE1, SV2.3
- new net N$25: IC1.RE2, SV2.4
- net N$23: now also SV2.2
- net VSS: now also SV2.1
Changed lines of the file:
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@@
 <part name="R4" library="rcl" library_urn="urn:adsk.eagle:library:334" deviceset="R-US_" device="R1206" package3d_urn="urn:adsk.eagle:package:23540/2" value="220"/>
 <part name="VSS35" library="supply1" library_urn="urn:adsk.eagle:library:371" deviceset="VSS" device=""/>
+<part name="SV2" library="con-lstb" library_urn="urn:adsk.eagle:library:162" deviceset="MA04-1" device="" package3d_urn="urn:adsk.eagle:package:8337/1" value="DEBUG"/>
+<part name="VSS36" library="supply1" library_urn="urn:adsk.eagle:library:371" deviceset="VSS" device=""/>
 </parts>
 <sheets>
@@
 <instance part="VSS35" gate="G$1" x="162.56" y="5.08" smashed="yes">
 <attribute name="VALUE" x="160.02" y="0" size="1.778" layer="96" rot="R90"/>
+</instance>
+<instance part="SV2" gate="1" x="152.4" y="12.7" smashed="yes" rot="R180">
+<attribute name="VALUE" x="153.67" y="22.86" size="1.778" layer="96" rot="R180"/>
+<attribute name="NAME" x="153.67" y="6.858" size="1.778" layer="95" rot="R180"/>
+</instance>
+<instance part="VSS36" gate="G$1" x="144.78" y="20.32" smashed="yes" rot="R180">
+<attribute name="VALUE" x="147.32" y="25.4" size="1.778" layer="96" rot="R270"/>
 </instance>
 </instances>
@@
 <pinref part="VSS35" gate="G$1" pin="VSS"/>
 <junction x="162.56" y="7.62"/>
+</segment>
+<segment>
+<pinref part="SV2" gate="1" pin="1"/>
+<pinref part="VSS36" gate="G$1" pin="VSS"/>
+<junction x="144.78" y="17.78"/>
 </segment>
 </net>
@@
 <pinref part="R4" gate="G$1" pin="2"/>
 <wire x1="162.56" y1="25.4" x2="162.56" y2="27.94" width="0.1524" layer="91"/>
-<wire x1="162.56" y1="27.94" x2="116.84" y2="27.94" width="0.1524" layer="91"/>
-</segment>
-</net>
+<wire x1="162.56" y1="27.94" x2="139.7" y2="27.94" width="0.1524" layer="91"/>
+<wire x1="139.7" y1="27.94" x2="116.84" y2="27.94" width="0.1524" layer="91"/>
+<wire x1="139.7" y1="27.94" x2="139.7" y2="15.24" width="0.1524" layer="91"/>
+<pinref part="SV2" gate="1" pin="2"/>
+<wire x1="139.7" y1="15.24" x2="144.78" y2="15.24" width="0.1524" layer="91"/>
+<junction x="76.2" y="50.8"/>
+<junction x="144.78" y="15.24"/>
+<junction x="139.7" y="27.94"/>
+</segment>
+</net>
+<net name="N$24" class="0">
+<segment>
+<pinref part="IC1" gate="G$1" pin="RE1"/>
+<wire x1="76.2" y1="53.34" x2="111.76" y2="53.34" width="0.1524" layer="91"/>
+<wire x1="111.76" y1="53.34" x2="111.76" y2="25.4" width="0.1524" layer="91"/>
+<wire x1="111.76" y1="25.4" x2="137.16" y2="25.4" width="0.1524" layer="91"/>
+<wire x1="137.16" y1="25.4" x2="137.16" y2="12.7" width="0.1524" layer="91"/>
+<pinref part="SV2" gate="1" pin="3"/>
+<wire x1="137.16" y1="12.7" x2="144.78" y2="12.7" width="0.1524" layer="91"/>
+<junction x="76.2" y="53.34"/>
+<junction x="144.78" y="12.7"/>
+</segment>
+</net>
+<net name="N$25" class="0">
+<segment>
+<pinref part="SV2" gate="1" pin="4"/>
+<junction x="144.78" y="10.16"/>
+<wire x1="134.62" y1="10.16" x2="144.78" y2="10.16" width="0.1524" layer="91"/>
+<wire x1="134.62" y1="22.86" x2="134.62" y2="10.16" width="0.1524" layer="91"/>
+<pinref part="IC1" gate="G$1" pin="RE2"/>
+<wire x1="76.2" y1="55.88" x2="81.28" y2="55.88" width="0.1524" layer="91"/>
+<wire x1="81.28" y1="55.88" x2="81.28" y2="48.26" width="0.1524" layer="91"/>
+<wire x1="81.28" y1="48.26" x2="106.68" y2="48.26" width="0.1524" layer="91"/>
+<wire x1="106.68" y1="48.26" x2="106.68" y2="22.86" width="0.1524" layer="91"/>
+<wire x1="106.68" y1="22.86" x2="134.62" y2="22.86" width="0.1524" layer="91"/>
+</segment>
+</net>

Commit message: update
Parts:
- added X3: 332-02, con-garry:332-02
Connections:
- net N$1: now also X3-2.S
- net VSS: now also X3-1.S
Changed lines of the file:
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@@
 <part name="SV2" library="con-lstb" library_urn="urn:adsk.eagle:library:162" deviceset="MA04-1" device="" package3d_urn="urn:adsk.eagle:package:8337/1" value="DEBUG"/>
 <part name="VSS36" library="supply1" library_urn="urn:adsk.eagle:library:371" deviceset="VSS" device=""/>
+<part name="X3" library="con-garry" library_urn="urn:adsk.eagle:library:147" deviceset="332-02" device="" package3d_urn="urn:adsk.eagle:package:6810/1"/>
+<part name="VSS37" library="supply1" library_urn="urn:adsk.eagle:library:371" deviceset="VSS" device=""/>
 </parts>
 <sheets>
@@
 <attribute name="VALUE" x="147.32" y="25.4" size="1.778" layer="96" rot="R270"/>
 </instance>
+<instance part="X3" gate="-1" x="73.66" y="-10.16" smashed="yes" rot="R90">
+<attribute name="NAME" x="74.422" y="-7.62" size="1.524" layer="95" rot="R90"/>
+<attribute name="VALUE" x="72.263" y="-10.922" size="1.778" layer="96" rot="R90"/>
+</instance>
+<instance part="X3" gate="-2" x="73.66" y="10.16" smashed="yes" rot="R90">
+<attribute name="NAME" x="74.422" y="12.7" size="1.524" layer="95" rot="R90"/>
+<attribute name="VALUE" x="72.263" y="9.398" size="1.778" layer="96" rot="R90"/>
+</instance>
+<instance part="VSS37" gate="G$1" x="73.66" y="-15.24" smashed="yes">
+<attribute name="VALUE" x="71.12" y="-20.32" size="1.778" layer="96" rot="R90"/>
+</instance>
 </instances>
 <busses>
@@
 <wire x1="63.5" y1="0" x2="58.42" y2="0" width="0.1524" layer="91"/>
 <junction x="63.5" y="-50.8"/>
+<wire x1="63.5" y1="0" x2="73.66" y2="0" width="0.1524" layer="91"/>
+<pinref part="X3" gate="-2" pin="S"/>
+<wire x1="73.66" y1="0" x2="73.66" y2="7.62" width="0.1524" layer="91"/>
+<junction x="63.5" y="0"/>
+<junction x="73.66" y="7.62"/>
 </segment>
 </net>
@@
 <junction x="144.78" y="17.78"/>
 </segment>
+<segment>
+<pinref part="X3" gate="-1" pin="S"/>
+<pinref part="VSS37" gate="G$1" pin="VSS"/>
+</segment>
 </net>
