File: host_board/pic_k42.brd (EAGLE design)
At the start: 55.6 x 67.3 mm, 39 parts, among them IC1 PIC18F57K42-E_PT, IC2 REF3440IDBVR, IC3 MAX232, K1 G6K-2P, Q1 ASF1, X1 332-02, X2 332-02, X3 332-02, X4 22-23-2101, X5 22-23-2101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

Commit message: update
Parts:
- moved C5 6.48 mm to (45.7, 19.1)
- moved Q1 6.35 mm to (61.0, 41.9)
- moved C21 5.24 mm to (45.7, 21.6)
- moved C1 5.08 mm to (48.3, 27.9)
- moved X1 5.08 mm to (53.3, 26.7)
- moved R3 5.08 mm to (48.3, 25.4)
- moved C2 3.81 mm to (66.0, 41.9), turned to 270 degrees
- moved R1 3.81 mm to (48.3, 33.0)
- moved R2 3.81 mm to (48.3, 30.5)
- moved X2 3.81 mm to (53.3, 31.8)
- moved C20 3.59 mm to (66.0, 7.62)
- moved C17 3.59 mm to (61.0, 7.62)
- moved C18 3.59 mm to (50.8, 7.62)
- moved C19 3.59 mm to (55.9, 7.62)
- moved IC3 2.54 mm to (59.7, 15.2)
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Connections:
- removed net N$17: K1.7, RS-232-2.3
- new net GND: C21.2, IC3.15, Q1.2
- new net N$62: K1.5, RS-232-2.3
- new net VCC: C21.1, IC3.16, Q1.4
- net N$14: now also K1.4, K1.7; no longer K1.2, K1.5
- net VDD: no longer C21.1, IC3.16, Q1.4
- net VSS: no longer C21.2, IC3.15, Q1.2
Routing:
- net VSS: track 10.2 -> 309.8 mm, vias 0 -> 1
- net N$18: track 37.6 -> 110.4 mm, vias 0 -> 1
- net GND: track 0.00 -> 58.6 mm, vias 0 -> 4
- net VCC: track 0.00 -> 54.6 mm, vias 0 -> 4
- net N$53: track 47.2 -> 95.9 mm, vias 1 -> 2
- net N$47: track 46.0 -> 79.8 mm
- net N$37: track 76.3 -> 45.6 mm, vias 0 -> 2
- net N$51: track 43.6 -> 63.9 mm, vias 2 -> 1
- net N$23: track 58.9 -> 42.3 mm
- net VDD: track 197.7 -> 213.3 mm, vias 5 -> 6
- net N$55: track 37.3 -> 51.8 mm, vias 1 -> 2
- net N$17: track 12.3 -> 0.00 mm
- net N$25: track 32.1 -> 20.1 mm
- net N$7: track 45.2 -> 56.6 mm, vias 3 -> 1
- net N$43: track 70.1 -> 81.1 mm
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- removed copper zone on layer 1, net VSS
- removed copper zone on layer 16, net VSS

Commit message: update
Parts:
- added S1: (no value), switch-omron:B3F-10XX
- moved OPTIONS 29.9 mm to (44.5, 12.7)
Connections:
- net N$1: now also S1.4
- net VSS: now also S1.2
Routing:
- net N$1: track 22.0 -> 114.4 mm, vias 0 -> 2
- net N$60: track 68.7 -> 29.6 mm
- net N$61: track 55.8 -> 81.0 mm
- net VSS: track 309.8 -> 321.4 mm
Changed lines of the file:
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@@
 <attribute name="VALUE" x="44.45" y="0" size="1.016" layer="27" ratio="10" rot="R90"/>
 </element>
-<element name="OPTIONS" library="con-molex" library_urn="urn:adsk.eagle:library:165" package="22-23-2021" value="22-23-2021" x="73.66" y="6.35" smashed="yes" rot="R180">
-<attribute name="MF" value="MOLEX" x="73.66" y="6.35" size="1.778" layer="27" rot="R180" display="off"/>
-<attribute name="MPN" value="22-23-2021" x="73.66" y="6.35" size="1.778" layer="27" rot="R180" display="off"/>
-<attribute name="NAME" x="76.2" y="2.54" size="1.016" layer="25" ratio="10" rot="R180"/>
-<attribute name="OC_FARNELL" value="1462926" x="73.66" y="6.35" size="1.778" layer="27" rot="R180" display="off"/>
-<attribute name="OC_NEWARK" value="25C3832" x="73.66" y="6.35" size="1.778" layer="27" rot="R180" display="off"/>
-<attribute name="VALUE" x="76.2" y="11.43" size="1.016" layer="27" ratio="10" rot="R180"/>
+<element name="OPTIONS" library="con-molex" library_urn="urn:adsk.eagle:library:165" package="22-23-2021" value="22-23-2021" x="44.45" y="12.7" smashed="yes" rot="R180">
+<attribute name="MF" value="MOLEX" x="44.45" y="12.7" size="1.778" layer="27" rot="R180" display="off"/>
+<attribute name="MPN" value="22-23-2021" x="44.45" y="12.7" size="1.778" layer="27" rot="R180" display="off"/>
+<attribute name="NAME" x="46.99" y="8.89" size="1.016" layer="25" ratio="10" rot="R180"/>
+<attribute name="OC_FARNELL" value="1462926" x="44.45" y="12.7" size="1.778" layer="27" rot="R180" display="off"/>
+<attribute name="OC_NEWARK" value="25C3832" x="44.45" y="12.7" size="1.778" layer="27" rot="R180" display="off"/>
+<attribute name="VALUE" x="46.99" y="17.78" size="1.016" layer="27" ratio="10" rot="R180"/>
+</element>
+<element name="S1" library="switch-omron" library_urn="urn:adsk.eagle:library:377" package="B3F-10XX" package3d_urn="urn:adsk.eagle:package:27496/1" value="" x="73.66" y="6.35" smashed="yes" rot="R270">
+<attribute name="MF" value="" x="73.66" y="6.35" size="1.778" layer="27" rot="R270" display="off"/>
+<attribute name="MPN" value="B3F-1000" x="73.66" y="6.35" size="1.778" layer="27" rot="R270" display="off"/>
+<attribute name="NAME" x="77.343" y="9.398" size="1.27" layer="25" ratio="10" rot="R270"/>
+<attribute name="OC_FARNELL" value="176432" x="73.66" y="6.35" size="1.778" layer="27" rot="R270" display="off"/>
+<attribute name="OC_NEWARK" value="36M3542" x="73.66" y="6.35" size="1.778" layer="27" rot="R270" display="off"/>
+<attribute name="VALUE" x="68.58" y="9.398" size="1.27" layer="27" ratio="10" rot="R270"/>
 </element>
 </elements>
@@
 <wire x1="30.48" y1="32.9184" x2="30.48" y2="33.02" width="0.1524" layer="16"/>
 <wire x1="44.3484" y1="33.2232" x2="44.45" y2="33.29" width="0.1524" layer="16"/>
+<contactref element="S1" pad="4"/>
+<wire x1="71.4756" y1="7.4676" x2="71.4756" y2="3.2004" width="0.1524" layer="16"/>
+<wire x1="76.6572" y1="12.6492" x2="71.4756" y2="7.4676" width="0.1524" layer="16"/>
+<wire x1="76.6572" y1="44.958" x2="76.6572" y2="12.6492" width="0.1524" layer="16"/>
+<wire x1="71.3232" y1="50.292" x2="76.6572" y2="44.958" width="0.1524" layer="16"/>
+<wire x1="70.7136" y1="50.292" x2="71.3232" y2="50.292" width="0.1524" layer="16"/>
+<wire x1="69.6468" y1="51.3588" x2="70.7136" y2="50.292" width="0.1524" layer="16"/>
+<wire x1="69.6468" y1="53.1876" x2="69.6468" y2="51.3588" width="0.1524" layer="16"/>
+<wire x1="68.58" y1="54.2544" x2="69.6468" y2="53.1876" width="0.1524" layer="16"/>
+<wire x1="60.96" y1="54.2544" x2="68.58" y2="54.2544" width="0.1524" layer="16"/>
+<wire x1="59.436" y1="52.7304" x2="60.96" y2="54.2544" width="0.1524" layer="16"/>
+<wire x1="59.436" y1="48.9204" x2="59.436" y2="52.7304" width="0.1524" layer="16"/>
+<wire x1="54.102" y1="43.5864" x2="59.436" y2="48.9204" width="0.1524" layer="16"/>
+<wire x1="52.578" y1="42.0624" x2="54.102" y2="43.5864" width="0.1524" layer="1"/>
+<wire x1="49.53" y1="39.0144" x2="52.578" y2="42.0624" width="0.1524" layer="16"/>
+<wire x1="49.53" y1="38.4048" x2="49.53" y2="39.0144" width="0.1524" layer="16"/>
+<wire x1="44.5008" y1="33.3756" x2="49.53" y2="38.4048" width="0.1524" layer="16"/>
+<wire x1="71.4756" y1="3.2004" x2="71.3994" y2="3.0988" width="0.1524" layer="16"/>
+<wire x1="44.5008" y1="33.3756" x2="44.45" y2="33.29" width="0.1524" layer="16"/>
+<via x="54.102" y="43.5864" extent="1-16" drill="0.35"/>
+<via x="52.578" y="42.0624" extent="1-16" drill="0.35"/>
 </signal>
 <signal name="N$2">
@@
 <wire x1="44.3484" y1="35.2044" x2="44.45" y2="35.29" width="0.1524" layer="1"/>
 <via x="71.1708" y="25.2984" extent="1-16" drill="0.35"/>
+<contactref element="S1" pad="2"/>
+<wire x1="73.6092" y1="3.048" x2="75.8952" y2="3.048" width="0.1524" layer="16"/>
+<wire x1="71.3232" y1="0.762" x2="73.6092" y2="3.048" width="0.1524" layer="16"/>
+<wire x1="67.818" y1="0.762" x2="71.3232" y2="0.762" width="0.1524" layer="16"/>
+<wire x1="66.04" y1="2.54" x2="67.818" y2="0.762" width="0.1524" layer="16"/>
+<wire x1="75.8952" y1="3.048" x2="75.9206" y2="3.0988" width="0.1524" layer="16"/>
 </signal>
 <signal name="N$6">
@@
 <wire x1="49.0728" y1="38.7096" x2="50.1396" y2="38.7096" width="0.1524" layer="1"/>
 <wire x1="48.6156" y1="38.2524" x2="49.0728" y2="38.7096" width="0.1524" layer="1"/>
-<wire x1="48.6156" y1="4.4196" x2="48.6156" y2="38.2524" width="0.1524" layer="1"/>
-<wire x1="49.3776" y1="3.6576" x2="48.6156" y2="4.4196" width="0.1524" layer="1"/>
-<wire x1="49.3776" y1="1.2192" x2="49.3776" y2="3.6576" width="0.1524" layer="1"/>
-<wire x1="50.4444" y1="0.1524" x2="49.3776" y2="1.2192" width="0.1524" layer="1"/>
-<wire x1="68.7324" y1="0.1524" x2="50.4444" y2="0.1524" width="0.1524" layer="1"/>
-<wire x1="74.93" y1="6.35" x2="68.7324" y2="0.1524" width="0.1524" layer="1"/>
+<wire x1="48.6156" y1="15.5956" x2="48.6156" y2="38.2524" width="0.1524" layer="1"/>
+<wire x1="45.72" y1="12.7" x2="48.6156" y2="15.5956" width="0.1524" layer="1"/>
 <wire x1="50.292" y1="37.7952" x2="50.32" y2="37.672" width="0.1524" layer="1"/>
 </signal>
@@
 <wire x1="73.4568" y1="25.6032" x2="72.5424" y2="25.6032" width="0.1524" layer="1"/>
 <wire x1="76.3524" y1="22.7076" x2="73.4568" y2="25.6032" width="0.1524" layer="1"/>
-<wire x1="76.3524" y1="10.3632" x2="76.3524" y2="22.7076" width="0.1524" layer="1"/>
-<wire x1="72.39" y1="6.4008" x2="76.3524" y2="10.3632" width="0.1524" layer="1"/>
+<wire x1="76.3524" y1="12.7" x2="76.3524" y2="22.7076" width="0.1524" layer="1"/>
 <wire x1="49.8348" y1="37.6428" x2="49.82" y2="37.672" width="0.1524" layer="1"/>
-<wire x1="72.39" y1="6.4008" x2="72.39" y2="6.35" width="0.1524" layer="1"/>
+<wire x1="76.3524" y1="12.7" x2="43.18" y2="12.7" width="0.1524" layer="1"/>
 <via x="50.1396" y="36.2712" extent="1-16" drill="0.35"/>
 <via x="69.9516" y="28.194" extent="1-16" drill="0.35"/>

Commit message: update
Parts:
- added C6: 0.1, rcl:C1206
- added IC4: ILAMP, ic-package:SOCKET-16
- added LED2: MODE, led:CHIPLED_1206
- added LSP1, LSP2, LSP3, LSP4: LSP10, solpad:LSP10
- added R5, R6, R7: 220, rcl:R1206
- added S2: MODESW, switch-omron:B3F-10XX
- S1: value (none) -> RESETSW
- moved S1 66.9 mm to (36.8, 62.2), turned to 0 degrees
- moved POWER 60.2 mm to (69.8, 2.54)
- moved X5 45.8 mm to (31.8, 40.6), turned to 90 degrees
- moved SV1 43.2 mm to (73.7, 39.4)
- moved C11 38.9 mm to (69.8, 7.62)
- moved OPTIONS 37.4 mm to (66.0, 43.2)
- moved RS232-1 36.9 mm to (49.5, 2.54), turned to 180 degrees
- moved X1 21.6 mm to (36.8, 40.6)
- moved X2 21.6 mm to (36.8, 45.7)
- moved RS-232-2 21.6 mm to (59.7, 2.54), turned to 180 degrees
- moved X3 18.2 mm to (36.8, 50.8)
- moved C5 18.0 mm to (48.3, 36.8), turned to 180 degrees
- moved C21 17.6 mm to (54.6, 36.8)
- moved R3 15.3 mm to (54.6, 39.4)
- moved K1 14.5 mm to (69.8, 15.2)
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Connections:
- new net N$17: IC4.1, R5.1
- new net N$55: IC4.14, LSP1.MP
- new net N$63: IC4.16, R6.2
- new net N$64: LED2.A, R7.1
- new net N$65: IC4.13, LSP2.MP
- new net N$67: IC4.3, LSP3.MP
- new net N$68: IC4.4, LSP4.MP
- net N$43: now also C6.1, IC1.8, S2.3, X7.10; no longer IC1.43, X6.1
- net N$46: now also R5.2
- net N$47: now also IC4.2
- net N$48: now also R6.1
- net N$49: now also IC4.15
- net N$52: now also IC1.43, R7.2, X6.1; no longer IC1.8, X7.10
- net VSS: now also C6.2, LED2.C, S2.2
Routing:
- net N$52: track 25.4 -> 135.8 mm, vias 3 -> 2
- net N$6: track 50.9 -> 152.5 mm, vias 4 -> 7
- net N$36: track 75.5 -> 148.6 mm, vias 1 -> 3
- net N$67: track 0.00 -> 72.5 mm, vias 0 -> 2
- net N$43: track 81.1 -> 146.2 mm, vias 1 -> 2
- net N$46: track 48.7 -> 108.3 mm, vias 0 -> 2
- net N$55: track 0.00 -> 48.3 mm
- net N$35: track 63.1 -> 102.1 mm, vias 2 -> 4
- net N$65: track 0.00 -> 37.2 mm
- net N$50: track 47.4 -> 81.7 mm, vias 3 -> 4
- net N$22: track 19.1 -> 51.4 mm
- net N$28: track 57.1 -> 88.7 mm, vias 2 -> 1
- net VCC: track 54.6 -> 85.4 mm, vias 4 -> 2
- net N$64: track 0.00 -> 29.0 mm
- net VSS: track 321.4 -> 347.2 mm, vias 1 -> 6
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- added copper zone on layer 1, net VDD
- added copper zone on layer 16, net VSS
Other:
- board size 55.6 x 67.3 mm -> 54.6 x 73.7 mm

Commit message: update
Parts:
- SPI: value 22-23-2101 -> LCD
- X1: value 332-02 -> RX-2
- X2: value 332-02 -> TX-2
- X3: value 332-02 -> RESETJMP
- X5: value 22-23-2101 -> PORTA
- X6: value 22-23-2101 -> PORTD
- X7: value 22-23-2101 -> PORTB
- moved LSP3 45.6 mm to (47.0, 11.4)
- moved LSP2 29.0 mm to (40.6, 27.9)
- moved LSP4 28.5 mm to (50.8, 11.4)
- moved LSP1 26.7 mm to (40.6, 31.8)
- moved R7 20.1 mm to (55.9, 11.4), turned to 0 degrees
- moved C6 12.7 mm to (62.2, 11.4), turned to 0 degrees
- moved IC3 10.9 mm to (61.0, 24.1), turned to 270 degrees
- moved IC4 8.13 mm to (49.5, 24.1), turned to 270 degrees
- moved R6 7.73 mm to (41.9, 36.8)
- moved X3 5.68 mm to (34.3, 55.9), turned to 270 degrees
- moved R5 5.24 mm to (41.9, 39.4)
- moved C2 1.27 mm to (66.0, 54.6), turned to 90 degrees
- moved K1 1.27 mm to (71.1, 15.2)
- moved SV1 1.27 mm to (73.7, 40.6)
- moved SV2 1.27 mm to (73.7, 55.9)
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- renumbered X4 to SPI
Routing:
- net N$36: track 148.6 -> 31.7 mm, vias 3 -> 1
- net N$6: track 152.5 -> 45.1 mm, vias 7 -> 3
- net N$51: track 82.7 -> 164.2 mm, vias 4 -> 3
- net N$49: track 56.7 -> 137.4 mm, vias 2 -> 3
- net N$35: track 102.1 -> 34.4 mm, vias 4 -> 1
- net N$67: track 72.5 -> 17.4 mm, vias 2 -> 0
- net N$50: track 81.7 -> 136.1 mm
- net N$44: track 86.4 -> 138.5 mm, vias 0 -> 2
- net N$56: track 51.6 -> 102.2 mm, vias 4 -> 5
- net N$57: track 40.8 -> 90.0 mm, vias 1 -> 6
- net N$9: track 4.04 -> 43.2 mm
- net N$20: track 94.5 -> 132.8 mm
- net N$23: track 40.8 -> 75.8 mm, vias 3 -> 2
- net N$37: track 41.3 -> 75.0 mm
- net N$40: track 60.3 -> 28.8 mm, vias 1 -> 2
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Other:
- board text added: "1.0"

Commit message: update
Parts:
- added R8, R9: 0, rcl:R1206
- moved SV1 2.54 mm to (73.7, 43.2)
- moved SV2 2.54 mm to (73.7, 58.4)
- moved X2 2.54 mm to (36.8, 48.3)
- moved X1 1.27 mm to (36.8, 41.9)
Connections:
- net GND: now also R9.1
- net VCC: now also R8.1
- net VDD: now also R8.2
- net VSS: now also R9.2
Routing:
- net N$40: track 28.8 -> 155.8 mm, vias 2 -> 4
- net N$51: track 164.2 -> 64.9 mm, vias 3 -> 4
- net N$8: track 64.3 -> 150.6 mm, vias 7 -> 6
- net N$50: track 136.1 -> 60.7 mm, vias 4 -> 3
- net VCC: track 55.3 -> 126.2 mm
- net N$47: track 77.7 -> 137.1 mm, vias 6 -> 4
- net N$44: track 138.5 -> 87.9 mm, vias 2 -> 0
- net N$6: track 45.1 -> 88.4 mm, vias 3 -> 4
- net N$46: track 121.5 -> 79.0 mm, vias 2 -> 3
- net N$56: track 102.2 -> 60.7 mm, vias 5 -> 3
- net N$37: track 75.0 -> 33.8 mm, vias 5 -> 3
- net N$20: track 132.8 -> 96.7 mm
- net GND: track 38.0 -> 72.0 mm, vias 0 -> 1
- net N$49: track 137.4 -> 169.2 mm, vias 3 -> 5
- net VDD: track 249.7 -> 219.7 mm, vias 7 -> 11
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Other:
- board text added: "1.1"
- board text removed: "1.0"
