File: host_board/pic_k42.brd (EAGLE design)
At the start: 55.9 x 78.7 mm, 57 parts, among them IC1 PIC18F57K42-E_PT, IC2 REF3440IDBVR, IC3 MAX232, IC4 ILAMP, K1 G6K-2P, Q1 ASF1, X1 RX-2, X2 TX-2, X3 RESETJMP, X4 MINI-USB-UX60A-MB-5ST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

Commit message: mbmc version
Parts:
- added R12: 220, rcl:R1206
Connections:
- new net N$70: C1.1, R12.1, R2.1, S4.4, X3.2
- net N$1: now also R12.2; no longer C1.1, R2.1, S4.4, X3.2
Routing:
- net N$70: track 0.00 -> 81.7 mm, vias 0 -> 4
- net N$1: track 131.1 -> 57.5 mm, vias 2 -> 1
- net N$45: track 161.9 -> 91.1 mm, vias 3 -> 2
- net N$38: track 32.8 -> 101.2 mm, vias 4 -> 2
- net N$35: track 49.1 -> 113.6 mm, vias 4 -> 3
- net N$43: track 141.7 -> 84.5 mm, vias 2 -> 5
- net N$8: track 68.7 -> 119.6 mm
- net N$22: track 54.8 -> 105.6 mm, vias 0 -> 4
- net N$7: track 93.3 -> 43.0 mm
- net N$23: track 64.4 -> 112.0 mm, vias 7 -> 1
- net VSS: track 323.5 -> 364.7 mm, vias 4 -> 3
- net GND: track 90.0 -> 130.2 mm, vias 4 -> 5
- net N$46: track 96.3 -> 61.8 mm, vias 2 -> 5
- net N$47: track 99.4 -> 129.4 mm, vias 3 -> 4
- net N$28: track 129.6 -> 100.8 mm, vias 3 -> 7
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