File: host_board/pic_k42.sch (EAGLE design)
At the start: 39 parts, among them IC1 PIC18F57K42-E_PT, IC2 REF3440IDBVR, IC3 MAX232, K1 G6K-2P, Q1 ASF1, X1 332-02, X2 332-02, X3 332-02, X4 22-23-2101, X5 22-23-2101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

Commit message: update
Connections:
- removed net N$17: K13.O, RS-232-2.3
- new net GND: C21.2, Q1.GND
- new net N$62: K13.S, RS-232-2.3
- new net VCC: C21.1, Q1.VCC
- net N$14: now also K12.S, K13.O; no longer K12.O, K13.S
- net VDD: no longer C21.1, IC3P.VCC, Q1.VCC
- net VSS: no longer C21.2, IC3P.GND, Q1.GND
Other:
- moved on the sheet: C21

Commit message: update
Parts:
- added S1: (no value), switch-omron:10-XX
Connections:
- net N$1: now also S1.P1
- net VSS: now also S1.S1
Changed lines of the file:
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@@
 <part name="VSS7" library="supply1" library_urn="urn:adsk.eagle:library:371" deviceset="VSS" device=""/>
 <part name="VDD10" library="supply1" library_urn="urn:adsk.eagle:library:371" deviceset="VDD" device=""/>
+<part name="S1" library="switch-omron" library_urn="urn:adsk.eagle:library:377" deviceset="10-XX" device="" package3d_urn="urn:adsk.eagle:package:27496/1"/>
+<part name="VSS15" library="supply1" library_urn="urn:adsk.eagle:library:371" deviceset="VSS" device=""/>
 </parts>
 <sheets>
@@
 <attribute name="VALUE" x="-109.22" y="73.66" size="1.778" layer="96"/>
 </instance>
+<instance part="S1" gate="1" x="152.4" y="-20.32" smashed="yes" rot="R180">
+<attribute name="NAME" x="158.75" y="-17.78" size="1.778" layer="95" rot="R270"/>
+<attribute name="VALUE" x="156.21" y="-23.495" size="1.778" layer="96" rot="R270"/>
+</instance>
+<instance part="VSS15" gate="G$1" x="149.86" y="-27.94" smashed="yes">
+<attribute name="VALUE" x="147.32" y="-33.02" size="1.778" layer="96" rot="R90"/>
+</instance>
 </instances>
 <busses>
@@
 <junction x="58.42" y="0"/>
 <pinref part="SV1" gate="1" pin="1"/>
-<wire x1="63.5" y1="-50.8" x2="63.5" y2="0" width="0.1524" layer="91"/>
+<wire x1="63.5" y1="-50.8" x2="63.5" y2="-17.78" width="0.1524" layer="91"/>
+<wire x1="63.5" y1="-17.78" x2="63.5" y2="0" width="0.1524" layer="91"/>
 <wire x1="63.5" y1="0" x2="58.42" y2="0" width="0.1524" layer="91"/>
 <junction x="63.5" y="-50.8"/>
@@
 <junction x="63.5" y="0"/>
 <junction x="73.66" y="7.62"/>
+<wire x1="63.5" y1="-17.78" x2="144.78" y2="-17.78" width="0.1524" layer="91"/>
+<pinref part="S1" gate="1" pin="P1"/>
+<wire x1="149.86" y1="-15.24" x2="144.78" y2="-15.24" width="0.1524" layer="91"/>
+<wire x1="144.78" y1="-15.24" x2="144.78" y2="-17.78" width="0.1524" layer="91"/>
+<junction x="63.5" y="-17.78"/>
+<junction x="149.86" y="-15.24"/>
 </segment>
 </net>
@@
 <pinref part="VSS14" gate="G$1" pin="VSS"/>
 </segment>
+<segment>
+<pinref part="S1" gate="1" pin="S1"/>
+<pinref part="VSS15" gate="G$1" pin="VSS"/>
+<junction x="149.86" y="-25.4"/>
+</segment>
 </net>

Commit message: update
Parts:
- added C6: 0.1, rcl:C-USC1206
- added IC4: ILAMP, ic-package:DIL16S
- added LED2: MODE, led:LEDCHIPLED_1206
- added LSP1, LSP2, LSP3, LSP4: LSP10, solpad:LSP10
- added R5, R6, R7: 220, rcl:R-US_R1206
- added S2: MODESW, switch-omron:10-XX
- S1: value (none) -> RESETSW
Connections:
- new net N$17: IC4.1, R5.1
- new net N$55: IC4.14, LSP1.MP
- new net N$63: IC4.16, R6.2
- new net N$64: LED2.A, R7.1
- new net N$65: IC4.13, LSP2.MP
- new net N$67: IC4.3, LSP3.MP
- new net N$68: IC4.4, LSP4.MP
- net N$43: now also C6.1, IC1.RB0, S2.P, X7-10.S; no longer IC1.RD1, X6-1.S
- net N$46: now also R5.2
- net N$47: now also IC4.2
- net N$48: now also R6.1
- net N$49: now also IC4.15
- net N$52: now also IC1.RD1, R7.2, X6-1.S; no longer IC1.RB0, X7-10.S
- net VSS: now also C6.2, LED2.C, S2.S1

Commit message: update
Parts:
- SPI: value 22-23-2101 -> LCD
- X1: value 332-02 -> RX-2
- X2: value 332-02 -> TX-2
- X3: value 332-02 -> RESETJMP
- X5: value 22-23-2101 -> PORTA
- X6: value 22-23-2101 -> PORTD
- X7: value 22-23-2101 -> PORTB
- renumbered X4 to SPI
Changed lines of the file:
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@@
 <part name="VSS33" library="supply1" library_urn="urn:adsk.eagle:library:371" deviceset="VSS" device=""/>
 <part name="VSS34" library="supply1" library_urn="urn:adsk.eagle:library:371" deviceset="VSS" device=""/>
-<part name="X1" library="con-garry" library_urn="urn:adsk.eagle:library:147" deviceset="332-02" device="" package3d_urn="urn:adsk.eagle:package:6810/1"/>
-<part name="X2" library="con-garry" library_urn="urn:adsk.eagle:library:147" deviceset="332-02" device="" package3d_urn="urn:adsk.eagle:package:6810/1"/>
+<part name="X1" library="con-garry" library_urn="urn:adsk.eagle:library:147" deviceset="332-02" device="" package3d_urn="urn:adsk.eagle:package:6810/1" value="RX-2"/>
+<part name="X2" library="con-garry" library_urn="urn:adsk.eagle:library:147" deviceset="332-02" device="" package3d_urn="urn:adsk.eagle:package:6810/1" value="TX-2"/>
 <part name="LED1" library="led" library_urn="urn:adsk.eagle:library:259" deviceset="LED" device="CHIPLED_1206" package3d_urn="urn:adsk.eagle:package:15823/2" value="RUN"/>
 <part name="R4" library="rcl" library_urn="urn:adsk.eagle:library:334" deviceset="R-US_" device="R1206" package3d_urn="urn:adsk.eagle:package:23540/2" value="220"/>
@@
 <part name="SV2" library="con-lstb" library_urn="urn:adsk.eagle:library:162" deviceset="MA04-1" device="" package3d_urn="urn:adsk.eagle:package:8337/1" value="DEBUG"/>
 <part name="VSS36" library="supply1" library_urn="urn:adsk.eagle:library:371" deviceset="VSS" device=""/>
-<part name="X3" library="con-garry" library_urn="urn:adsk.eagle:library:147" deviceset="332-02" device="" package3d_urn="urn:adsk.eagle:package:6810/1"/>
+<part name="X3" library="con-garry" library_urn="urn:adsk.eagle:library:147" deviceset="332-02" device="" package3d_urn="urn:adsk.eagle:package:6810/1" value="RESETJMP"/>
 <part name="VSS37" library="supply1" library_urn="urn:adsk.eagle:library:371" deviceset="VSS" device=""/>
 <part name="K1" library="relay" library_urn="urn:adsk.eagle:library:339" deviceset="G6K" device="-2P" package3d_urn="urn:adsk.eagle:package:24346/1"/>
 <part name="VSS9" library="supply1" library_urn="urn:adsk.eagle:library:371" deviceset="VSS" device=""/>
-<part name="X4" library="con-molex" library_urn="urn:adsk.eagle:library:165" deviceset="22-23-2101" device=""/>
-<part name="X5" library="con-molex" library_urn="urn:adsk.eagle:library:165" deviceset="22-23-2101" device=""/>
-<part name="X6" library="con-molex" library_urn="urn:adsk.eagle:library:165" deviceset="22-23-2101" device=""/>
+<part name="SPI" library="con-molex" library_urn="urn:adsk.eagle:library:165" deviceset="22-23-2101" device="" value="LCD"/>
+<part name="X5" library="con-molex" library_urn="urn:adsk.eagle:library:165" deviceset="22-23-2101" device="" value="PORTA"/>
+<part name="X6" library="con-molex" library_urn="urn:adsk.eagle:library:165" deviceset="22-23-2101" device="" value="PORTD"/>
 <part name="VDD7" library="supply1" library_urn="urn:adsk.eagle:library:371" deviceset="VDD" device=""/>
 <part name="VSS10" library="supply1" library_urn="urn:adsk.eagle:library:371" deviceset="VSS" device=""/>
@@
 <part name="VDD8" library="supply1" library_urn="urn:adsk.eagle:library:371" deviceset="VDD" device=""/>
 <part name="VSS12" library="supply1" library_urn="urn:adsk.eagle:library:371" deviceset="VSS" device=""/>
-<part name="X7" library="con-molex" library_urn="urn:adsk.eagle:library:165" deviceset="22-23-2101" device=""/>
+<part name="X7" library="con-molex" library_urn="urn:adsk.eagle:library:165" deviceset="22-23-2101" device="" value="PORTB"/>
 <part name="VSS13" library="supply1" library_urn="urn:adsk.eagle:library:371" deviceset="VSS" device=""/>
 <part name="VDD9" library="supply1" library_urn="urn:adsk.eagle:library:371" deviceset="VDD" device=""/>
@@
 <attribute name="VALUE" x="-78.74" y="-25.4" size="1.778" layer="96" rot="R90"/>
 </instance>
-<instance part="X4" gate="-1" x="144.78" y="86.36" smashed="yes">
+<instance part="SPI" gate="-1" x="144.78" y="86.36" smashed="yes">
 <attribute name="NAME" x="147.32" y="85.598" size="1.524" layer="95"/>
 <attribute name="VALUE" x="144.018" y="87.757" size="1.778" layer="96"/>
 </instance>
-<instance part="X4" gate="-2" x="144.78" y="83.82" smashed="yes">
+<instance part="SPI" gate="-2" x="144.78" y="83.82" smashed="yes">
 <attribute name="NAME" x="147.32" y="83.058" size="1.524" layer="95"/>
 </instance>
-<instance part="X4" gate="-3" x="144.78" y="81.28" smashed="yes">
+<instance part="SPI" gate="-3" x="144.78" y="81.28" smashed="yes">
 <attribute name="NAME" x="147.32" y="80.518" size="1.524" layer="95"/>
 </instance>
-<instance part="X4" gate="-4" x="144.78" y="78.74" smashed="yes">
+<instance part="SPI" gate="-4" x="144.78" y="78.74" smashed="yes">
 <attribute name="NAME" x="147.32" y="77.978" size="1.524" layer="95"/>
 </instance>
-<instance part="X4" gate="-5" x="144.78" y="76.2" smashed="yes">
+<instance part="SPI" gate="-5" x="144.78" y="76.2" smashed="yes">
 <attribute name="NAME" x="147.32" y="75.438" size="1.524" layer="95"/>
 </instance>
-<instance part="X4" gate="-6" x="144.78" y="73.66" smashed="yes">
+<instance part="SPI" gate="-6" x="144.78" y="73.66" smashed="yes">
 <attribute name="NAME" x="147.32" y="72.898" size="1.524" layer="95"/>
 </instance>
-<instance part="X4" gate="-7" x="144.78" y="71.12" smashed="yes">
+<instance part="SPI" gate="-7" x="144.78" y="71.12" smashed="yes">
 <attribute name="NAME" x="147.32" y="70.358" size="1.524" layer="95"/>
 </instance>
-<instance part="X4" gate="-8" x="144.78" y="68.58" smashed="yes">
+<instance part="SPI" gate="-8" x="144.78" y="68.58" smashed="yes">
 <attribute name="NAME" x="147.32" y="67.818" size="1.524" layer="95"/>
 </instance>
-<instance part="X4" gate="-9" x="144.78" y="66.04" smashed="yes">
+<instance part="SPI" gate="-9" x="144.78" y="66.04" smashed="yes">
 <attribute name="NAME" x="147.32" y="65.278" size="1.524" layer="95"/>
 </instance>
-<instance part="X4" gate="-10" x="144.78" y="63.5" smashed="yes">
+<instance part="SPI" gate="-10" x="144.78" y="63.5" smashed="yes">
 <attribute name="NAME" x="147.32" y="62.738" size="1.524" layer="95"/>
 </instance>
@@
 <segment>
 <pinref part="VDD7" gate="G$1" pin="VDD"/>
-<pinref part="X4" gate="-7" pin="S"/>
+<pinref part="SPI" gate="-7" pin="S"/>
 <wire x1="124.46" y1="71.12" x2="129.54" y2="71.12" width="0.1524" layer="91"/>
 <pinref part="C5" gate="G$1" pin="1"/>
@@
 <wire x1="129.54" y1="60.96" x2="132.08" y2="60.96" width="0.1524" layer="91"/>
 <wire x1="132.08" y1="60.96" x2="132.08" y2="68.58" width="0.1524" layer="91"/>
-<pinref part="X4" gate="-8" pin="S"/>
+<pinref part="SPI" gate="-8" pin="S"/>
 <wire x1="132.08" y1="68.58" x2="142.24" y2="68.58" width="0.1524" layer="91"/>
 <pinref part="C5" gate="G$1" pin="2"/>
@@
 <wire x1="139.7" y1="114.3" x2="139.7" y2="86.36" width="0.1524" layer="91"/>
 <wire x1="139.7" y1="86.36" x2="142.24" y2="86.36" width="0.1524" layer="91"/>
-<pinref part="X4" gate="-1" pin="S"/>
+<pinref part="SPI" gate="-1" pin="S"/>
 <junction x="142.24" y="86.36"/>
 <wire x1="142.24" y1="86.36" x2="144.78" y2="86.36" width="0.1524" layer="91"/>
@@
 <wire x1="43.18" y1="111.76" x2="137.16" y2="111.76" width="0.1524" layer="91"/>
 <wire x1="137.16" y1="111.76" x2="137.16" y2="83.82" width="0.1524" layer="91"/>
-<pinref part="X4" gate="-2" pin="S"/>
+<pinref part="SPI" gate="-2" pin="S"/>
 <wire x1="137.16" y1="83.82" x2="142.24" y2="83.82" width="0.1524" layer="91"/>
 <junction x="142.24" y="83.82"/>
@@
 <wire x1="58.42" y1="109.22" x2="134.62" y2="109.22" width="0.1524" layer="91"/>
 <wire x1="134.62" y1="109.22" x2="134.62" y2="81.28" width="0.1524" layer="91"/>
-<pinref part="X4" gate="-3" pin="S"/>
+<pinref part="SPI" gate="-3" pin="S"/>
 <wire x1="134.62" y1="81.28" x2="142.24" y2="81.28" width="0.1524" layer="91"/>
 <junction x="142.24" y="81.28"/>
@@
 <wire x1="81.28" y1="106.68" x2="132.08" y2="106.68" width="0.1524" layer="91"/>
 <wire x1="132.08" y1="106.68" x2="132.08" y2="78.74" width="0.1524" layer="91"/>
-<pinref part="X4" gate="-4" pin="S"/>
+<pinref part="SPI" gate="-4" pin="S"/>
 <wire x1="132.08" y1="78.74" x2="142.24" y2="78.74" width="0.1524" layer="91"/>
 <junction x="142.24" y="78.74"/>
@@
 <wire x1="60.96" y1="104.14" x2="129.54" y2="104.14" width="0.1524" layer="91"/>
 <wire x1="129.54" y1="104.14" x2="129.54" y2="76.2" width="0.1524" layer="91"/>
-<pinref part="X4" gate="-5" pin="S"/>
+<pinref part="SPI" gate="-5" pin="S"/>
 <wire x1="129.54" y1="76.2" x2="142.24" y2="76.2" width="0.1524" layer="91"/>
 <junction x="142.24" y="76.2"/>
@@
 <wire x1="127" y1="101.6" x2="127" y2="73.66" width="0.1524" layer="91"/>
 <wire x1="127" y1="73.66" x2="142.24" y2="73.66" width="0.1524" layer="91"/>
-<pinref part="X4" gate="-6" pin="S"/>
+<pinref part="SPI" gate="-6" pin="S"/>
 <junction x="142.24" y="73.66"/>
 <wire x1="142.24" y1="73.66" x2="144.78" y2="73.66" width="0.1524" layer="91"/>
@@
 <wire x1="137.16" y1="58.42" x2="137.16" y2="63.5" width="0.1524" layer="91"/>
 <wire x1="137.16" y1="63.5" x2="142.24" y2="63.5" width="0.1524" layer="91"/>
-<pinref part="X4" gate="-10" pin="S"/>
+<pinref part="SPI" gate="-10" pin="S"/>
 <junction x="142.24" y="63.5"/>
 <wire x1="142.24" y1="63.5" x2="144.78" y2="63.5" width="0.1524" layer="91"/>
@@
 <wire x1="111.76" y1="55.88" x2="139.7" y2="55.88" width="0.1524" layer="91"/>
 <wire x1="139.7" y1="55.88" x2="139.7" y2="66.04" width="0.1524" layer="91"/>
-<pinref part="X4" gate="-9" pin="S"/>
+<pinref part="SPI" gate="-9" pin="S"/>
 <wire x1="139.7" y1="66.04" x2="142.24" y2="66.04" width="0.1524" layer="91"/>
 <junction x="76.2" y="73.66"/>

Commit message: update
Parts:
- added R8, R9: 0, rcl:R-US_R1206
Connections:
- net GND: now also R9.1
- net VCC: now also R8.1
- net VDD: now also R8.2
- net VSS: now also R9.2
Changed lines of the file:
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@@
 <part name="VDD9" library="supply1" library_urn="urn:adsk.eagle:library:371" deviceset="VDD" device=""/>
 <part name="OPTIONS" library="con-molex" library_urn="urn:adsk.eagle:library:165" deviceset="22-23-2021" device=""/>
-<part name="VSS14" library="supply1" library_urn="urn:adsk.eagle:library:371" deviceset="VSS" device=""/>
 <part name="GND1" library="supply1" library_urn="urn:adsk.eagle:library:371" deviceset="GND" device=""/>
 <part name="GND2" library="supply1" library_urn="urn:adsk.eagle:library:371" deviceset="GND" device=""/>
@@
 <part name="VDD5" library="supply1" library_urn="urn:adsk.eagle:library:371" deviceset="VDD" device=""/>
 <part name="VSS7" library="supply1" library_urn="urn:adsk.eagle:library:371" deviceset="VSS" device=""/>
-<part name="VDD10" library="supply1" library_urn="urn:adsk.eagle:library:371" deviceset="VDD" device=""/>
 <part name="S1" library="switch-omron" library_urn="urn:adsk.eagle:library:377" deviceset="10-XX" device="" package3d_urn="urn:adsk.eagle:package:27496/1" value="RESETSW"/>
 <part name="VSS15" library="supply1" library_urn="urn:adsk.eagle:library:371" deviceset="VSS" device=""/>
@@
 <part name="LSP3" library="solpad" library_urn="urn:adsk.eagle:library:364" deviceset="LSP10" device="" package3d_urn="urn:adsk.eagle:package:26501/1"/>
 <part name="LSP4" library="solpad" library_urn="urn:adsk.eagle:library:364" deviceset="LSP10" device="" package3d_urn="urn:adsk.eagle:package:26501/1"/>
+<part name="R8" library="rcl" library_urn="urn:adsk.eagle:library:334" deviceset="R-US_" device="R1206" package3d_urn="urn:adsk.eagle:package:23540/2" value="0"/>
+<part name="R9" library="rcl" library_urn="urn:adsk.eagle:library:334" deviceset="R-US_" device="R1206" package3d_urn="urn:adsk.eagle:package:23540/2" value="0"/>
 </parts>
 <sheets>
@@
 <attribute name="NAME" x="27.178" y="-7.62" size="1.524" layer="95" rot="R270"/>
 </instance>
-<instance part="VSS14" gate="G$1" x="-106.68" y="60.96" smashed="yes" rot="R90">
-<attribute name="VALUE" x="-101.6" y="58.42" size="1.778" layer="96" rot="R180"/>
-</instance>
 <instance part="GND1" gate="1" x="132.08" y="-2.54" smashed="yes">
 <attribute name="VALUE" x="129.54" y="-5.08" size="1.778" layer="96"/>
 </instance>
-<instance part="GND2" gate="1" x="-101.6" y="53.34" smashed="yes">
-<attribute name="VALUE" x="-104.14" y="50.8" size="1.778" layer="96"/>
+<instance part="GND2" gate="1" x="-99.06" y="53.34" smashed="yes">
+<attribute name="VALUE" x="-101.6" y="50.8" size="1.778" layer="96"/>
 </instance>
 <instance part="P+1" gate="VCC" x="134.62" y="-10.16" smashed="yes" rot="R270">
@@
 <attribute name="VALUE" x="-88.9" y="78.74" size="1.778" layer="96" rot="R180"/>
 </instance>
-<instance part="P+4" gate="VCC" x="-111.76" y="71.12" smashed="yes" rot="R90">
-<attribute name="VALUE" x="-109.22" y="68.58" size="1.778" layer="96" rot="R180"/>
-</instance>
-<instance part="VDD5" gate="G$1" x="-106.68" y="66.04" smashed="yes" rot="R270">
-<attribute name="VALUE" x="-109.22" y="68.58" size="1.778" layer="96"/>
-</instance>
-<instance part="VSS7" gate="G$1" x="-109.22" y="53.34" smashed="yes">
-<attribute name="VALUE" x="-111.76" y="48.26" size="1.778" layer="96" rot="R90"/>
-</instance>
-<instance part="VDD10" gate="G$1" x="-106.68" y="71.12" smashed="yes" rot="R270">
-<attribute name="VALUE" x="-109.22" y="73.66" size="1.778" layer="96"/>
+<instance part="P+4" gate="VCC" x="-96.52" y="71.12" smashed="yes">
+<attribute name="VALUE" x="-99.06" y="68.58" size="1.778" layer="96" rot="R90"/>
+</instance>
+<instance part="VDD5" gate="G$1" x="-116.84" y="66.04" smashed="yes" rot="R180">
+<attribute name="VALUE" x="-114.3" y="68.58" size="1.778" layer="96" rot="R270"/>
+</instance>
+<instance part="VSS7" gate="G$1" x="-116.84" y="53.34" smashed="yes">
+<attribute name="VALUE" x="-119.38" y="48.26" size="1.778" layer="96" rot="R90"/>
 </instance>
 <instance part="S1" gate="1" x="152.4" y="-20.32" smashed="yes" rot="R180">
@@
 <instance part="LSP4" gate="1" x="-114.3" y="99.06" smashed="yes" rot="R90">
 <attribute name="NAME" x="-117.221" y="97.79" size="1.778" layer="95" rot="R90"/>
+</instance>
+<instance part="R8" gate="G$1" x="-106.68" y="68.58" smashed="yes" rot="R180">
+<attribute name="NAME" x="-102.87" y="67.0814" size="1.778" layer="95" rot="R180"/>
+<attribute name="VALUE" x="-102.87" y="71.882" size="1.778" layer="96" rot="R180"/>
+</instance>
+<instance part="R9" gate="G$1" x="-106.68" y="55.88" smashed="yes" rot="R180">
+<attribute name="NAME" x="-105.41" y="54.3814" size="1.778" layer="95" rot="R180"/>
+<attribute name="VALUE" x="-102.87" y="59.182" size="1.778" layer="96" rot="R180"/>
 </instance>
 </instances>
@@
 </segment>
 <segment>
-<wire x1="-109.22" y1="66.04" x2="-109.22" y2="71.12" width="0.1524" layer="91"/>
-<pinref part="P+4" gate="VCC" pin="VCC"/>
-<pinref part="VDD10" gate="G$1" pin="VDD"/>
-<junction x="-109.22" y="71.12"/>
 <pinref part="VDD5" gate="G$1" pin="VDD"/>
+<pinref part="R8" gate="G$1" pin="2"/>
+<wire x1="-116.84" y1="68.58" x2="-111.76" y2="68.58" width="0.1524" layer="91"/>
+<junction x="-111.76" y="68.58"/>
+<junction x="-116.84" y="68.58"/>
 </segment>
 </net>
@@
 </segment>
 <segment>
-<wire x1="-101.6" y1="55.88" x2="-109.22" y2="55.88" width="0.1524" layer="91"/>
-<wire x1="-109.22" y1="55.88" x2="-109.22" y2="60.96" width="0.1524" layer="91"/>
-<pinref part="GND2" gate="1" pin="GND"/>
-<pinref part="VSS7" gate="G$1" pin="VSS"/>
-<junction x="-109.22" y="55.88"/>
-<pinref part="VSS14" gate="G$1" pin="VSS"/>
-</segment>
-<segment>
 <pinref part="S1" gate="1" pin="S1"/>
 <pinref part="VSS15" gate="G$1" pin="VSS"/>
@@
 <pinref part="VSS18" gate="G$1" pin="VSS"/>
 <junction x="-116.84" y="27.94"/>
+</segment>
+<segment>
+<pinref part="VSS7" gate="G$1" pin="VSS"/>
+<pinref part="R9" gate="G$1" pin="2"/>
+<wire x1="-116.84" y1="55.88" x2="-111.76" y2="55.88" width="0.1524" layer="91"/>
+<junction x="-116.84" y="55.88"/>
+<junction x="-111.76" y="55.88"/>
 </segment>
 </net>
@@
 <junction x="-81.28" y="81.28"/>
 </segment>
+<segment>
+<pinref part="GND2" gate="1" pin="GND"/>
+<pinref part="R9" gate="G$1" pin="1"/>
+<wire x1="-99.06" y1="55.88" x2="-101.6" y2="55.88" width="0.1524" layer="91"/>
+<junction x="-101.6" y="55.88"/>
+<junction x="-99.06" y="55.88"/>
+</segment>
 </net>
 <net name="VCC" class="0">
@@
 <pinref part="C21" gate="G$1" pin="1"/>
 <pinref part="P+3" gate="VCC" pin="VCC"/>
+</segment>
+<segment>
+<pinref part="P+4" gate="VCC" pin="VCC"/>
+<pinref part="R8" gate="G$1" pin="1"/>
+<wire x1="-96.52" y1="68.58" x2="-101.6" y2="68.58" width="0.1524" layer="91"/>
+<junction x="-101.6" y="68.58"/>
+<junction x="-96.52" y="68.58"/>
 </segment>
 </net>
@@
 </sheet>
 </sheets>
-<errors>
-</errors>
 </schematic>
 </drawing>
