File: host_board/pic_k42.sch (EAGLE design)
At the start: 53 parts, among them IC1 PIC18F57K42-E_PT, IC2 REF3440IDBVR, IC3 MAX232, IC4 ILAMP, K1 G6K-2P, Q1 ASF1, X1 RX-2, X2 TX-2, X3 RESETJMP, X5 PORTA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

Commit message: update board to 1.2 spec
Parts:
- added C7: 0.1, rcl:C-USC1206
Connections:
- net GND: now also C7.2
- net VCC: now also C7.1
Changed lines of the file:
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@@
 <part name="R8" library="rcl" library_urn="urn:adsk.eagle:library:334" deviceset="R-US_" device="R1206" package3d_urn="urn:adsk.eagle:package:23540/2" value="0"/>
 <part name="R9" library="rcl" library_urn="urn:adsk.eagle:library:334" deviceset="R-US_" device="R1206" package3d_urn="urn:adsk.eagle:package:23540/2" value="0"/>
+<part name="C7" library="rcl" library_urn="urn:adsk.eagle:library:334" deviceset="C-US" device="C1206" package3d_urn="urn:adsk.eagle:package:23618/2" value="0.1"/>
+<part name="P+2" library="supply1" library_urn="urn:adsk.eagle:library:371" deviceset="VCC" device=""/>
+<part name="GND4" library="supply1" library_urn="urn:adsk.eagle:library:371" deviceset="GND" device=""/>
 </parts>
 <sheets>
@@
 <attribute name="NAME" x="-105.41" y="54.3814" size="1.778" layer="95" rot="R180"/>
 <attribute name="VALUE" x="-102.87" y="59.182" size="1.778" layer="96" rot="R180"/>
+</instance>
+<instance part="C7" gate="G$1" x="-83.82" y="68.58" smashed="yes" rot="R90">
+<attribute name="NAME" x="-84.455" y="69.596" size="1.778" layer="95" rot="R90"/>
+<attribute name="VALUE" x="-79.629" y="69.596" size="1.778" layer="96" rot="R90"/>
+</instance>
+<instance part="P+2" gate="VCC" x="-88.9" y="68.58" smashed="yes" rot="R90">
+<attribute name="VALUE" x="-86.36" y="66.04" size="1.778" layer="96" rot="R180"/>
+</instance>
+<instance part="GND4" gate="1" x="-78.74" y="66.04" smashed="yes">
+<attribute name="VALUE" x="-81.28" y="63.5" size="1.778" layer="96"/>
 </instance>
 </instances>
@@
 <junction x="-99.06" y="55.88"/>
 </segment>
+<segment>
+<pinref part="C7" gate="G$1" pin="2"/>
+<pinref part="GND4" gate="1" pin="GND"/>
+<junction x="-78.74" y="68.58"/>
+</segment>
 </net>
 <net name="VCC" class="0">
@@
 <pinref part="C21" gate="G$1" pin="1"/>
 <pinref part="P+3" gate="VCC" pin="VCC"/>
+<junction x="-88.9" y="81.28"/>
 </segment>
 <segment>
@@
 <junction x="-96.52" y="68.58"/>
 </segment>
-</net>
+<segment>
+<pinref part="C7" gate="G$1" pin="1"/>
+<pinref part="P+2" gate="VCC" pin="VCC"/>
+<junction x="-86.36" y="68.58"/>
+</segment>
+</net>

Commit message: update
Parts:
- removed R3: 0, rcl:R-US_R1206
Connections:
- removed net N$3: C1.2, R3.2
- net VSS: now also C1.2; no longer R3.1
Changed lines of the file:
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@@
 <part name="VDD2" library="supply1" library_urn="urn:adsk.eagle:library:371" deviceset="VDD" device=""/>
 <part name="VSS2" library="supply1" library_urn="urn:adsk.eagle:library:371" deviceset="VSS" device=""/>
-<part name="R3" library="rcl" library_urn="urn:adsk.eagle:library:334" deviceset="R-US_" device="R1206" package3d_urn="urn:adsk.eagle:package:23540/2" value="0"/>
 <part name="VDD3" library="supply1" library_urn="urn:adsk.eagle:library:371" deviceset="VDD" device=""/>
 <part name="VDD4" library="supply1" library_urn="urn:adsk.eagle:library:371" deviceset="VDD" device=""/>
@@
 <attribute name="VALUE" x="48.26" y="-2.54" size="1.778" layer="96" rot="R180"/>
 </instance>
-<instance part="VSS1" gate="G$1" x="58.42" y="-20.32" smashed="yes">
-<attribute name="VALUE" x="55.88" y="-25.4" size="1.778" layer="96" rot="R90"/>
+<instance part="VSS1" gate="G$1" x="58.42" y="-10.16" smashed="yes">
+<attribute name="VALUE" x="55.88" y="-15.24" size="1.778" layer="96" rot="R90"/>
 </instance>
 <instance part="VDD2" gate="G$1" x="58.42" y="-22.86" smashed="yes" rot="R90">
@@
 <instance part="VSS2" gate="G$1" x="55.88" y="-30.48" smashed="yes" rot="R270">
 <attribute name="VALUE" x="50.8" y="-27.94" size="1.778" layer="96"/>
-</instance>
-<instance part="R3" gate="G$1" x="58.42" y="-12.7" smashed="yes" rot="R90">
-<attribute name="NAME" x="56.9214" y="-16.51" size="1.778" layer="95" rot="R90"/>
-<attribute name="VALUE" x="61.722" y="-16.51" size="1.778" layer="96" rot="R90"/>
 </instance>
 <instance part="VDD3" gate="G$1" x="17.78" y="55.88" smashed="yes" rot="R180">
@@
 </segment>
 <segment>
-<pinref part="VSS1" gate="G$1" pin="VSS"/>
-<junction x="58.42" y="-17.78"/>
-<pinref part="R3" gate="G$1" pin="1"/>
-</segment>
-<segment>
 <pinref part="IC1" gate="G$1" pin="VSS_2"/>
 <wire x1="76.2" y1="60.96" x2="86.36" y2="60.96" width="0.1524" layer="91"/>
@@
 <junction x="-116.84" y="55.88"/>
 <junction x="-111.76" y="55.88"/>
+</segment>
+<segment>
+<pinref part="C1" gate="G$1" pin="2"/>
+<pinref part="VSS1" gate="G$1" pin="VSS"/>
+<junction x="58.42" y="-7.62"/>
 </segment>
 </net>
@@
 </segment>
 </net>
-<net name="N$3" class="0">
-<segment>
-<pinref part="C1" gate="G$1" pin="2"/>
-<pinref part="R3" gate="G$1" pin="2"/>
-<junction x="58.42" y="-7.62"/>
-</segment>
-</net>

Commit message: update
Parts:
- removed LSP1, LSP2, LSP3, LSP4: LSP10, solpad:LSP10
- removed OPTIONS: 22-23-2021, con-molex:22-23-2021
- added C9: 0.1, rcl:C-USC1206
- added LED3: DBLED, led:LEDCHIPLED_1206
- added R10, R11, R3: 220, rcl:R-US_R1206
- IC4: device ic-package:DIL16S -> ic-package:DIL8S
Connections:
- removed net N$67: IC4.3, LSP3.MP
- removed net N$68: IC4.4, LSP4.MP
- new net N$17: IC4.8, R6.2
- net GND: now also C9.2
- net N$25: now also R11.2
- net N$49: now also IC4.7; no longer IC4.15
- net N$55: now also IC4.5, R3.2; no longer IC4.14, LSP1.MP
- net N$58: now also R10.2
- net N$59: now also IC4.3
- net N$60: now also IC4.6; no longer OPTIONS-1.S
- net N$61: now also R3.1; no longer OPTIONS-2.S
- net N$63: now also IC4.4, R10.1; no longer IC4.16, R6.2
- net N$65: now also LED3.A, R11.1; no longer IC4.13, LSP2.MP
- net VCC: now also C9.1, Q1.OE
- net VDD: no longer Q1.OE
- net VSS: now also LED3.C

Commit message: update
Parts:
- added JMP2, JMP3: 0R-JUMPA, jump-0r-smd:0R-JUMPA
- added SV3: USBH, con-lstb:MA03-1
- added X4: MINI-USB-UX60A-MB-5ST, con-hirose:MINI-USB-UX60A-MB-5ST
Connections:
- new net N$67: SV3.1, X4.4
- new net N$68: SV3.2, X4.3
- new net N$69: SV3.3, X4.2
- net GND: now also JMP2-0R.2
- net VCC: now also JMP3-0R.2
- net VDD: now also JMP3-0R.1, X4.1
- net VSS: now also JMP2-0R.1, X4.5
Changed lines of the file:
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@@
 <part name="LED3" library="led" library_urn="urn:adsk.eagle:library:259" deviceset="LED" device="CHIPLED_1206" package3d_urn="urn:adsk.eagle:package:15823/2" value="DBLED"/>
 <part name="VSS14" library="supply1" library_urn="urn:adsk.eagle:library:371" deviceset="VSS" device=""/>
+<part name="GND5" library="supply1" library_urn="urn:adsk.eagle:library:371" deviceset="GND" device=""/>
+<part name="P+7" library="supply1" library_urn="urn:adsk.eagle:library:371" deviceset="VCC" device=""/>
+<part name="JMP2" library="jump-0r-smd" library_urn="urn:adsk.eagle:library:251" deviceset="0R-JUMP" device="A" package3d_urn="urn:adsk.eagle:package:15385/1"/>
+<part name="JMP3" library="jump-0r-smd" library_urn="urn:adsk.eagle:library:251" deviceset="0R-JUMP" device="A" package3d_urn="urn:adsk.eagle:package:15385/1"/>
+<part name="VSS19" library="supply1" library_urn="urn:adsk.eagle:library:371" deviceset="VSS" device=""/>
+<part name="VDD6" library="supply1" library_urn="urn:adsk.eagle:library:371" deviceset="VDD" device=""/>
+<part name="SV3" library="con-lstb" library_urn="urn:adsk.eagle:library:162" deviceset="MA03-1" device="" package3d_urn="urn:adsk.eagle:package:8339/1" value="USBH"/>
+<part name="X4" library="con-hirose" library_urn="urn:adsk.eagle:library:152" deviceset="MINI-USB-" device="UX60A-MB-5ST" package3d_urn="urn:adsk.eagle:package:7263/1"/>
 </parts>
 <sheets>
@@
 <instance part="VSS14" gate="G$1" x="149.86" y="40.64" smashed="yes" rot="R90">
 <attribute name="VALUE" x="154.94" y="38.1" size="1.778" layer="96" rot="R180"/>
+</instance>
+<instance part="GND5" gate="1" x="-109.22" y="48.26" smashed="yes">
+<attribute name="VALUE" x="-111.76" y="45.72" size="1.778" layer="96"/>
+</instance>
+<instance part="P+7" gate="VCC" x="-109.22" y="60.96" smashed="yes" rot="R180"/>
+<instance part="JMP2" gate="-0R" x="-111.76" y="53.34" smashed="yes">
+<attribute name="NAME" x="-109.22" y="54.61" size="1.778" layer="95"/>
+</instance>
+<instance part="JMP2" gate="G$2" x="-114.3" y="55.88" smashed="yes"/>
+<instance part="JMP3" gate="-0R" x="-111.76" y="66.04" smashed="yes">
+<attribute name="NAME" x="-109.22" y="67.31" size="1.778" layer="95"/>
+</instance>
+<instance part="JMP3" gate="G$2" x="-114.3" y="68.58" smashed="yes"/>
+<instance part="VSS19" gate="G$1" x="-78.74" y="-38.1" smashed="yes" rot="R90">
+<attribute name="VALUE" x="-73.66" y="-40.64" size="1.778" layer="96" rot="R180"/>
+</instance>
+<instance part="VDD6" gate="G$1" x="-78.74" y="-48.26" smashed="yes" rot="R270">
+<attribute name="VALUE" x="-81.28" y="-45.72" size="1.778" layer="96"/>
+</instance>
+<instance part="SV3" gate="G$1" x="-63.5" y="-43.18" smashed="yes" rot="R180">
+<attribute name="VALUE" x="-62.23" y="-35.56" size="1.778" layer="96" rot="R180"/>
+<attribute name="NAME" x="-62.23" y="-49.022" size="1.778" layer="95" rot="R180"/>
+</instance>
+<instance part="X4" gate="G$1" x="-86.36" y="-43.18" smashed="yes" rot="R180">
+<attribute name="NAME" x="-83.82" y="-54.61" size="1.778" layer="95" rot="R180"/>
+<attribute name="VALUE" x="-96.52" y="-35.56" size="1.778" layer="96" rot="R270"/>
 </instance>
 </instances>
@@
 <pinref part="R8" gate="G$1" pin="2"/>
 <wire x1="-116.84" y1="68.58" x2="-111.76" y2="68.58" width="0.3048" layer="91"/>
+<junction x="-116.84" y="68.58"/>
+<pinref part="JMP3" gate="-0R" pin="1"/>
 <junction x="-111.76" y="68.58"/>
-<junction x="-116.84" y="68.58"/>
+</segment>
+<segment>
+<pinref part="VDD6" gate="G$1" pin="VDD"/>
+<pinref part="X4" gate="G$1" pin="1"/>
+<junction x="-81.28" y="-48.26"/>
 </segment>
 </net>
@@
 <wire x1="-116.84" y1="55.88" x2="-111.76" y2="55.88" width="0.3048" layer="91"/>
 <junction x="-116.84" y="55.88"/>
+<pinref part="JMP2" gate="-0R" pin="1"/>
 <junction x="-111.76" y="55.88"/>
 </segment>
@@
 <pinref part="VSS14" gate="G$1" pin="VSS"/>
 <junction x="147.32" y="40.64"/>
+</segment>
+<segment>
+<pinref part="VSS19" gate="G$1" pin="VSS"/>
+<pinref part="X4" gate="G$1" pin="5"/>
+<junction x="-81.28" y="-38.1"/>
 </segment>
 </net>
@@
 <junction x="147.32" y="0"/>
 </segment>
+<segment>
+<pinref part="GND5" gate="1" pin="GND"/>
+<wire x1="-109.22" y1="53.34" x2="-109.22" y2="50.8" width="0.1524" layer="91"/>
+<junction x="-109.22" y="50.8"/>
+<pinref part="JMP2" gate="-0R" pin="2"/>
+<junction x="-109.22" y="53.34"/>
+</segment>
 </net>
 <net name="VCC" class="0">
@@
 <pinref part="P+6" gate="VCC" pin="VCC"/>
 <junction x="139.7" y="0"/>
+</segment>
+<segment>
+<pinref part="JMP3" gate="-0R" pin="2"/>
+<pinref part="P+7" gate="VCC" pin="VCC"/>
+<wire x1="-109.22" y1="66.04" x2="-109.22" y2="63.5" width="0.1524" layer="91"/>
+<junction x="-109.22" y="66.04"/>
+<junction x="-109.22" y="63.5"/>
 </segment>
 </net>
@@
 </segment>
 </net>
+<net name="N$67" class="0">
+<segment>
+<pinref part="SV3" gate="G$1" pin="1"/>
+<wire x1="-81.28" y1="-40.64" x2="-71.12" y2="-40.64" width="0.1524" layer="91"/>
+<junction x="-71.12" y="-40.64"/>
+<pinref part="X4" gate="G$1" pin="4"/>
+<junction x="-81.28" y="-40.64"/>
+</segment>
+</net>
+<net name="N$68" class="0">
+<segment>
+<wire x1="-81.28" y1="-43.18" x2="-71.12" y2="-43.18" width="0.1524" layer="91"/>
+<pinref part="SV3" gate="G$1" pin="2"/>
+<junction x="-71.12" y="-43.18"/>
+<wire x1="-71.12" y1="-43.18" x2="-68.58" y2="-43.18" width="0.1524" layer="91"/>
+<pinref part="X4" gate="G$1" pin="3"/>
+<junction x="-81.28" y="-43.18"/>
+</segment>
+</net>
+<net name="N$69" class="0">
+<segment>
+<pinref part="SV3" gate="G$1" pin="3"/>
+<wire x1="-81.28" y1="-45.72" x2="-71.12" y2="-45.72" width="0.1524" layer="91"/>
+<junction x="-71.12" y="-45.72"/>
+<pinref part="X4" gate="G$1" pin="2"/>
+<junction x="-81.28" y="-45.72"/>
+</segment>
+</net>

Commit message: update
Parts:
- removed LED1: RUN, led:LEDCHIPLED_1206
- removed LED2: MODE, led:LEDCHIPLED_1206
- removed S1: RESETSW, switch-omron:10-XX
- removed S2: MODESW, switch-omron:10-XX
- added S3: MODE SW, SamacSys_Parts:B3W-9000-Y1N
- added S4: RESET SW, SamacSys_Parts:B3W-9000-Y1N
Connections:
- net N$1: now also S4.4; no longer S1.P1
- net N$21: now also S4.+; no longer LED1.A
- net N$43: now also S3.4; no longer S2.P
- net N$64: now also S3.+; no longer LED2.A
- net VSS: now also S3.-, S3.2, S4.-, S4.2; no longer LED1.C, LED2.C, S1.S1, S2.S1

Commit message: up
Parts:
- added TP1, TP2: TPB1,27, testpad:TPB1,27
Connections:
- net VDD: now also TP2.TP
- net VSS: now also TP1.TP
Changed lines of the file:
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@@
 <?xml version="1.0" encoding="utf-8"?>
 <!DOCTYPE eagle SYSTEM "eagle.dtd">
-<eagle version="9.4.0">
+<eagle version="9.5.0">
 <drawing>
 <settings>
@@
 <part name="VSS32" library="supply1" library_urn="urn:adsk.eagle:library:371" deviceset="VSS" device=""/>
 <part name="VSS38" library="supply1" library_urn="urn:adsk.eagle:library:371" deviceset="VSS" device=""/>
+<part name="TP1" library="testpad" library_urn="urn:adsk.eagle:library:385" deviceset="TP" device="B1,27" package3d_urn="urn:adsk.eagle:package:27944/2"/>
+<part name="VSS15" library="supply1" library_urn="urn:adsk.eagle:library:371" deviceset="VSS" device=""/>
+<part name="TP2" library="testpad" library_urn="urn:adsk.eagle:library:385" deviceset="TP" device="B1,27" package3d_urn="urn:adsk.eagle:package:27944/2"/>
+<part name="VDD10" library="supply1" library_urn="urn:adsk.eagle:library:371" deviceset="VDD" device=""/>
 </parts>
 <sheets>
@@
 <instance part="VSS38" gate="G$1" x="167.64" y="-50.8" smashed="yes">
 <attribute name="VALUE" x="165.1" y="-55.88" size="1.778" layer="96" rot="R90"/>
+</instance>
+<instance part="TP1" gate="G$1" x="-111.76" y="-40.64" smashed="yes">
+<attribute name="NAME" x="-113.03" y="-39.37" size="1.778" layer="95"/>
+<attribute name="TP_SIGNAL_NAME" x="-110.49" y="-41.91" size="1.778" layer="97"/>
+</instance>
+<instance part="VSS15" gate="G$1" x="-111.76" y="-48.26" smashed="yes">
+<attribute name="VALUE" x="-114.3" y="-53.34" size="1.778" layer="96" rot="R90"/>
+</instance>
+<instance part="TP2" gate="G$1" x="-106.68" y="-40.64" smashed="yes">
+<attribute name="NAME" x="-107.95" y="-39.37" size="1.778" layer="95"/>
+<attribute name="TP_SIGNAL_NAME" x="-105.41" y="-41.91" size="1.778" layer="97"/>
+</instance>
+<instance part="VDD10" gate="G$1" x="-106.68" y="-48.26" smashed="yes" rot="R180">
+<attribute name="VALUE" x="-104.14" y="-45.72" size="1.778" layer="96" rot="R270"/>
 </instance>
 </instances>
@@
 <junction x="-81.28" y="-48.26"/>
 </segment>
+<segment>
+<pinref part="TP2" gate="G$1" pin="TP"/>
+<pinref part="VDD10" gate="G$1" pin="VDD"/>
+<wire x1="-106.68" y1="-45.72" x2="-106.68" y2="-43.18" width="0.1524" layer="91"/>
+</segment>
 </net>
 <net name="VSS" class="0">
@@
 <junction x="167.64" y="-48.26"/>
 </segment>
+<segment>
+<pinref part="TP1" gate="G$1" pin="TP"/>
+<pinref part="VSS15" gate="G$1" pin="VSS"/>
+<wire x1="-111.76" y1="-43.18" x2="-111.76" y2="-45.72" width="0.1524" layer="91"/>
+</segment>
 </net>

Commit message: up
Connections:
- net N$30 renamed LCD_MOSI
- net N$31 renamed LCD_SCK
- net N$33 renamed LCD_CS
- net N$52 renamed MODE_LED
Changed lines of the file:
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@@
 <?xml version="1.0" encoding="utf-8"?>
 <!DOCTYPE eagle SYSTEM "eagle.dtd">
-<eagle version="9.5.0">
+<eagle version="9.6.2">
 <drawing>
 <settings>
@@
 <wire x1="58.42" y1="17.78" x2="58.42" y2="10.16" width="0.1524" layer="91"/>
 <junction x="58.42" y="17.78"/>
+<junction x="58.42" y="10.16"/>
 </segment>
 </net>
@@
 <junction x="129.54" y="68.58"/>
 <junction x="142.24" y="71.12"/>
+<junction x="124.46" y="71.12"/>
 </segment>
 <segment>
@@
 <pinref part="VDD10" gate="G$1" pin="VDD"/>
 <wire x1="-106.68" y1="-45.72" x2="-106.68" y2="-43.18" width="0.1524" layer="91"/>
+<junction x="-106.68" y="-43.18"/>
+<junction x="-106.68" y="-45.72"/>
 </segment>
 </net>
@@
 <pinref part="C12" gate="G$1" pin="2"/>
 <pinref part="VSS24" gate="G$1" pin="VSS"/>
+<junction x="-30.48" y="-48.26"/>
 </segment>
 <segment>
 <pinref part="C11" gate="G$1" pin="2"/>
 <pinref part="VSS25" gate="G$1" pin="VSS"/>
+<junction x="-17.78" y="-48.26"/>
 </segment>
 <segment>
@@
 <pinref part="C14" gate="G$1" pin="2"/>
 <pinref part="VSS27" gate="G$1" pin="VSS"/>
+<junction x="99.06" y="-55.88"/>
 </segment>
 <segment>
 <pinref part="C15" gate="G$1" pin="2"/>
 <pinref part="VSS28" gate="G$1" pin="VSS"/>
+<junction x="109.22" y="-55.88"/>
 </segment>
 <segment>
 <pinref part="C13" gate="G$1" pin="2"/>
 <pinref part="VSS29" gate="G$1" pin="VSS"/>
+<junction x="127" y="-35.56"/>
 </segment>
 <segment>
 <pinref part="C16" gate="G$1" pin="2"/>
 <pinref part="VSS30" gate="G$1" pin="VSS"/>
+<junction x="127" y="-27.94"/>
 </segment>
 <segment>
@@
 <junction x="129.54" y="60.96"/>
 <junction x="142.24" y="68.58"/>
+<junction x="124.46" y="60.96"/>
 </segment>
 <segment>
@@
 <pinref part="VSS15" gate="G$1" pin="VSS"/>
 <wire x1="-111.76" y1="-43.18" x2="-111.76" y2="-45.72" width="0.1524" layer="91"/>
+<junction x="-111.76" y="-43.18"/>
+<junction x="-111.76" y="-45.72"/>
 </segment>
 </net>
@@
 </segment>
 </net>
-<net name="N$30" class="0">
+<net name="LCD_MOSI" class="0">
 <segment>
 <pinref part="IC1" gate="G$1" pin="RC5"/>
@@
 <junction x="142.24" y="83.82"/>
 <junction x="43.18" y="88.9"/>
-</segment>
-</net>
-<net name="N$31" class="0">
+<label x="111.76" y="83.82" size="1.778" layer="95"/>
+</segment>
+</net>
+<net name="LCD_SCK" class="0">
 <segment>
 <pinref part="IC1" gate="G$1" pin="RC3"/>
@@
 <junction x="142.24" y="81.28"/>
 <junction x="58.42" y="88.9"/>
+<label x="111.76" y="81.28" size="1.778" layer="95"/>
 </segment>
 </net>
@@
 </segment>
 </net>
-<net name="N$33" class="0">
+<net name="LCD_CS" class="0">
 <segment>
 <pinref part="IC1" gate="G$1" pin="RC2"/>
@@
 <junction x="142.24" y="76.2"/>
 <junction x="60.96" y="88.9"/>
+<label x="111.76" y="76.2" size="1.778" layer="95"/>
 </segment>
 </net>
@@
 </segment>
 </net>
-<net name="N$52" class="0">
+<net name="MODE_LED" class="0">
 <segment>
 <pinref part="R7" gate="G$1" pin="2"/>
@@
 <junction x="-25.4" y="63.5"/>
 <junction x="-116.84" y="45.72"/>
+<label x="-111.76" y="40.64" size="1.778" layer="95"/>
 </segment>
 </net>
@@
 <pinref part="Q1" gate="G$1" pin="VCC"/>
 <pinref part="P+1" gate="VCC" pin="VCC"/>
-</segment>
-<segment>
+<junction x="132.08" y="-10.16"/>
+</segment>
+<segment>
