File: host_board/mbmc_io.brd (EAGLE design)
At the start: 116.5 x 81.3 mm, 44 parts, among them X4 22-23-2101

Commit message: up
Parts:
- added C6: 0.1, rcl:C0805
- added J1: 1-1586043-4, 1-1586043-4:TE_1-1586043-4
- added J2: 1586044-4, 1586044-4:TE_1586044-4
- added OUTP: 22-23-2101, con-molex:22-23-2101
- moved R22 46.0 mm to (57.1, 47.0)
- moved R23 35.9 mm to (52.1, 47.0)
- moved R30 35.9 mm to (16.5, 47.0)
- moved C1 29.3 mm to (109.2, 66.0)
- moved R24 25.9 mm to (47.0, 47.0)
- moved R29 25.9 mm to (21.6, 47.0)
- moved R25 16.1 mm to (41.9, 47.0)
- moved R28 16.1 mm to (26.7, 47.0)
- moved IC1 11.5 mm to (20.3, 58.4)
- moved R26 7.18 mm to (36.8, 47.0)
- moved R27 7.18 mm to (31.8, 47.0)
- moved R11 5.08 mm to (11.4, 47.0)
- moved R12 3.81 mm to (11.4, 43.2)
- moved R13 3.81 mm to (16.5, 43.2)
- moved R14 3.81 mm to (21.6, 43.2)
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- renumbered X4 to INP
Connections:
- new net +12V: J2.3
- new net +24V: C6.1, IC1.10, J2.4, OUTP.8
- new net N$44: INP.10, U$1.IN1
- new net N$46: INP.1, U$1.IN2
- new net N$47: INP.2, U$1.IN3
- new net N$48: INP.3, U$1.IN4
- new net N$49: INP.4, U$1.IN5
- new net N$50: INP.5, U$1.IN6
- new net N$51: INP.6, U$1.IN7
- new net N$52: INP.7, U$1.IN8
- new net N$53: IC1.18, OUTP.10
- new net N$54: IC1.17, OUTP.1
- new net N$55: IC1.16, OUTP.2
- new net N$56: IC1.15, OUTP.3
- new net N$57: IC1.14, OUTP.4
- new net N$58: IC1.13, OUTP.5
- new net N$59: IC1.12, OUTP.6
- new net N$60: IC1.11, OUTP.7
- new net N$62: SPI_IN.6, SPI_OUT.6
- new net N$63: SPI_IN.5, SPI_OUT.5
- new net N$64: SPI_IN.4, SPI_OUT.4
- new net N$65: SPI_IN.3, SPI_OUT.3
- new net N$66: SPI_IN.2, SPI_OUT.2
- new net N$67: SPI_IN.1, SPI_OUT.1
- net VDD: now also J2.2
- net VSS: now also C6.2, J2.1, OUTP.9
Routing:
- net +24V: track 0.00 -> 88.4 mm
- net N$32: track 153.0 -> 96.1 mm, vias 0 -> 2
- net VDD: track 187.2 -> 230.3 mm
- net N$10: track 81.9 -> 45.7 mm, vias 0 -> 1
- net N$20: track 49.2 -> 13.7 mm, vias 1 -> 0
- net N$38: track 116.7 -> 84.4 mm, vias 0 -> 1
- net N$44: track 0.00 -> 31.0 mm
- net N$53: track 0.00 -> 30.2 mm
- net N$40: track 100.3 -> 121.7 mm, vias 1 -> 2
- net N$19: track 32.6 -> 12.1 mm, vias 1 -> 0
- net N$52: track 0.00 -> 20.4 mm
- net N$46: track 0.00 -> 19.7 mm
- net N$51: track 0.00 -> 19.7 mm
- net N$31: track 160.4 -> 140.9 mm
- net N$34: track 117.1 -> 97.6 mm, vias 1 -> 0
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
Commit message: up
Parts:
- added C10, C11, C7, C8, C9: 0.1, rcl:C0805
- added C12: 22uf, rcl:C0805
- added IC3: REF02 5 VOLTS, linear:DIL08
- added IC4: 5 VOLTS, linear:TO220V
- added IC5: 12 VOLTS, linear:TO220V
- added IC6: 3.3 VOLTS, linear:TO220V
- added LED1: 24 on, led:CHIPLED_1206
- added LED2: 12 on, led:CHIPLED_1206
- added LED3: 5 on, led:CHIPLED_1206
- added LED4: 3.3 on, led:CHIPLED_1206
- added LED5: debug8, led:CHIPLED_1206
- added R31, R32, R33, R34, R35: (no value), rcl:R0805
- added SL1: 3.3 GLORY, con-amp-quick:02P
- IC1: value (none) -> ULN2803
- IC2: value (none) -> DIP Socket
- moved C4 5.39 mm to (74.9, 11.4)
- moved J2 3.81 mm to (97.8, 50.8)
Connections:
- new net +3V3: C8.1, IC6.3, J1.13, R34.2, SL1.2
- new net N$24: J1.2, R14.1
- new net N$61: C7.1, IC3.6, J1.14
- new net N$68: J1.4, R16.1
- new net N$69: J1.9, R11.1
- new net N$70: J1.3, R15.1
- new net N$71: J1.10, R10.3, R20.1, R20.2
- new net N$72: J1.5, R12.1
- new net N$73: J1.6, R17.1
- new net N$74: J1.1, R13.1
- new net N$76: LED1.A, R31.1
- new net N$77: LED2.A, R32.1
- new net N$78: LED3.A, R33.1
- new net N$79: LED4.A, R34.1
- new net N$80: LED5.A, R35.1
- new net N$81: R35.2, U$1.OUT8
- net +12V: now also C11.1, C12.1, C9.1, IC3.2, IC5.3, R32.2
- net +24V: now also IC4.1, IC5.1, IC6.1, R31.2
- net N$10: now also J1.8, R19.2; no longer R10.3, R20.2
- net N$8: now also J1.7, R18.1
- net N$9: now also R19.1; no longer R19.2
- net VDD: now also C10.1, IC4.3, J1.12, R33.2
- net VSS: now also C10.2, C11.2, C12.2, C7.2, C8.2, C9.2, IC3.4, IC4.2, IC5.2, IC6.2, J1.11, LED1.C, LED2.C, LED3.C, LED4.C, LED5.C, SL1.1
Routing:
- net +12V: track 0.00 -> 90.0 mm, vias 0 -> 2
- net +3V3: track 0.00 -> 88.9 mm, vias 0 -> 2
- net VSS: track 103.5 -> 191.6 mm, vias 7 -> 6
- net N$77: track 0.00 -> 87.3 mm
- net N$33: track 98.2 -> 171.2 mm, vias 1 -> 0
- net N$69: track 0.00 -> 71.8 mm, vias 0 -> 1
- net N$71: track 0.00 -> 68.4 mm, vias 0 -> 1
- net N$72: track 0.00 -> 62.6 mm, vias 0 -> 1
- net N$78: track 0.00 -> 57.8 mm
- net N$79: track 0.00 -> 47.2 mm, vias 0 -> 2
- net N$3: track 68.9 -> 115.1 mm, vias 1 -> 0
- net N$70: track 0.00 -> 44.7 mm, vias 0 -> 1
- net N$74: track 0.00 -> 44.6 mm, vias 0 -> 2
- net VDD: track 230.3 -> 274.6 mm, vias 2 -> 3
- net N$76: track 0.00 -> 40.8 mm
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Other:
- board text added: "FGB@MCHP 1.0"
- board text added: "MBMC IO BOARD"
- board text added: "POWER"

Commit message: up
Parts:
- added SL2: PWM, con-amp-quick:02P
- added SL3: MISC INP, con-amp-quick:04P
- moved SL1 8.89 mm to (67.3, 26.7)
- moved C6 2.54 mm to (26.7, 66.0)
Connections:
- new net N$82: P-D.1, SL2.2
- new net N$83: SL3.2, U$1.OUT6
- new net N$84: SL3.3, U$1.OUT7
- net N$81: now also SL3.4
- net VSS: now also SL2.1, SL3.1
Routing:
- net VSS: track 191.6 -> 495.7 mm, vias 6 -> 4
- net N$3: track 115.1 -> 55.1 mm, vias 0 -> 1
- net N$33: track 171.2 -> 134.7 mm
- net N$84: track 0.00 -> 35.4 mm, vias 0 -> 2
- net N$71: track 68.4 -> 103.7 mm
- net N$77: track 87.3 -> 51.9 mm, vias 0 -> 2
- net N$74: track 44.6 -> 75.0 mm, vias 2 -> 0
- net N$81: track 29.4 -> 59.1 mm, vias 2 -> 3
- net N$13: track 60.5 -> 31.4 mm, vias 0 -> 2
- net N$36: track 77.8 -> 48.8 mm
- net N$83: track 0.00 -> 28.6 mm, vias 0 -> 1
- net VDD: track 274.6 -> 302.0 mm
- net N$15: track 46.1 -> 69.9 mm
- net +3V3: track 88.9 -> 110.4 mm, vias 2 -> 0
- net N$82: track 0.00 -> 18.9 mm
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- removed copper zone on layer 16, net VSS

Commit message: up, order pcb
Parts:
- R1, R10, R2, R3, R4, R5, R6, R7, R8, R9: value (none) -> 200
- R11, R12, R15, R16, R17, R18, R19, R20: value (none) -> 9.85k
- R13, R14: value (none) -> 811
- R21, R22: value (none) -> 3820
- R23, R24, R25, R26, R27, R28, R29, R30: value (none) -> 1.28k
- R31: value (none) -> 10k
- R32: value (none) -> 5k
- R33, R34, R35: value (none) -> 1k
Routing:
- net VDD: track 302.0 -> 258.0 mm, vias 3 -> 5
- net N$74: track 75.0 -> 44.6 mm, vias 0 -> 3
- net N$31: track 150.2 -> 129.6 mm, vias 0 -> 1
- net N$14: track 59.8 -> 39.4 mm, vias 1 -> 3
- net N$32: track 139.5 -> 155.6 mm
- net +3V3: track 110.4 -> 94.8 mm, vias 0 -> 1
- net VSS: track 495.7 -> 480.5 mm, vias 4 -> 6
- net N$43: track 75.9 -> 62.2 mm, vias 1 -> 2
- net N$71: track 103.7 -> 92.2 mm, vias 1 -> 2
- net N$36: track 48.8 -> 60.1 mm
- net N$72: track 61.5 -> 72.4 mm
- net +24V: track 139.7 -> 129.1 mm
- net N$77: track 51.9 -> 41.9 mm
- net N$38: track 122.6 -> 112.7 mm
- net +12V: track 93.8 -> 84.5 mm, vias 2 -> 4
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