File: host_board/mbmc_io.brd (EAGLE design)
At the start: 116.5 x 81.3 mm, 71 parts, among them IC1 ULN2803, IC2 DIP Socket, IC3 REF02 5 VOLTS, IC4 5 VOLTS, IC5 12 VOLTS, IC6 3.3 VOLTS, J1 1-1586043-4, J2 1586044-4

Commit message: up
Parts:
- R19: value 9.85k -> 811
- R28: value 1.28k -> 3820
Changed lines of the file:
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@@
 <attribute name="VALUE" x="41.275" y="40.64" size="1.27" layer="27"/>
 </element>
-<element name="R19" library="rcl" library_urn="urn:adsk.eagle:library:334" package="R0805" package3d_urn="urn:adsk.eagle:package:23553/2" value="9.85k" x="46.99" y="43.18" smashed="yes">
+<element name="R19" library="rcl" library_urn="urn:adsk.eagle:library:334" package="R0805" package3d_urn="urn:adsk.eagle:package:23553/2" value="811" x="46.99" y="43.18" smashed="yes">
 <attribute name="NAME" x="46.355" y="44.45" size="1.27" layer="25"/>
 <attribute name="POPULARITY" value="85" x="88.9" y="-13.97" size="1.778" layer="27" display="off"/>
@@
 <attribute name="VALUE" x="31.115" y="44.45" size="1.27" layer="27"/>
 </element>
-<element name="R28" library="rcl" library_urn="urn:adsk.eagle:library:334" package="R0805" package3d_urn="urn:adsk.eagle:package:23553/2" value="1.28k" x="26.67" y="46.99" smashed="yes">
+<element name="R28" library="rcl" library_urn="urn:adsk.eagle:library:334" package="R0805" package3d_urn="urn:adsk.eagle:package:23553/2" value="3820" x="26.67" y="46.99" smashed="yes">
 <attribute name="NAME" x="26.035" y="48.26" size="1.27" layer="25"/>
 <attribute name="POPULARITY" value="85" x="68.58" y="-15.24" size="1.778" layer="27" display="off"/>

Commit message: up
Parts:
- added INT0, VREF4095: TPB1,27, testpad:B1,27
Connections:
- new net N$85: P-A.3, VREF4095.TP
- new net N$87: INT0.TP, P-B.10
- net N$43: now also P-D.3; no longer P-A.3
- net N$81: now also P-D.2
Routing:
- net VSS: track 480.5 -> 429.3 mm, vias 6 -> 10
- net N$34: track 151.8 -> 110.1 mm, vias 1 -> 2
- net N$43: track 62.2 -> 25.7 mm, vias 2 -> 1
- net N$77: track 41.9 -> 70.4 mm, vias 2 -> 0
- net N$33: track 132.9 -> 105.8 mm
- net N$14: track 39.4 -> 63.5 mm, vias 3 -> 1
- net N$31: track 129.6 -> 106.5 mm, vias 1 -> 0
- net N$74: track 44.6 -> 65.1 mm, vias 3 -> 0
- net N$32: track 155.6 -> 136.4 mm, vias 0 -> 1
- net +3V3: track 94.8 -> 76.1 mm
- net +24V: track 129.1 -> 112.8 mm, vias 1 -> 2
- net +12V: track 84.5 -> 100.2 mm, vias 4 -> 3
- net N$38: track 112.7 -> 97.1 mm, vias 1 -> 2
- net N$37: track 103.9 -> 118.0 mm
- net VDD: track 258.0 -> 245.3 mm, vias 5 -> 3
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Other:
- board text added: "FGB@MCHP 1.1"
- board text removed: "FGB@MCHP 1.0"

Commit message: up
Connections:
- removed net N$83: SL3.2, U$1.OUT6
- new net N$86: P-D.2, SL3.2, U$1.OUT6
- net N$35: now also IC2.8
- net N$36: now also IC2.7, U$1.EN_L
- net N$81: no longer P-D.2
- net VSS: now also IC2.1; no longer U$1.EN_L
Routing:
- net N$35: track 50.9 -> 177.1 mm, vias 0 -> 1
- net N$36: track 51.4 -> 142.1 mm, vias 1 -> 6
- net N$86: track 0.00 -> 40.9 mm, vias 0 -> 1
- net N$34: track 110.1 -> 141.8 mm, vias 2 -> 1
- net N$83: track 30.7 -> 0.00 mm, vias 1 -> 0
- net VDD: track 245.3 -> 270.7 mm
- net N$32: track 136.4 -> 112.1 mm, vias 1 -> 3
- net N$74: track 65.1 -> 42.1 mm, vias 0 -> 3
- net N$15: track 64.5 -> 45.1 mm, vias 1 -> 3
- net +24V: track 112.8 -> 96.8 mm
- net +3V3: track 76.1 -> 91.3 mm, vias 1 -> 2
- net N$72: track 72.3 -> 58.9 mm
- net N$71: track 90.7 -> 77.5 mm
- net +12V: track 100.2 -> 87.6 mm, vias 3 -> 6
- net N$78: track 50.3 -> 62.3 mm
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
Commit message: up
Parts:
- moved IC6 3.81 mm to (39.4, 57.1)
- moved IC1 2.54 mm to (17.8, 58.4)
Connections:
- new net N$83: R10.3, R20.1
- new net N$88: R18.1, R7.3
- net N$71: no longer R10.3, R20.1
- net N$8: no longer R18.1, R7.3
Routing:
- net N$71: track 77.5 -> 22.0 mm, vias 2 -> 1
- net N$78: track 62.3 -> 104.4 mm, vias 2 -> 0
- net N$34: track 141.8 -> 101.0 mm, vias 1 -> 2
- net N$83: track 0.00 -> 39.6 mm, vias 0 -> 1
- net VDD: track 270.7 -> 237.1 mm, vias 3 -> 2
- net N$32: track 112.1 -> 143.8 mm, vias 3 -> 1
- net N$77: track 69.7 -> 42.2 mm, vias 0 -> 2
- net N$10: track 24.5 -> 51.0 mm, vias 1 -> 0
- net VSS: track 437.5 -> 462.9 mm, vias 3 -> 5
- net N$15: track 45.1 -> 66.8 mm, vias 3 -> 2
- net N$37: track 114.6 -> 93.1 mm
- net N$24: track 53.2 -> 32.5 mm, vias 0 -> 2
- net N$16: track 37.2 -> 21.9 mm, vias 0 -> 1
- net N$8: track 51.9 -> 37.1 mm, vias 0 -> 2
- net N$73: track 29.8 -> 44.0 mm
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
Commit message: up
Parts:
- added REF12V, REF24V, REF3.3V, REFVDD, REFVSS, VREF5VREF: TPB1,27, testpad:B1,27
- added SL4: SPI SEL, con-amp-quick:04P
- moved C1 29.2 mm to (80.0, 64.8), turned to 270 degrees
- moved SPI_OUT 1.27 mm to (94.0, 72.4)
Connections:
- net +12V: now also REF12V.TP
- net +24V: now also REF24V.TP
- net +3V3: now also REF3.3V.TP
- net N$39: now also SL4.3
- net N$45: now also SL4.4
- net N$61: now also VREF5VREF.TP
- net VDD: now also REFVDD.TP, SL4.2
- net VSS: now also REFVSS.TP, SL4.1
Routing:
- net N$34: track 101.0 -> 170.6 mm, vias 2 -> 0
- net N$78: track 104.4 -> 54.1 mm, vias 0 -> 4
- net VDD: track 237.1 -> 268.5 mm
- net N$37: track 93.1 -> 123.0 mm
- net N$10: track 51.0 -> 26.3 mm, vias 0 -> 2
- net N$32: track 143.8 -> 121.6 mm, vias 1 -> 0
- net N$40: track 100.0 -> 120.7 mm
- net N$36: track 151.1 -> 168.8 mm
- net +3V3: track 92.8 -> 110.0 mm, vias 3 -> 2
- net N$15: track 66.8 -> 50.5 mm
- net N$69: track 77.9 -> 61.6 mm, vias 0 -> 2
- net N$43: track 18.6 -> 31.8 mm
- net N$35: track 169.6 -> 157.5 mm, vias 0 -> 1
- net N$68: track 30.7 -> 41.9 mm, vias 0 -> 3
- net N$8: track 37.1 -> 46.3 mm
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