File: host_board/mbmc_io.sch (EAGLE design)
At the start: 40 parts, among them X1 22-23-2101, X2 22-23-2101, X3 22-23-2101, X4 22-23-2101

Commit message: up
Parts:
- added C5: 0.1, rcl:C-USC0805
- added IC1: (no value), uln-udn:ULN2803A
- added IC2: (no value), ic-package:DIL8S
- added U$1: MAX6818, MAX6818:MAX6818
- renumbered X1 to P-B, X2 to P-A, X3 to P-D
Connections:
- new net N$31: IC1.I1, P-D-4.S
- new net N$32: IC1.I2, P-D-5.S
- new net N$33: IC1.I3, P-D-6.S
- new net N$34: IC1.I4, P-D-7.S
- new net N$35: IC1.I5, P-B-6.S
- new net N$36: IC1.I6, P-B-7.S
- new net N$37: IC1.I7, IC2.5
- new net N$38: IC1.I8, IC2.6
- new net N$39: SPI_IN-9.S, SPI_OUT-9.S, U$1.OUT1
- new net N$40: P-B-1.S, U$1.CH_L
- new net N$41: P-D-9.S, U$1.OUT3
- new net N$42: P-D-8.S, U$1.OUT4
- new net N$43: P-A-3.S, U$1.OUT5
- new net N$45: SPI_IN-10.S, SPI_OUT-10.S, U$1.OUT2
- net VDD: now also C5.1, U$1.VCC
- net VSS: now also C5.2, IC1.GND, U$1.EN_L, U$1.GND

Commit message: up
Parts:
- added C6: 0.1, rcl:C-USC0805
- added J1: 1-1586043-4, 1-1586043-4:1-1586043-4
- added J2: 1586044-4, 1586044-4:1586044-4
- added OUTP: 22-23-2101, con-molex:22-23-2101
- renumbered X4 to INP
Connections:
- new net +12V: J2.3
- new net +24V: C6.1, IC1.CD+, J2.4, OUTP-8.S
- new net N$44: INP-10.S, U$1.IN1
- new net N$46: INP-1.S, U$1.IN2
- new net N$47: INP-2.S, U$1.IN3
- new net N$48: INP-3.S, U$1.IN4
- new net N$49: INP-4.S, U$1.IN5
- new net N$50: INP-5.S, U$1.IN6
- new net N$51: INP-6.S, U$1.IN7
- new net N$52: INP-7.S, U$1.IN8
- new net N$53: IC1.O1, OUTP-10.S
- new net N$54: IC1.O2, OUTP-1.S
- new net N$55: IC1.O3, OUTP-2.S
- new net N$56: IC1.O4, OUTP-3.S
- new net N$57: IC1.O5, OUTP-4.S
- new net N$58: IC1.O6, OUTP-5.S
- new net N$59: IC1.O7, OUTP-6.S
- new net N$60: IC1.O8, OUTP-7.S
- new net N$62: SPI_IN-6.S, SPI_OUT-6.S
- new net N$63: SPI_IN-5.S, SPI_OUT-5.S
- new net N$64: SPI_IN-4.S, SPI_OUT-4.S
- new net N$65: SPI_IN-3.S, SPI_OUT-3.S
- new net N$66: SPI_IN-2.S, SPI_OUT-2.S
- new net N$67: SPI_IN-1.S, SPI_OUT-1.S
- net VDD: now also J2.2
- net VSS: now also C6.2, J2.1, OUTP-9.S
Other:
- moved on the sheet: IC1

Commit message: up
Parts:
- added C10, C11, C7, C8, C9: 0.1, rcl:C-USC0805
- added C12: 22uf, rcl:C-USC0805
- added IC3: REF02 5 VOLTS, linear:REF02Z
- added IC4: 5 VOLTS, linear:7805TV
- added IC5: 12 VOLTS, linear:7805TV
- added IC6: 3.3 VOLTS, linear:7805TV
- added LED1: 24 on, led:LEDCHIPLED_1206
- added LED2: 12 on, led:LEDCHIPLED_1206
- added LED3: 5 on, led:LEDCHIPLED_1206
- added LED4: 3.3 on, led:LEDCHIPLED_1206
- added LED5: debug8, led:LEDCHIPLED_1206
- added R31, R32, R33, R34, R35: (no value), rcl:R-US_R0805
- added SL1: 3.3 GLORY, con-amp-quick:M02
- IC1: value (none) -> ULN2803
- IC2: value (none) -> DIP Socket
Connections:
- new net +3V3: C8.1, IC6.VO, J1.13, R34.2, SL1.2
- new net N$24: J1.2, R14.1
- new net N$61: C7.1, IC3.VO, J1.14
- new net N$68: J1.4, R16.1
- new net N$69: J1.9, R11.1
- new net N$70: J1.3, R15.1
- new net N$71: J1.10, R10.E, R20.1, R20.2
- new net N$72: J1.5, R12.1
- new net N$73: J1.6, R17.1
- new net N$74: J1.1, R13.1
- new net N$76: LED1.A, R31.1
- new net N$77: LED2.A, R32.1
- new net N$78: LED3.A, R33.1
- new net N$79: LED4.A, R34.1
- new net N$80: LED5.A, R35.1
- new net N$81: R35.2, U$1.OUT8
- net +12V: now also C11.1, C12.1, C9.1, IC3.V+, IC5.VO, R32.2
- net +24V: now also IC4.VI, IC5.VI, IC6.VI, R31.2
- net N$10: now also J1.8, R19.2; no longer R10.E, R20.2
- net N$8: now also J1.7, R18.1
- net N$9: now also R19.1; no longer R19.2
- net VDD: now also C10.1, IC4.VO, J1.12, R33.2
- net VSS: now also C10.2, C11.2, C12.2, C7.2, C8.2, C9.2, IC3.GND, IC4.GND, IC5.GND, IC6.GND, J1.11, LED1.C, LED2.C, LED3.C, LED4.C, LED5.C, SL1.1
Other:
- moved on the sheet: R17, R18, R19, R20, R25

Commit message: up
Parts:
- added SL2: PWM, con-amp-quick:M02
- added SL3: MISC INP, con-amp-quick:M04
Connections:
- new net N$82: P-D-1.S, SL2.2
- new net N$83: SL3.2, U$1.OUT6
- new net N$84: SL3.3, U$1.OUT7
- net N$81: now also SL3.4
- net VSS: now also SL2.1, SL3.1
Changed lines of the file:
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@@
 <part name="+3V4" library="supply1" library_urn="urn:adsk.eagle:library:371" deviceset="+3V3" device=""/>
 <part name="VSS35" library="supply1" library_urn="urn:adsk.eagle:library:371" deviceset="VSS" device=""/>
+<part name="SL2" library="con-amp-quick" library_urn="urn:adsk.eagle:library:125" deviceset="M02" device="" package3d_urn="urn:adsk.eagle:package:5956/1" value="PWM"/>
+<part name="VSS36" library="supply1" library_urn="urn:adsk.eagle:library:371" deviceset="VSS" device=""/>
+<part name="SL3" library="con-amp-quick" library_urn="urn:adsk.eagle:library:125" deviceset="M04" device="" package3d_urn="urn:adsk.eagle:package:5958/1" value="MISC INP"/>
+<part name="VSS37" library="supply1" library_urn="urn:adsk.eagle:library:371" deviceset="VSS" device=""/>
 </parts>
 <sheets>
@@
 <instance part="VSS35" gate="G$1" x="-33.02" y="-68.58" smashed="yes" rot="R180">
 <attribute name="VALUE" x="-30.48" y="-63.5" size="1.778" layer="96" rot="R270"/>
+</instance>
+<instance part="SL2" gate="G$1" x="73.66" y="-2.54" smashed="yes" rot="R180">
+<attribute name="VALUE" x="76.2" y="2.54" size="1.778" layer="96" rot="R180"/>
+<attribute name="NAME" x="76.2" y="-8.382" size="1.778" layer="95" rot="R180"/>
+</instance>
+<instance part="VSS36" gate="G$1" x="66.04" y="7.62" smashed="yes" rot="R180">
+<attribute name="VALUE" x="68.58" y="12.7" size="1.778" layer="96" rot="R270"/>
+</instance>
+<instance part="SL3" gate="G$1" x="195.58" y="83.82" smashed="yes" rot="R270">
+<attribute name="VALUE" x="187.96" y="88.9" size="1.778" layer="96" rot="R270"/>
+<attribute name="NAME" x="203.962" y="88.9" size="1.778" layer="95" rot="R270"/>
+</instance>
+<instance part="VSS37" gate="G$1" x="185.42" y="78.74" smashed="yes" rot="R270">
+<attribute name="VALUE" x="180.34" y="81.28" size="1.778" layer="96"/>
 </instance>
 </instances>
@@
 <wire x1="-33.02" y1="-71.12" x2="-33.02" y2="-76.2" width="0.1524" layer="91"/>
 </segment>
+<segment>
+<pinref part="SL2" gate="G$1" pin="1"/>
+<pinref part="VSS36" gate="G$1" pin="VSS"/>
+<wire x1="66.04" y1="5.08" x2="66.04" y2="-2.54" width="0.1524" layer="91"/>
+<junction x="66.04" y="-2.54"/>
+<junction x="66.04" y="5.08"/>
+</segment>
+<segment>
+<pinref part="SL3" gate="G$1" pin="1"/>
+<pinref part="VSS37" gate="G$1" pin="VSS"/>
+<wire x1="187.96" y1="78.74" x2="193.04" y2="78.74" width="0.1524" layer="91"/>
+<junction x="193.04" y="78.74"/>
+</segment>
 </net>
 <net name="N$21" class="0">
@@
 <wire x1="190.5" y1="-43.18" x2="190.5" y2="-76.2" width="0.1524" layer="91"/>
 <junction x="190.5" y="-43.18"/>
-</segment>
-</net>
+<wire x1="190.5" y1="-43.18" x2="218.44" y2="-43.18" width="0.1524" layer="91"/>
+<wire x1="218.44" y1="-43.18" x2="218.44" y2="48.26" width="0.1524" layer="91"/>
+<wire x1="218.44" y1="48.26" x2="200.66" y2="48.26" width="0.1524" layer="91"/>
+<pinref part="SL3" gate="G$1" pin="4"/>
+<wire x1="200.66" y1="48.26" x2="200.66" y2="78.74" width="0.1524" layer="91"/>
+<junction x="200.66" y="78.74"/>
+</segment>
+</net>
+<net name="N$82" class="0">
+<segment>
+<pinref part="P-D" gate="-1" pin="S"/>
+<pinref part="SL2" gate="G$1" pin="2"/>
+<wire x1="55.88" y1="-5.08" x2="66.04" y2="-5.08" width="0.1524" layer="91"/>
+<junction x="55.88" y="-5.08"/>
+<junction x="66.04" y="-5.08"/>
+</segment>
+</net>
+<net name="N$83" class="0">
+<segment>
+<pinref part="U$1" gate="G$1" pin="OUT6"/>
+<wire x1="190.5" y1="-33.02" x2="213.36" y2="-33.02" width="0.1524" layer="91"/>
+<wire x1="213.36" y1="-33.02" x2="213.36" y2="43.18" width="0.1524" layer="91"/>
+<wire x1="213.36" y1="43.18" x2="195.58" y2="43.18" width="0.1524" layer="91"/>
+<pinref part="SL3" gate="G$1" pin="2"/>
+<wire x1="195.58" y1="43.18" x2="195.58" y2="78.74" width="0.1524" layer="91"/>
+<junction x="190.5" y="-33.02"/>
+<junction x="195.58" y="78.74"/>
+</segment>
+</net>
+<net name="N$84" class="0">
+<segment>
+<pinref part="U$1" gate="G$1" pin="OUT7"/>
+<wire x1="190.5" y1="-38.1" x2="215.9" y2="-38.1" width="0.1524" layer="91"/>
+<wire x1="215.9" y1="-38.1" x2="215.9" y2="45.72" width="0.1524" layer="91"/>
+<wire x1="215.9" y1="45.72" x2="198.12" y2="45.72" width="0.1524" layer="91"/>
+<wire x1="198.12" y1="45.72" x2="198.12" y2="78.74" width="0.1524" layer="91"/>
+<junction x="190.5" y="-38.1"/>
+<pinref part="SL3" gate="G$1" pin="3"/>
+<junction x="198.12" y="78.74"/>
+<wire x1="198.12" y1="78.74" x2="198.12" y2="81.28" width="0.1524" layer="91"/>
+</segment>
+</net>

Commit message: up, order pcb
Parts:
- R1, R10, R2, R3, R4, R5, R6, R7, R8, R9: value (none) -> 200
- R11, R12, R15, R16, R17, R18, R19, R20: value (none) -> 9.85k
- R13, R14: value (none) -> 811
- R21, R22: value (none) -> 3820
- R23, R24, R25, R26, R27, R28, R29, R30: value (none) -> 1.28k
- R31: value (none) -> 10k
- R32: value (none) -> 5k
- R33, R34, R35: value (none) -> 1k

Commit message: up
Parts:
- R19: value 9.85k -> 811
- R28: value 1.28k -> 3820
Changed lines of the file:
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@@
 <part name="R17" library="rcl" library_urn="urn:adsk.eagle:library:334" deviceset="R-US_" device="R0805" package3d_urn="urn:adsk.eagle:package:23553/2" value="9.85k"/>
 <part name="R18" library="rcl" library_urn="urn:adsk.eagle:library:334" deviceset="R-US_" device="R0805" package3d_urn="urn:adsk.eagle:package:23553/2" value="9.85k"/>
-<part name="R19" library="rcl" library_urn="urn:adsk.eagle:library:334" deviceset="R-US_" device="R0805" package3d_urn="urn:adsk.eagle:package:23553/2" value="9.85k"/>
+<part name="R19" library="rcl" library_urn="urn:adsk.eagle:library:334" deviceset="R-US_" device="R0805" package3d_urn="urn:adsk.eagle:package:23553/2" value="811"/>
 <part name="R20" library="rcl" library_urn="urn:adsk.eagle:library:334" deviceset="R-US_" device="R0805" package3d_urn="urn:adsk.eagle:package:23553/2" value="9.85k"/>
 <part name="R21" library="rcl" library_urn="urn:adsk.eagle:library:334" deviceset="R-US_" device="R0805" package3d_urn="urn:adsk.eagle:package:23553/2" value="3820"/>
@@
 <part name="R26" library="rcl" library_urn="urn:adsk.eagle:library:334" deviceset="R-US_" device="R0805" package3d_urn="urn:adsk.eagle:package:23553/2" value="1.28k"/>
 <part name="R27" library="rcl" library_urn="urn:adsk.eagle:library:334" deviceset="R-US_" device="R0805" package3d_urn="urn:adsk.eagle:package:23553/2" value="1.28k"/>
-<part name="R28" library="rcl" library_urn="urn:adsk.eagle:library:334" deviceset="R-US_" device="R0805" package3d_urn="urn:adsk.eagle:package:23553/2" value="1.28k"/>
+<part name="R28" library="rcl" library_urn="urn:adsk.eagle:library:334" deviceset="R-US_" device="R0805" package3d_urn="urn:adsk.eagle:package:23553/2" value="3820"/>
 <part name="R29" library="rcl" library_urn="urn:adsk.eagle:library:334" deviceset="R-US_" device="R0805" package3d_urn="urn:adsk.eagle:package:23553/2" value="1.28k"/>
 <part name="R30" library="rcl" library_urn="urn:adsk.eagle:library:334" deviceset="R-US_" device="R0805" package3d_urn="urn:adsk.eagle:package:23553/2" value="1.28k"/>

Commit message: up
Parts:
- added INT0, VREF4095: TPB1,27, testpad:TPB1,27
Connections:
- new net N$85: P-A-3.S, VREF4095.TP
- new net N$87: INT0.TP, P-B-10.S
- net N$43: now also P-D-3.S; no longer P-A-3.S
- net N$81: now also P-D-2.S
Changed lines of the file:
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@@
 <part name="SL3" library="con-amp-quick" library_urn="urn:adsk.eagle:library:125" deviceset="M04" device="" package3d_urn="urn:adsk.eagle:package:5958/1" value="MISC INP"/>
 <part name="VSS37" library="supply1" library_urn="urn:adsk.eagle:library:371" deviceset="VSS" device=""/>
+<part name="VREF4095" library="testpad" library_urn="urn:adsk.eagle:library:385" deviceset="TP" device="B1,27" package3d_urn="urn:adsk.eagle:package:27944/2"/>
+<part name="INT0" library="testpad" library_urn="urn:adsk.eagle:library:385" deviceset="TP" device="B1,27" package3d_urn="urn:adsk.eagle:package:27944/2"/>
 </parts>
 <sheets>
@@
 <instance part="VSS37" gate="G$1" x="185.42" y="78.74" smashed="yes" rot="R270">
 <attribute name="VALUE" x="180.34" y="81.28" size="1.778" layer="96"/>
+</instance>
+<instance part="VREF4095" gate="G$1" x="-5.08" y="96.52" smashed="yes">
+<attribute name="NAME" x="-6.35" y="97.79" size="1.778" layer="95"/>
+<attribute name="TP_SIGNAL_NAME" x="-3.81" y="95.25" size="1.778" layer="97"/>
+</instance>
+<instance part="INT0" gate="G$1" x="-15.24" y="33.02" smashed="yes">
+<attribute name="NAME" x="-16.51" y="34.29" size="1.778" layer="95"/>
+<attribute name="TP_SIGNAL_NAME" x="-13.97" y="31.75" size="1.778" layer="97"/>
 </instance>
 </instances>
@@
 <wire x1="198.12" y1="2.54" x2="190.5" y2="2.54" width="0.1524" layer="91"/>
 <junction x="190.5" y="2.54"/>
+<junction x="17.78" y="33.02"/>
 </segment>
 </net>
@@
 <net name="N$43" class="0">
 <segment>
-<pinref part="P-A" gate="-3" pin="S"/>
-<wire x1="17.78" y1="68.58" x2="-15.24" y2="68.58" width="0.1524" layer="91"/>
-<wire x1="-15.24" y1="68.58" x2="-15.24" y2="-22.86" width="0.1524" layer="91"/>
-<wire x1="-15.24" y1="-22.86" x2="78.74" y2="-22.86" width="0.1524" layer="91"/>
 <wire x1="78.74" y1="-22.86" x2="78.74" y2="-27.94" width="0.1524" layer="91"/>
 <wire x1="78.74" y1="-27.94" x2="121.92" y2="-27.94" width="0.1524" layer="91"/>
-<junction x="17.78" y="68.58"/>
 <wire x1="121.92" y1="-27.94" x2="121.92" y2="-63.5" width="0.1524" layer="91"/>
 <wire x1="121.92" y1="-63.5" x2="205.74" y2="-63.5" width="0.1524" layer="91"/>
@@
 <wire x1="205.74" y1="-27.94" x2="190.5" y2="-27.94" width="0.1524" layer="91"/>
 <junction x="190.5" y="-27.94"/>
+<pinref part="P-D" gate="-3" pin="S"/>
+<wire x1="55.88" y1="0" x2="25.4" y2="0" width="0.1524" layer="91"/>
+<wire x1="25.4" y1="0" x2="25.4" y2="-22.86" width="0.1524" layer="91"/>
+<wire x1="25.4" y1="-22.86" x2="78.74" y2="-22.86" width="0.1524" layer="91"/>
+<junction x="55.88" y="0"/>
 </segment>
 </net>
@@
 <net name="N$81" class="0">
 <segment>
-<wire x1="30.48" y1="-76.2" x2="190.5" y2="-76.2" width="0.1524" layer="91"/>
+<wire x1="30.48" y1="-76.2" x2="111.76" y2="-76.2" width="0.1524" layer="91"/>
 <pinref part="R35" gate="G$1" pin="2"/>
 <junction x="22.86" y="-58.42"/>
+<wire x1="111.76" y1="-76.2" x2="190.5" y2="-76.2" width="0.1524" layer="91"/>
 <wire x1="22.86" y1="-58.42" x2="30.48" y2="-58.42" width="0.1524" layer="91"/>
 <wire x1="30.48" y1="-58.42" x2="30.48" y2="-76.2" width="0.1524" layer="91"/>
@@
 <wire x1="200.66" y1="48.26" x2="200.66" y2="78.74" width="0.1524" layer="91"/>
 <junction x="200.66" y="78.74"/>
+<pinref part="P-D" gate="-2" pin="S"/>
+<wire x1="55.88" y1="-2.54" x2="27.94" y2="-2.54" width="0.1524" layer="91"/>
+<wire x1="27.94" y1="-2.54" x2="27.94" y2="-20.32" width="0.1524" layer="91"/>
+<wire x1="27.94" y1="-20.32" x2="111.76" y2="-20.32" width="0.1524" layer="91"/>
+<wire x1="111.76" y1="-20.32" x2="111.76" y2="-76.2" width="0.1524" layer="91"/>
+<junction x="55.88" y="-2.54"/>
+<junction x="111.76" y="-76.2"/>
 </segment>
 </net>
@@
 </segment>
 </net>
+<net name="N$85" class="0">
+<segment>
+<pinref part="VREF4095" gate="G$1" pin="TP"/>
+<wire x1="5.08" y1="68.58" x2="5.08" y2="93.98" width="0.1524" layer="91"/>
+<wire x1="5.08" y1="93.98" x2="-5.08" y2="93.98" width="0.1524" layer="91"/>
+<junction x="-5.08" y="93.98"/>
+<pinref part="P-A" gate="-3" pin="S"/>
+<wire x1="17.78" y1="68.58" x2="5.08" y2="68.58" width="0.1524" layer="91"/>
+<junction x="17.78" y="68.58"/>
+</segment>
+</net>
+<net name="N$87" class="0">
+<segment>
+<pinref part="INT0" gate="G$1" pin="TP"/>
+<wire x1="-15.24" y1="30.48" x2="-15.24" y2="25.4" width="0.1524" layer="91"/>
+<wire x1="-15.24" y1="25.4" x2="27.94" y2="25.4" width="0.1524" layer="91"/>
+<wire x1="27.94" y1="25.4" x2="27.94" y2="55.88" width="0.1524" layer="91"/>
+<pinref part="P-B" gate="-10" pin="S"/>
+<wire x1="27.94" y1="55.88" x2="17.78" y2="55.88" width="0.1524" layer="91"/>
+<junction x="-15.24" y="30.48"/>
+<junction x="17.78" y="55.88"/>
+</segment>
+</net>

Commit message: up
Connections:
- removed net N$83: SL3.2, U$1.OUT6
- new net N$86: P-D-2.S, SL3.2, U$1.OUT6
- net N$35: now also IC2.8
- net N$36: now also IC2.7, U$1.EN_L
- net N$81: no longer P-D-2.S
- net VSS: now also IC2.1; no longer U$1.EN_L
Changed lines of the file:
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@@
 <part name="C5" library="rcl" library_urn="urn:adsk.eagle:library:334" deviceset="C-US" device="C0805" package3d_urn="urn:adsk.eagle:package:23617/2" value="0.1"/>
 <part name="VSS19" library="supply1" library_urn="urn:adsk.eagle:library:371" deviceset="VSS" device=""/>
-<part name="VSS20" library="supply1" library_urn="urn:adsk.eagle:library:371" deviceset="VSS" device=""/>
 <part name="OUTP" library="con-molex" library_urn="urn:adsk.eagle:library:165" deviceset="22-23-2101" device="" package3d_urn="urn:adsk.eagle:package:8078641/1"/>
 <part name="VSS4" library="supply1" library_urn="urn:adsk.eagle:library:371" deviceset="VSS" device=""/>
@@
 <part name="VREF4095" library="testpad" library_urn="urn:adsk.eagle:library:385" deviceset="TP" device="B1,27" package3d_urn="urn:adsk.eagle:package:27944/2"/>
 <part name="INT0" library="testpad" library_urn="urn:adsk.eagle:library:385" deviceset="TP" device="B1,27" package3d_urn="urn:adsk.eagle:package:27944/2"/>
+<part name="VSS20" library="supply1" library_urn="urn:adsk.eagle:library:371" deviceset="VSS" device=""/>
 </parts>
 <sheets>
@@
 <attribute name="VALUE" x="172.72" y="12.7" size="1.778" layer="96" rot="R90"/>
 </instance>
-<instance part="VSS20" gate="G$1" x="193.04" y="7.62" smashed="yes" rot="R90">
-<attribute name="VALUE" x="198.12" y="5.08" size="1.778" layer="96" rot="R180"/>
-</instance>
 <instance part="OUTP" gate="-1" x="93.98" y="-45.72" smashed="yes">
 <attribute name="NAME" x="96.52" y="-46.482" size="1.524" layer="95"/>
@@
 <attribute name="NAME" x="-16.51" y="34.29" size="1.778" layer="95"/>
 <attribute name="TP_SIGNAL_NAME" x="-13.97" y="31.75" size="1.778" layer="97"/>
+</instance>
+<instance part="VSS20" gate="G$1" x="-17.78" y="-35.56" smashed="yes" rot="R180">
+<attribute name="VALUE" x="-15.24" y="-30.48" size="1.778" layer="96" rot="R270"/>
 </instance>
 </instances>
@@
 </segment>
 </net>
-<net name="VSS" class="1">
+<net name="VSS" class="0">
 <segment>
 <pinref part="R29" gate="G$1" pin="2"/>
@@
 <pinref part="VSS19" gate="G$1" pin="VSS"/>
 <junction x="175.26" y="20.32"/>
-</segment>
-<segment>
-<pinref part="U$1" gate="G$1" pin="EN_L"/>
-<pinref part="VSS20" gate="G$1" pin="VSS"/>
-<junction x="190.5" y="7.62"/>
 </segment>
 <segment>
@@
 <junction x="193.04" y="78.74"/>
 </segment>
+<segment>
+<pinref part="IC2" gate="G$1" pin="1"/>
+<pinref part="VSS20" gate="G$1" pin="VSS"/>
+</segment>
 </net>
 <net name="N$21" class="0">
@@
 <junction x="30.48" y="-38.1"/>
 <junction x="17.78" y="45.72"/>
+<pinref part="IC2" gate="G$1" pin="8"/>
+<wire x1="20.32" y1="-38.1" x2="-2.54" y2="-38.1" width="0.1524" layer="91"/>
+<junction x="-2.54" y="-38.1"/>
+<junction x="20.32" y="-38.1"/>
 </segment>
 </net>
@@
 <pinref part="P-B" gate="-7" pin="S"/>
 <wire x1="17.78" y1="48.26" x2="22.86" y2="48.26" width="0.1524" layer="91"/>
-<wire x1="22.86" y1="48.26" x2="22.86" y2="-40.64" width="0.1524" layer="91"/>
+<wire x1="22.86" y1="48.26" x2="22.86" y2="22.86" width="0.1524" layer="91"/>
 <pinref part="IC1" gate="G$1" pin="I6"/>
+<wire x1="22.86" y1="22.86" x2="22.86" y2="-40.64" width="0.1524" layer="91"/>
 <wire x1="22.86" y1="-40.64" x2="30.48" y2="-40.64" width="0.1524" layer="91"/>
 <junction x="30.48" y="-40.64"/>
 <junction x="17.78" y="48.26"/>
+<pinref part="IC2" gate="G$1" pin="7"/>
+<wire x1="22.86" y1="-40.64" x2="-2.54" y2="-40.64" width="0.1524" layer="91"/>
+<junction x="-2.54" y="-40.64"/>
+<junction x="22.86" y="-40.64"/>
+<pinref part="U$1" gate="G$1" pin="EN_L"/>
+<wire x1="190.5" y1="7.62" x2="190.5" y2="30.48" width="0.1524" layer="91"/>
+<wire x1="190.5" y1="30.48" x2="160.02" y2="30.48" width="0.1524" layer="91"/>
+<wire x1="160.02" y1="30.48" x2="160.02" y2="20.32" width="0.1524" layer="91"/>
+<wire x1="160.02" y1="20.32" x2="111.76" y2="20.32" width="0.1524" layer="91"/>
+<wire x1="111.76" y1="20.32" x2="111.76" y2="25.4" width="0.1524" layer="91"/>
+<wire x1="111.76" y1="25.4" x2="30.48" y2="25.4" width="0.1524" layer="91"/>
+<wire x1="30.48" y1="25.4" x2="30.48" y2="22.86" width="0.1524" layer="91"/>
+<wire x1="30.48" y1="22.86" x2="22.86" y2="22.86" width="0.1524" layer="91"/>
+<junction x="22.86" y="22.86"/>
+<junction x="190.5" y="7.62"/>
 </segment>
 </net>
@@
 <net name="N$81" class="0">
 <segment>
-<wire x1="30.48" y1="-76.2" x2="111.76" y2="-76.2" width="0.1524" layer="91"/>
+<wire x1="30.48" y1="-76.2" x2="190.5" y2="-76.2" width="0.1524" layer="91"/>
 <pinref part="R35" gate="G$1" pin="2"/>
 <junction x="22.86" y="-58.42"/>
-<wire x1="111.76" y1="-76.2" x2="190.5" y2="-76.2" width="0.1524" layer="91"/>
 <wire x1="22.86" y1="-58.42" x2="30.48" y2="-58.42" width="0.1524" layer="91"/>
 <wire x1="30.48" y1="-58.42" x2="30.48" y2="-76.2" width="0.1524" layer="91"/>
@@
 <wire x1="200.66" y1="48.26" x2="200.66" y2="78.74" width="0.1524" layer="91"/>
 <junction x="200.66" y="78.74"/>
-<pinref part="P-D" gate="-2" pin="S"/>
-<wire x1="55.88" y1="-2.54" x2="27.94" y2="-2.54" width="0.1524" layer="91"/>
-<wire x1="27.94" y1="-2.54" x2="27.94" y2="-20.32" width="0.1524" layer="91"/>
-<wire x1="27.94" y1="-20.32" x2="111.76" y2="-20.32" width="0.1524" layer="91"/>
-<wire x1="111.76" y1="-20.32" x2="111.76" y2="-76.2" width="0.1524" layer="91"/>
-<junction x="55.88" y="-2.54"/>
-<junction x="111.76" y="-76.2"/>
 </segment>
 </net>
@@
 <junction x="55.88" y="-5.08"/>
 <junction x="66.04" y="-5.08"/>
-</segment>
-</net>
-<net name="N$83" class="0">
-<segment>
-<pinref part="U$1" gate="G$1" pin="OUT6"/>
-<wire x1="190.5" y1="-33.02" x2="213.36" y2="-33.02" width="0.1524" layer="91"/>
-<wire x1="213.36" y1="-33.02" x2="213.36" y2="43.18" width="0.1524" layer="91"/>
-<wire x1="213.36" y1="43.18" x2="195.58" y2="43.18" width="0.1524" layer="91"/>
-<pinref part="SL3" gate="G$1" pin="2"/>
-<wire x1="195.58" y1="43.18" x2="195.58" y2="78.74" width="0.1524" layer="91"/>
-<junction x="190.5" y="-33.02"/>
-<junction x="195.58" y="78.74"/>
 </segment>
 </net>
@@
 </segment>
 </net>
+<net name="N$86" class="0">
+<segment>
+<pinref part="P-D" gate="-2" pin="S"/>
+<junction x="55.88" y="-2.54"/>
+<wire x1="55.88" y1="-2.54" x2="27.94" y2="-2.54" width="0.1524" layer="91"/>
+<wire x1="27.94" y1="-2.54" x2="27.94" y2="-20.32" width="0.1524" layer="91"/>
+<wire x1="27.94" y1="-20.32" x2="111.76" y2="-20.32" width="0.1524" layer="91"/>
+<wire x1="111.76" y1="-20.32" x2="111.76" y2="-81.28" width="0.1524" layer="91"/>
+<pinref part="U$1" gate="G$1" pin="OUT6"/>
+<wire x1="190.5" y1="-33.02" x2="198.12" y2="-33.02" width="0.1524" layer="91"/>
+<wire x1="198.12" y1="-33.02" x2="213.36" y2="-33.02" width="0.1524" layer="91"/>
+<wire x1="213.36" y1="-33.02" x2="213.36" y2="43.18" width="0.1524" layer="91"/>
+<wire x1="213.36" y1="43.18" x2="195.58" y2="43.18" width="0.1524" layer="91"/>
+<pinref part="SL3" gate="G$1" pin="2"/>
+<wire x1="195.58" y1="43.18" x2="195.58" y2="78.74" width="0.1524" layer="91"/>
+<junction x="190.5" y="-33.02"/>
+<junction x="195.58" y="78.74"/>
+<wire x1="111.76" y1="-81.28" x2="198.12" y2="-81.28" width="0.1524" layer="91"/>
+<wire x1="198.12" y1="-81.28" x2="198.12" y2="-33.02" width="0.1524" layer="91"/>
+<junction x="198.12" y="-33.02"/>
+</segment>
+</net>
