File: host_board/hall_sensor100a.sch (EAGLE design)
At the start: 5 parts, among them IC1 REF02HCSA, IC2 CSLT6B100, X1 22-23-2051

Commit message: up
Parts:
- added PAD1, PAD2: (no value), wirepad:2,15/1,0
- added U$1: L01ZXXXS05A1, l01z:L01ZXXXS05A1
Connections:
- net GND: now also PAD1.P, PAD2.P, U$1.GND
- net N$1: now also U$1.VCC
- net N$2: now also U$1.VOUT
Changed lines of the file:
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@@
 <part name="SUPPLY7" library="supply2" library_urn="urn:adsk.eagle:library:372" deviceset="GND" device=""/>
 <part name="SUPPLY8" library="supply2" library_urn="urn:adsk.eagle:library:372" deviceset="GND" device=""/>
+<part name="U$1" library="l01z" deviceset="L01ZXXXS05" device="A1" package3d_urn="urn:adsk.eagle:package:15042033/1"/>
+<part name="SUPPLY9" library="supply2" library_urn="urn:adsk.eagle:library:372" deviceset="GND" device=""/>
+<part name="PAD1" library="wirepad" library_urn="urn:adsk.eagle:library:412" deviceset="2,15/1,0" device="" package3d_urn="urn:adsk.eagle:package:30831/1"/>
+<part name="PAD2" library="wirepad" library_urn="urn:adsk.eagle:library:412" deviceset="2,15/1,0" device="" package3d_urn="urn:adsk.eagle:package:30831/1"/>
+<part name="SUPPLY10" library="supply2" library_urn="urn:adsk.eagle:library:372" deviceset="GND" device=""/>
+<part name="SUPPLY11" library="supply2" library_urn="urn:adsk.eagle:library:372" deviceset="GND" device=""/>
 </parts>
 <sheets>
@@
 <attribute name="VALUE" x="5.715" y="65.405" size="1.778" layer="96"/>
 </instance>
+<instance part="U$1" gate="G$1" x="68.58" y="27.94" smashed="yes">
+<attribute name="NAME" x="27.94" y="43.18" size="1.27" layer="95"/>
+<attribute name="VALUE" x="27.94" y="22.86" size="1.27" layer="96"/>
+</instance>
+<instance part="SUPPLY9" gate="GND" x="2.54" y="33.02" smashed="yes" rot="R270">
+<attribute name="VALUE" x="-0.635" y="34.925" size="1.778" layer="96" rot="R270"/>
+</instance>
+<instance part="PAD1" gate="1" x="71.12" y="22.86" smashed="yes">
+<attribute name="NAME" x="69.977" y="24.7142" size="1.778" layer="95"/>
+<attribute name="VALUE" x="69.977" y="19.558" size="1.778" layer="96"/>
+</instance>
+<instance part="PAD2" gate="1" x="86.36" y="22.86" smashed="yes">
+<attribute name="NAME" x="85.217" y="24.7142" size="1.778" layer="95"/>
+<attribute name="VALUE" x="85.217" y="19.558" size="1.778" layer="96"/>
+</instance>
+<instance part="SUPPLY10" gate="GND" x="73.66" y="20.32" smashed="yes">
+<attribute name="VALUE" x="71.755" y="17.145" size="1.778" layer="96"/>
+</instance>
+<instance part="SUPPLY11" gate="GND" x="88.9" y="20.32" smashed="yes">
+<attribute name="VALUE" x="86.995" y="17.145" size="1.778" layer="96"/>
+</instance>
 </instances>
 <busses>
@@
 <pinref part="SUPPLY8" gate="GND" pin="GND"/>
 <junction x="7.62" y="71.12"/>
+</segment>
+<segment>
+<pinref part="U$1" gate="G$1" pin="GND"/>
+<pinref part="SUPPLY9" gate="GND" pin="GND"/>
+<junction x="5.08" y="33.02"/>
+</segment>
+<segment>
+<pinref part="PAD1" gate="1" pin="P"/>
+<pinref part="SUPPLY10" gate="GND" pin="GND"/>
+</segment>
+<segment>
+<pinref part="PAD2" gate="1" pin="P"/>
+<pinref part="SUPPLY11" gate="GND" pin="GND"/>
 </segment>
 </net>
@@
 <junction x="101.6" y="58.42"/>
 <junction x="35.56" y="55.88"/>
+<pinref part="U$1" gate="G$1" pin="VOUT"/>
+<wire x1="5.08" y1="40.64" x2="5.08" y2="48.26" width="0.1524" layer="91"/>
+<wire x1="5.08" y1="48.26" x2="35.56" y2="48.26" width="0.1524" layer="91"/>
+<wire x1="35.56" y1="48.26" x2="35.56" y2="55.88" width="0.1524" layer="91"/>
+<junction x="5.08" y="40.64"/>
 </segment>
 </net>
@@
 <pinref part="C1" gate="G$1" pin="1"/>
 <junction x="7.62" y="78.74"/>
-</segment>
-</net>
+<wire x1="0" y1="55.88" x2="-5.08" y2="55.88" width="0.1524" layer="91"/>
+<wire x1="-5.08" y1="55.88" x2="-5.08" y2="25.4" width="0.1524" layer="91"/>
+<pinref part="U$1" gate="G$1" pin="VCC"/>
+<wire x1="-5.08" y1="25.4" x2="5.08" y2="25.4" width="0.1524" layer="91"/>
+<junction x="5.08" y="25.4"/>
+</segment>
+</net>

Commit message: up
Parts:
- added C3: 22uf, rcl:C-USC0805
- added C4: 2.2uf, rcl:C-USC0805
- added IC3: MAX5322EAI+, MAX5322EAI+:MAX5322EAI+
Connections:
- net +12V: now also C4.1
- net GND: now also C3.2, C4.2
- net N$1: now also C3.1
Changed lines of the file:
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@@
 <?xml version="1.0" encoding="utf-8"?>
 <!DOCTYPE eagle SYSTEM "eagle.dtd">
-<eagle version="9.5.1">
+<eagle version="9.5.2">
 <drawing>
 <settings>
@@
 <part name="SUPPLY10" library="supply2" library_urn="urn:adsk.eagle:library:372" deviceset="GND" device=""/>
 <part name="SUPPLY11" library="supply2" library_urn="urn:adsk.eagle:library:372" deviceset="GND" device=""/>
+<part name="C3" library="rcl" library_urn="urn:adsk.eagle:library:334" deviceset="C-US" device="C0805" package3d_urn="urn:adsk.eagle:package:23617/2" value="22uf"/>
+<part name="SUPPLY12" library="supply2" library_urn="urn:adsk.eagle:library:372" deviceset="GND" device=""/>
+<part name="C4" library="rcl" library_urn="urn:adsk.eagle:library:334" deviceset="C-US" device="C0805" package3d_urn="urn:adsk.eagle:package:23617/2" value="2.2uf"/>
+<part name="SUPPLY13" library="supply2" library_urn="urn:adsk.eagle:library:372" deviceset="GND" device=""/>
+<part name="IC3" library="MAX5322EAI+" deviceset="MAX5322EAI+" device=""/>
 </parts>
 <sheets>
@@
 <attribute name="VALUE" x="86.995" y="17.145" size="1.778" layer="96"/>
 </instance>
+<instance part="C3" gate="G$1" x="17.78" y="76.2" smashed="yes">
+<attribute name="NAME" x="18.796" y="76.835" size="1.778" layer="95"/>
+<attribute name="VALUE" x="18.796" y="72.009" size="1.778" layer="96"/>
+</instance>
+<instance part="SUPPLY12" gate="GND" x="17.78" y="68.58" smashed="yes">
+<attribute name="VALUE" x="15.875" y="65.405" size="1.778" layer="96"/>
+</instance>
+<instance part="C4" gate="G$1" x="81.28" y="53.34" smashed="yes">
+<attribute name="NAME" x="82.296" y="53.975" size="1.778" layer="95"/>
+<attribute name="VALUE" x="82.296" y="49.149" size="1.778" layer="96"/>
+</instance>
+<instance part="SUPPLY13" gate="GND" x="81.28" y="45.72" smashed="yes">
+<attribute name="VALUE" x="79.375" y="42.545" size="1.778" layer="96"/>
+</instance>
+<instance part="IC3" gate="G$1" x="27.94" y="116.84" smashed="yes">
+<attribute name="NAME" x="64.77" y="124.46" size="1.778" layer="95" align="center-left"/>
+<attribute name="VALUE" x="64.77" y="121.92" size="1.778" layer="96" align="center-left"/>
+</instance>
 </instances>
 <busses>
@@
 <pinref part="SUPPLY11" gate="GND" pin="GND"/>
 </segment>
+<segment>
+<pinref part="C3" gate="G$1" pin="2"/>
+<pinref part="SUPPLY12" gate="GND" pin="GND"/>
+<junction x="17.78" y="71.12"/>
+</segment>
+<segment>
+<pinref part="C4" gate="G$1" pin="2"/>
+<pinref part="SUPPLY13" gate="GND" pin="GND"/>
+<junction x="81.28" y="48.26"/>
+</segment>
 </net>
 <net name="+12V" class="1">
@@
 <pinref part="IC1" gate="G$1" pin="V-IN"/>
 <pinref part="SUPPLY5" gate="+12V" pin="+12V"/>
-<wire x1="86.36" y1="55.88" x2="78.74" y2="55.88" width="0.1524" layer="91"/>
+<wire x1="86.36" y1="55.88" x2="81.28" y2="55.88" width="0.1524" layer="91"/>
 <pinref part="C2" gate="G$1" pin="1"/>
 <junction x="86.36" y="55.88"/>
 <junction x="78.74" y="55.88"/>
+<pinref part="C4" gate="G$1" pin="1"/>
+<wire x1="81.28" y1="55.88" x2="78.74" y2="55.88" width="0.1524" layer="91"/>
+<junction x="81.28" y="55.88"/>
 </segment>
 </net>
@@
 <wire x1="0" y1="55.88" x2="0" y2="78.74" width="0.1524" layer="91"/>
 <wire x1="0" y1="78.74" x2="7.62" y2="78.74" width="0.1524" layer="91"/>
-<wire x1="7.62" y1="78.74" x2="81.28" y2="78.74" width="0.1524" layer="91"/>
+<wire x1="7.62" y1="78.74" x2="17.78" y2="78.74" width="0.1524" layer="91"/>
+<wire x1="17.78" y1="78.74" x2="81.28" y2="78.74" width="0.1524" layer="91"/>
 <wire x1="81.28" y1="78.74" x2="81.28" y2="63.5" width="0.1524" layer="91"/>
 <pinref part="IC1" gate="G$1" pin="V-OUT"/>
@@
 <wire x1="-5.08" y1="25.4" x2="5.08" y2="25.4" width="0.1524" layer="91"/>
 <junction x="5.08" y="25.4"/>
+<pinref part="C3" gate="G$1" pin="1"/>
+<junction x="17.78" y="78.74"/>
 </segment>
 </net>

Commit message: up
Parts:
- added C5, C7: 0.1, rcl:C-USC0805
- added C6: 22uf, rcl:C-USC0805
- added DAC_OUT, SPI_IN: 22-23-2101, con-molex:22-23-2101
Connections:
- new net N$10: C5.1, C6.1, IC3.!CLR, IC3.!SHDN, IC3.UNI/!BIPA, IC3.UNI/!BIPB, IC3.VCC, SPI_IN-7.S
- new net N$11: C5.2, C6.2, IC3.DGND, SPI_IN-8.S
- new net N$12: IC3.!LDAC, SPI_IN-4.S
- new net N$4: DAC_OUT-2.S, IC3.OUTA
- new net N$5: DAC_OUT-3.S, IC3.OUTB
- new net N$6: IC3.DIN, SPI_IN-2.S
- new net N$7: IC3.DOUT, SPI_IN-1.S
- new net N$8: IC3.SCLK, SPI_IN-3.S
- new net N$9: IC3.!CS, SPI_IN-9.S
- net +12V: now also C7.1, DAC_OUT-10.S, IC3.VDD
- net GND: now also C7.2, DAC_OUT-1.S, IC3.AGND, IC3.SGNDA, IC3.SGNDB, IC3.VSS
- net N$1: now also DAC_OUT-7.S, IC3.REFA, IC3.REFB

Commit message: up
Parts:
- added R1, R2, R3: 50, rcl:R-US_M0805
- added R4: 4.7k, rcl:R-US_M0805
Connections:
- new net N$13: IC3.SCLK, R2.2
- new net N$14: IC3.!CS, R3.2
- new net N$3: IC3.DIN, R1.2
- net N$10: now also R4.2
- net N$12: now also R4.1
- net N$6: now also R1.1; no longer IC3.DIN
- net N$8: now also R2.1; no longer IC3.SCLK
- net N$9: now also R3.1; no longer IC3.!CS
Changed lines of the file:
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@@
 <part name="C7" library="rcl" library_urn="urn:adsk.eagle:library:334" deviceset="C-US" device="C0805" package3d_urn="urn:adsk.eagle:package:23617/2" value="0.1"/>
 <part name="SUPPLY17" library="supply2" library_urn="urn:adsk.eagle:library:372" deviceset="GND" device=""/>
+<part name="R1" library="rcl" library_urn="urn:adsk.eagle:library:334" deviceset="R-US_" device="M0805" package3d_urn="urn:adsk.eagle:package:23556/2" value="50"/>
+<part name="R2" library="rcl" library_urn="urn:adsk.eagle:library:334" deviceset="R-US_" device="M0805" package3d_urn="urn:adsk.eagle:package:23556/2" value="50"/>
+<part name="R3" library="rcl" library_urn="urn:adsk.eagle:library:334" deviceset="R-US_" device="M0805" package3d_urn="urn:adsk.eagle:package:23556/2" value="50"/>
+<part name="R4" library="rcl" library_urn="urn:adsk.eagle:library:334" deviceset="R-US_" device="M0805" package3d_urn="urn:adsk.eagle:package:23556/2" value="4.7k"/>
 </parts>
 <sheets>
@@
 <instance part="SUPPLY17" gate="GND" x="106.68" y="81.28" smashed="yes">
 <attribute name="VALUE" x="104.775" y="78.105" size="1.778" layer="96"/>
+</instance>
+<instance part="R1" gate="G$1" x="22.86" y="91.44" smashed="yes">
+<attribute name="NAME" x="19.05" y="92.9386" size="1.778" layer="95"/>
+<attribute name="VALUE" x="19.05" y="88.138" size="1.778" layer="96"/>
+</instance>
+<instance part="R2" gate="G$1" x="22.86" y="93.98" smashed="yes">
+<attribute name="NAME" x="19.05" y="95.4786" size="1.778" layer="95"/>
+<attribute name="VALUE" x="19.05" y="90.678" size="1.778" layer="96"/>
+</instance>
+<instance part="R3" gate="G$1" x="22.86" y="88.9" smashed="yes">
+<attribute name="NAME" x="19.05" y="90.3986" size="1.778" layer="95"/>
+<attribute name="VALUE" x="19.05" y="85.598" size="1.778" layer="96"/>
+</instance>
+<instance part="R4" gate="G$1" x="5.08" y="104.14" smashed="yes" rot="R180">
+<attribute name="NAME" x="8.89" y="102.6414" size="1.778" layer="95" rot="R180"/>
+<attribute name="VALUE" x="8.89" y="107.442" size="1.778" layer="96" rot="R180"/>
 </instance>
 </instances>
@@
 <wire x1="-2.54" y1="93.98" x2="12.7" y2="93.98" width="0.1524" layer="91"/>
 <wire x1="12.7" y1="93.98" x2="12.7" y2="91.44" width="0.1524" layer="91"/>
-<pinref part="IC3" gate="G$1" pin="DIN"/>
-<wire x1="12.7" y1="91.44" x2="27.94" y2="91.44" width="0.1524" layer="91"/>
 <junction x="-2.54" y="93.98"/>
-<junction x="27.94" y="91.44"/>
+<pinref part="R1" gate="G$1" pin="1"/>
+<wire x1="17.78" y1="91.44" x2="12.7" y2="91.44" width="0.1524" layer="91"/>
+<junction x="17.78" y="91.44"/>
 </segment>
 </net>
@@
 <net name="N$8" class="0">
 <segment>
-<pinref part="IC3" gate="G$1" pin="SCLK"/>
-<wire x1="27.94" y1="93.98" x2="17.78" y2="93.98" width="0.1524" layer="91"/>
 <wire x1="17.78" y1="93.98" x2="17.78" y2="99.06" width="0.1524" layer="91"/>
 <wire x1="17.78" y1="99.06" x2="12.7" y2="99.06" width="0.1524" layer="91"/>
@@
 <wire x1="12.7" y1="96.52" x2="-2.54" y2="96.52" width="0.1524" layer="91"/>
 <junction x="-2.54" y="96.52"/>
-<junction x="27.94" y="93.98"/>
+<pinref part="R2" gate="G$1" pin="1"/>
+<junction x="17.78" y="93.98"/>
 </segment>
 </net>
 <net name="N$9" class="0">
 <segment>
+<wire x1="17.78" y1="86.36" x2="17.78" y2="88.9" width="0.1524" layer="91"/>
+<pinref part="R3" gate="G$1" pin="1"/>
+<junction x="17.78" y="88.9"/>
 <pinref part="SPI_IN" gate="-9" pin="S"/>
-<wire x1="-2.54" y1="111.76" x2="7.62" y2="111.76" width="0.1524" layer="91"/>
-<wire x1="7.62" y1="111.76" x2="7.62" y2="86.36" width="0.1524" layer="91"/>
-<wire x1="7.62" y1="86.36" x2="17.78" y2="86.36" width="0.1524" layer="91"/>
-<wire x1="17.78" y1="86.36" x2="17.78" y2="88.9" width="0.1524" layer="91"/>
-<pinref part="IC3" gate="G$1" pin="!CS"/>
-<wire x1="17.78" y1="88.9" x2="27.94" y2="88.9" width="0.1524" layer="91"/>
+<wire x1="-2.54" y1="111.76" x2="-20.32" y2="111.76" width="0.1524" layer="91"/>
+<wire x1="-20.32" y1="111.76" x2="-20.32" y2="86.36" width="0.1524" layer="91"/>
+<wire x1="-20.32" y1="86.36" x2="17.78" y2="86.36" width="0.1524" layer="91"/>
 <junction x="-2.54" y="111.76"/>
-<junction x="27.94" y="88.9"/>
 </segment>
 </net>
@@
 <segment>
 <pinref part="SPI_IN" gate="-7" pin="S"/>
-<wire x1="-2.54" y1="106.68" x2="12.7" y2="106.68" width="0.1524" layer="91"/>
+<wire x1="-2.54" y1="106.68" x2="0" y2="106.68" width="0.1524" layer="91"/>
+<wire x1="0" y1="106.68" x2="12.7" y2="106.68" width="0.1524" layer="91"/>
 <wire x1="12.7" y1="106.68" x2="20.32" y2="106.68" width="0.1524" layer="91"/>
 <wire x1="20.32" y1="106.68" x2="20.32" y2="99.06" width="0.1524" layer="91"/>
@@
 <pinref part="C6" gate="G$1" pin="1"/>
 <junction x="20.32" y="111.76"/>
+<pinref part="R4" gate="G$1" pin="2"/>
+<wire x1="0" y1="104.14" x2="0" y2="106.68" width="0.1524" layer="91"/>
+<junction x="0" y="104.14"/>
+<junction x="0" y="106.68"/>
 </segment>
 </net>
@@
 <junction x="-2.54" y="99.06"/>
 <junction x="27.94" y="106.68"/>
-</segment>
-</net>
+<pinref part="R4" gate="G$1" pin="1"/>
+<junction x="10.16" y="104.14"/>
+</segment>
+</net>
+<net name="N$3" class="0">
+<segment>
+<pinref part="IC3" gate="G$1" pin="DIN"/>
+<pinref part="R1" gate="G$1" pin="2"/>
+<junction x="27.94" y="91.44"/>
+</segment>
+</net>
+<net name="N$13" class="0">
+<segment>
+<pinref part="IC3" gate="G$1" pin="SCLK"/>
+<pinref part="R2" gate="G$1" pin="2"/>
+<junction x="27.94" y="93.98"/>
+</segment>
+</net>
+<net name="N$14" class="0">
+<segment>
+<pinref part="IC3" gate="G$1" pin="!CS"/>
+<pinref part="R3" gate="G$1" pin="2"/>
+<junction x="27.94" y="88.9"/>
+</segment>
+</net>

Commit message: up
Parts:
- added D1: btb1, diode:SCHOTTKY-DIODEDO35-7
- added D2: btb2, diode:SCHOTTKY-DIODEDO35-7
- added LED1: 12v_led, led:LEDCHIPLED_1206
- added LED2: 5v_led, led:LEDCHIPLED_1206
- added R5, R6: 4.7k, rcl:R-US_M0805
Connections:
- new net DGND: C5.2, C6.2, D1.C, D2.A, IC3.DGND, LED2.C, SPI_IN-8.S
- new net N$15: DAC_OUT-6.S, IC1.TEMP
- new net N$16: LED2.A, R6.2
- net +12V: now also R5.1
- net GND: now also D1.A, D2.C, LED1.C
- net N$10: now also R6.1
- net N$11: now also LED1.A, R5.2; no longer C5.2, C6.2, IC3.DGND, SPI_IN-8.S
Changed lines of the file:
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@@
 <layer number="97" name="Info" color="7" fill="1" visible="yes" active="yes"/>
 <layer number="98" name="Guide" color="6" fill="1" visible="yes" active="yes"/>
+<layer number="99" name="SpiceOrder" color="5" fill="1" visible="yes" active="yes"/>
 </layers>
 <schematic xreflabel="%F%N/%S.%C%R" xrefpart="/%S.%C%R">
@@
 <part name="R3" library="rcl" library_urn="urn:adsk.eagle:library:334" deviceset="R-US_" device="M0805" package3d_urn="urn:adsk.eagle:package:23556/2" value="50"/>
 <part name="R4" library="rcl" library_urn="urn:adsk.eagle:library:334" deviceset="R-US_" device="M0805" package3d_urn="urn:adsk.eagle:package:23556/2" value="4.7k"/>
+<part name="SUPPLY18" library="supply2" library_urn="urn:adsk.eagle:library:372" deviceset="DGND" device=""/>
+<part name="D1" library="diode" library_urn="urn:adsk.eagle:library:210" deviceset="SCHOTTKY-DIODE" device="DO35-7" package3d_urn="urn:adsk.eagle:package:43339/2" value="btb1"/>
+<part name="D2" library="diode" library_urn="urn:adsk.eagle:library:210" deviceset="SCHOTTKY-DIODE" device="DO35-7" package3d_urn="urn:adsk.eagle:package:43339/2" value="btb2"/>
+<part name="SUPPLY19" library="supply2" library_urn="urn:adsk.eagle:library:372" deviceset="DGND" device=""/>
+<part name="SUPPLY20" library="supply2" library_urn="urn:adsk.eagle:library:372" deviceset="GND" device=""/>
+<part name="LED1" library="led" library_urn="urn:adsk.eagle:library:259" deviceset="LED" device="CHIPLED_1206" package3d_urn="urn:adsk.eagle:package:15823/2" value="12v_led"/>
+<part name="R5" library="rcl" library_urn="urn:adsk.eagle:library:334" deviceset="R-US_" device="M0805" package3d_urn="urn:adsk.eagle:package:23556/2" value="4.7k"/>
+<part name="SUPPLY21" library="supply2" library_urn="urn:adsk.eagle:library:372" deviceset="GND" device=""/>
+<part name="SUPPLY22" library="supply2" library_urn="urn:adsk.eagle:library:372" deviceset="+12V" device=""/>
+<part name="R6" library="rcl" library_urn="urn:adsk.eagle:library:334" deviceset="R-US_" device="M0805" package3d_urn="urn:adsk.eagle:package:23556/2" value="4.7k"/>
+<part name="LED2" library="led" library_urn="urn:adsk.eagle:library:259" deviceset="LED" device="CHIPLED_1206" package3d_urn="urn:adsk.eagle:package:15823/2" value="5v_led"/>
+<part name="SUPPLY23" library="supply2" library_urn="urn:adsk.eagle:library:372" deviceset="DGND" device=""/>
 </parts>
 <sheets>
@@
 <attribute name="NAME" x="8.89" y="102.6414" size="1.778" layer="95" rot="R180"/>
 <attribute name="VALUE" x="8.89" y="107.442" size="1.778" layer="96" rot="R180"/>
+</instance>
+<instance part="SUPPLY18" gate="G$1" x="5.08" y="121.92" smashed="yes" rot="R180">
+<attribute name="VALUE" x="7.747" y="125.095" size="1.778" layer="96" rot="R180"/>
+</instance>
+<instance part="D1" gate="G$1" x="-17.78" y="76.2" smashed="yes">
+<attribute name="NAME" x="-20.066" y="78.105" size="1.778" layer="95"/>
+<attribute name="VALUE" x="-20.066" y="72.771" size="1.778" layer="96"/>
+</instance>
+<instance part="D2" gate="G$1" x="-17.78" y="66.04" smashed="yes" rot="R180">
+<attribute name="NAME" x="-15.494" y="64.135" size="1.778" layer="95" rot="R180"/>
+<attribute name="VALUE" x="-15.494" y="69.469" size="1.778" layer="96" rot="R180"/>
+</instance>
+<instance part="SUPPLY19" gate="G$1" x="-12.7" y="71.12" smashed="yes" rot="R90">
+<attribute name="VALUE" x="-9.525" y="68.453" size="1.778" layer="96" rot="R90"/>
+</instance>
+<instance part="SUPPLY20" gate="GND" x="-22.86" y="71.12" smashed="yes" rot="R270">
+<attribute name="VALUE" x="-26.035" y="73.025" size="1.778" layer="96" rot="R270"/>
+</instance>
+<instance part="LED1" gate="G$1" x="-20.32" y="43.18" smashed="yes">
+<attribute name="NAME" x="-16.764" y="38.608" size="1.778" layer="95" rot="R90"/>
+<attribute name="VALUE" x="-14.605" y="38.608" size="1.778" layer="96" rot="R90"/>
+</instance>
+<instance part="R5" gate="G$1" x="-20.32" y="50.8" smashed="yes" rot="R270">
+<attribute name="NAME" x="-18.8214" y="54.61" size="1.778" layer="95" rot="R270"/>
+<attribute name="VALUE" x="-23.622" y="54.61" size="1.778" layer="96" rot="R270"/>
+</instance>
+<instance part="SUPPLY21" gate="GND" x="-20.32" y="35.56" smashed="yes">
+<attribute name="VALUE" x="-22.225" y="32.385" size="1.778" layer="96"/>
+</instance>
+<instance part="SUPPLY22" gate="+12V" x="-17.78" y="55.88" smashed="yes" rot="R270">
+<attribute name="VALUE" x="-14.605" y="58.42" size="1.778" layer="96" rot="R270"/>
+</instance>
+<instance part="R6" gate="G$1" x="-25.4" y="119.38" smashed="yes" rot="R270">
+<attribute name="NAME" x="-23.9014" y="123.19" size="1.778" layer="95" rot="R270"/>
+<attribute name="VALUE" x="-28.702" y="123.19" size="1.778" layer="96" rot="R270"/>
+</instance>
+<instance part="LED2" gate="G$1" x="-25.4" y="111.76" smashed="yes">
+<attribute name="NAME" x="-21.844" y="107.188" size="1.778" layer="95" rot="R90"/>
+<attribute name="VALUE" x="-19.685" y="107.188" size="1.778" layer="96" rot="R90"/>
+</instance>
+<instance part="SUPPLY23" gate="G$1" x="-25.4" y="104.14" smashed="yes">
+<attribute name="VALUE" x="-28.067" y="100.965" size="1.778" layer="96"/>
 </instance>
 </instances>
@@
 <junction x="106.68" y="83.82"/>
 </segment>
+<segment>
+<pinref part="D1" gate="G$1" pin="A"/>
+<pinref part="D2" gate="G$1" pin="C"/>
+<wire x1="-20.32" y1="76.2" x2="-20.32" y2="71.12" width="0.1524" layer="91"/>
+<pinref part="SUPPLY20" gate="GND" pin="GND"/>
+<wire x1="-20.32" y1="71.12" x2="-20.32" y2="66.04" width="0.1524" layer="91"/>
+<junction x="-20.32" y="71.12"/>
+</segment>
+<segment>
+<pinref part="LED1" gate="G$1" pin="C"/>
+<pinref part="SUPPLY21" gate="GND" pin="GND"/>
+<junction x="-20.32" y="38.1"/>
+</segment>
 </net>
 <net name="+12V" class="1">
@@
 <junction x="106.68" y="91.44"/>
 <pinref part="C7" gate="G$1" pin="1"/>
+</segment>
+<segment>
+<pinref part="R5" gate="G$1" pin="1"/>
+<pinref part="SUPPLY22" gate="+12V" pin="+12V"/>
+<junction x="-20.32" y="55.88"/>
 </segment>
 </net>
@@
 <junction x="0" y="104.14"/>
 <junction x="0" y="106.68"/>
-</segment>
-</net>
-<net name="N$11" class="1">
+<pinref part="R6" gate="G$1" pin="1"/>
+<wire x1="-25.4" y1="124.46" x2="0" y2="124.46" width="0.1524" layer="91"/>
+<wire x1="0" y1="124.46" x2="0" y2="106.68" width="0.1524" layer="91"/>
+<junction x="-25.4" y="124.46"/>
+</segment>
+</net>
+<net name="DGND" class="1">
 <segment>
 <pinref part="SPI_IN" gate="-8" pin="S"/>
@@
 <wire x1="12.7" y1="119.38" x2="20.32" y2="119.38" width="0.1524" layer="91"/>
 <junction x="20.32" y="119.38"/>
+<pinref part="SUPPLY18" gate="G$1" pin="DGND"/>
+<junction x="5.08" y="119.38"/>
+</segment>
+<segment>
+<pinref part="D2" gate="G$1" pin="A"/>
+<pinref part="D1" gate="G$1" pin="C"/>
+<wire x1="-15.24" y1="66.04" x2="-15.24" y2="71.12" width="0.1524" layer="91"/>
+<pinref part="SUPPLY19" gate="G$1" pin="DGND"/>
+<wire x1="-15.24" y1="71.12" x2="-15.24" y2="76.2" width="0.1524" layer="91"/>
+<junction x="-15.24" y="71.12"/>
+</segment>
+<segment>
+<pinref part="LED2" gate="G$1" pin="C"/>
+<pinref part="SUPPLY23" gate="G$1" pin="DGND"/>
+<junction x="-25.4" y="106.68"/>
 </segment>
 </net>
@@
 </segment>
 </net>
+<net name="N$15" class="0">
+<segment>
+<pinref part="IC1" gate="G$1" pin="TEMP"/>
+<wire x1="78.74" y1="60.96" x2="91.44" y2="60.96" width="0.1524" layer="91"/>
+<pinref part="DAC_OUT" gate="-6" pin="S"/>
+<wire x1="91.44" y1="60.96" x2="91.44" y2="101.6" width="0.1524" layer="91"/>
+<wire x1="91.44" y1="101.6" x2="106.68" y2="101.6" width="0.1524" layer="91"/>
+<junction x="78.74" y="60.96"/>
+<junction x="106.68" y="101.6"/>
+</segment>
+</net>
+<net name="N$11" class="0">
+<segment>
+<pinref part="LED1" gate="G$1" pin="A"/>
+<pinref part="R5" gate="G$1" pin="2"/>
+<junction x="-20.32" y="45.72"/>
+</segment>
+</net>
+<net name="N$16" class="0">
+<segment>
+<pinref part="R6" gate="G$1" pin="2"/>
+<pinref part="LED2" gate="G$1" pin="A"/>
+<junction x="-25.4" y="114.3"/>
+</segment>
+</net>
