File: host_board/hall_sensor100a.sch (EAGLE design)
At the start: 26 parts, among them IC1 REF02HCSA, IC2 CSLT6B100, IC3 MAX5322EAI+, X1 22-23-2051

Commit message: up
Parts:
- added PAD3: DUD, wirepad:2,15/1,0
Connections:
- net GND: now also PAD3.P
Changed lines of the file:
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@@
 <part name="LED2" library="led" library_urn="urn:adsk.eagle:library:259" deviceset="LED" device="CHIPLED_1206" package3d_urn="urn:adsk.eagle:package:15823/2" value="5v_led"/>
 <part name="SUPPLY23" library="supply2" library_urn="urn:adsk.eagle:library:372" deviceset="DGND" device=""/>
+<part name="PAD3" library="wirepad" library_urn="urn:adsk.eagle:library:412" deviceset="2,15/1,0" device="" package3d_urn="urn:adsk.eagle:package:30831/1" value="DUD"/>
+<part name="SUPPLY24" library="supply2" library_urn="urn:adsk.eagle:library:372" deviceset="GND" device=""/>
 </parts>
 <sheets>
@@
 <instance part="SUPPLY23" gate="G$1" x="-25.4" y="104.14" smashed="yes">
 <attribute name="VALUE" x="-28.067" y="100.965" size="1.778" layer="96"/>
+</instance>
+<instance part="PAD3" gate="1" x="99.06" y="22.86" smashed="yes">
+<attribute name="NAME" x="97.917" y="24.7142" size="1.778" layer="95"/>
+<attribute name="VALUE" x="97.917" y="19.558" size="1.778" layer="96"/>
+</instance>
+<instance part="SUPPLY24" gate="GND" x="101.6" y="20.32" smashed="yes">
+<attribute name="VALUE" x="99.695" y="17.145" size="1.778" layer="96"/>
 </instance>
 </instances>
@@
 <junction x="-20.32" y="38.1"/>
 </segment>
+<segment>
+<pinref part="PAD3" gate="1" pin="P"/>
+<pinref part="SUPPLY24" gate="GND" pin="GND"/>
+</segment>
 </net>

Commit message: up
Parts:
- added PAD4: DUD2, wirepad:2,15/1,0
- added SV1: MON1, con-lstb:MA04-1
- PAD3: value DUD -> DUD1
Connections:
- net DGND: now also PAD4.P
- net GND: now also SV1.1
- net N$1: now also SV1.2
- net N$15: now also SV1.3
- net N$2: now also SV1.4
Changed lines of the file:
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@@
 <part name="LED2" library="led" library_urn="urn:adsk.eagle:library:259" deviceset="LED" device="CHIPLED_1206" package3d_urn="urn:adsk.eagle:package:15823/2" value="5v_led"/>
 <part name="SUPPLY23" library="supply2" library_urn="urn:adsk.eagle:library:372" deviceset="DGND" device=""/>
-<part name="PAD3" library="wirepad" library_urn="urn:adsk.eagle:library:412" deviceset="2,15/1,0" device="" package3d_urn="urn:adsk.eagle:package:30831/1" value="DUD"/>
+<part name="PAD3" library="wirepad" library_urn="urn:adsk.eagle:library:412" deviceset="2,15/1,0" device="" package3d_urn="urn:adsk.eagle:package:30831/1" value="DUD1"/>
 <part name="SUPPLY24" library="supply2" library_urn="urn:adsk.eagle:library:372" deviceset="GND" device=""/>
+<part name="SV1" library="con-lstb" library_urn="urn:adsk.eagle:library:162" deviceset="MA04-1" device="" package3d_urn="urn:adsk.eagle:package:8337/1" value="MON1"/>
+<part name="SUPPLY25" library="supply2" library_urn="urn:adsk.eagle:library:372" deviceset="GND" device=""/>
+<part name="PAD4" library="wirepad" library_urn="urn:adsk.eagle:library:412" deviceset="2,15/1,0" device="" package3d_urn="urn:adsk.eagle:package:30831/1" value="DUD2"/>
+<part name="SUPPLY26" library="supply2" library_urn="urn:adsk.eagle:library:372" deviceset="DGND" device=""/>
 </parts>
 <sheets>
@@
 <instance part="SUPPLY24" gate="GND" x="101.6" y="20.32" smashed="yes">
 <attribute name="VALUE" x="99.695" y="17.145" size="1.778" layer="96"/>
+</instance>
+<instance part="SV1" gate="1" x="127" y="71.12" smashed="yes" rot="R180">
+<attribute name="VALUE" x="128.27" y="81.28" size="1.778" layer="96" rot="R180"/>
+<attribute name="NAME" x="128.27" y="65.278" size="1.778" layer="95" rot="R180"/>
+</instance>
+<instance part="SUPPLY25" gate="GND" x="119.38" y="78.74" smashed="yes" rot="R180">
+<attribute name="VALUE" x="121.285" y="81.915" size="1.778" layer="96" rot="R180"/>
+</instance>
+<instance part="PAD4" gate="1" x="111.76" y="22.86" smashed="yes">
+<attribute name="NAME" x="110.617" y="24.7142" size="1.778" layer="95"/>
+<attribute name="VALUE" x="110.617" y="19.558" size="1.778" layer="96"/>
+</instance>
+<instance part="SUPPLY26" gate="G$1" x="114.3" y="20.32" smashed="yes">
+<attribute name="VALUE" x="111.633" y="17.145" size="1.778" layer="96"/>
 </instance>
 </instances>
@@
 <pinref part="SUPPLY24" gate="GND" pin="GND"/>
 </segment>
+<segment>
+<pinref part="SV1" gate="1" pin="1"/>
+<pinref part="SUPPLY25" gate="GND" pin="GND"/>
+<junction x="119.38" y="76.2"/>
+</segment>
 </net>
 <net name="+12V" class="1">
@@
 <wire x1="35.56" y1="55.88" x2="35.56" y2="76.2" width="0.1524" layer="91"/>
 <wire x1="35.56" y1="76.2" x2="96.52" y2="76.2" width="0.1524" layer="91"/>
-<wire x1="96.52" y1="76.2" x2="96.52" y2="58.42" width="0.1524" layer="91"/>
+<wire x1="96.52" y1="76.2" x2="96.52" y2="68.58" width="0.1524" layer="91"/>
 <pinref part="X1" gate="-2" pin="S"/>
+<wire x1="96.52" y1="68.58" x2="96.52" y2="58.42" width="0.1524" layer="91"/>
 <wire x1="96.52" y1="58.42" x2="101.6" y2="58.42" width="0.1524" layer="91"/>
 <junction x="101.6" y="58.42"/>
@@
 <wire x1="35.56" y1="48.26" x2="35.56" y2="55.88" width="0.1524" layer="91"/>
 <junction x="5.08" y="40.64"/>
+<pinref part="SV1" gate="1" pin="4"/>
+<wire x1="119.38" y1="68.58" x2="96.52" y2="68.58" width="0.1524" layer="91"/>
+<junction x="96.52" y="68.58"/>
+<junction x="119.38" y="68.58"/>
 </segment>
 </net>
@@
 <wire x1="17.78" y1="78.74" x2="78.74" y2="78.74" width="0.1524" layer="91"/>
 <wire x1="78.74" y1="78.74" x2="81.28" y2="78.74" width="0.1524" layer="91"/>
-<wire x1="81.28" y1="78.74" x2="81.28" y2="63.5" width="0.1524" layer="91"/>
+<wire x1="81.28" y1="78.74" x2="81.28" y2="73.66" width="0.1524" layer="91"/>
 <pinref part="IC1" gate="G$1" pin="V-OUT"/>
+<wire x1="81.28" y1="73.66" x2="81.28" y2="63.5" width="0.1524" layer="91"/>
 <wire x1="81.28" y1="63.5" x2="78.74" y2="63.5" width="0.1524" layer="91"/>
 <junction x="0" y="55.88"/>
@@
 <junction x="78.74" y="99.06"/>
 <junction x="106.68" y="99.06"/>
+<wire x1="81.28" y1="73.66" x2="119.38" y2="73.66" width="0.1524" layer="91"/>
+<junction x="81.28" y="73.66"/>
+<pinref part="SV1" gate="1" pin="2"/>
+<junction x="119.38" y="73.66"/>
+<wire x1="119.38" y1="73.66" x2="121.92" y2="73.66" width="0.1524" layer="91"/>
 </segment>
 </net>
@@
 <junction x="-25.4" y="106.68"/>
 </segment>
+<segment>
+<pinref part="PAD4" gate="1" pin="P"/>
+<pinref part="SUPPLY26" gate="G$1" pin="DGND"/>
+</segment>
 </net>
 <net name="N$12" class="0">
@@
 <wire x1="78.74" y1="60.96" x2="91.44" y2="60.96" width="0.1524" layer="91"/>
 <pinref part="DAC_OUT" gate="-6" pin="S"/>
-<wire x1="91.44" y1="60.96" x2="91.44" y2="101.6" width="0.1524" layer="91"/>
+<wire x1="91.44" y1="60.96" x2="91.44" y2="71.12" width="0.1524" layer="91"/>
+<wire x1="91.44" y1="71.12" x2="91.44" y2="101.6" width="0.1524" layer="91"/>
 <wire x1="91.44" y1="101.6" x2="106.68" y2="101.6" width="0.1524" layer="91"/>
 <junction x="78.74" y="60.96"/>
 <junction x="106.68" y="101.6"/>
-</segment>
-</net>
+<pinref part="SV1" gate="1" pin="3"/>
+<wire x1="119.38" y1="71.12" x2="91.44" y2="71.12" width="0.1524" layer="91"/>
+<junction x="91.44" y="71.12"/>
+<junction x="119.38" y="71.12"/>
+</segment>
+</net>
