File: host_board/hall_sensor100a.brd (EAGLE design)
At the start: 36.5 x 26.7 mm, 5 parts, among them IC1 REF02HCSA, IC2 CSLT6B100, X1 22-23-2051

Commit message: up
Parts:
- added PAD1, PAD2: (no value), wirepad:2,15/1,0
- added U$1: L01ZXXXS05A1, l01z:DIP2540W53P254L2900H508Q6B
- moved X1 4.02 mm to (24.1, 38.1)
- moved IC1 3.59 mm to (16.5, 39.4)
- moved IC2 3.59 mm to (5.08, 39.4)
- moved C1 2.84 mm to (16.5, 45.7)
- moved C2 2.84 mm to (16.5, 33.0)
Connections:
- net GND: now also PAD1.1, PAD2.1, U$1.2
- net N$1: now also U$1.3
- net N$2: now also U$1.1
Routing:
- net N$2: track 19.6 -> 63.6 mm
- net N$1: track 28.2 -> 62.2 mm
- net +12V: track 28.5 -> 14.9 mm
- net GND: track 23.5 -> 21.5 mm
Other:
- board size 36.5 x 26.7 mm -> 46.7 x 47 mm

Commit message: up
Parts:
- added C3: 22uf, rcl:C0805
- added C4: 2.2uf, rcl:C0805
- added IC3: MAX5322EAI+, MAX5322EAI+:SOP65P778X199-28N
Connections:
- net +12V: now also C4.1
- net GND: now also C3.2, C4.2
- net N$1: now also C3.1
Changed lines of the file:
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@@
 <?xml version="1.0" encoding="utf-8"?>
 <!DOCTYPE eagle SYSTEM "eagle.dtd">
-<eagle version="9.5.1">
+<eagle version="9.5.2">
 <drawing>
 <settings>
@@
 <attribute name="VALUE" x="25.4" y="54.34" size="0.0254" layer="27"/>
 </element>
+<element name="C3" library="rcl" library_urn="urn:adsk.eagle:library:334" package="C0805" package3d_urn="urn:adsk.eagle:package:23617/2" value="22uf" x="-7.62" y="25.4" smashed="yes">
+<attribute name="NAME" x="-8.89" y="26.67" size="1.27" layer="25"/>
+<attribute name="POPULARITY" value="63" x="-7.62" y="25.4" size="1.778" layer="27" display="off"/>
+<attribute name="SPICEPREFIX" value="C" x="-7.62" y="25.4" size="1.778" layer="27" display="off"/>
+<attribute name="VALUE" x="-8.89" y="22.86" size="1.27" layer="27"/>
+</element>
+<element name="C4" library="rcl" library_urn="urn:adsk.eagle:library:334" package="C0805" package3d_urn="urn:adsk.eagle:package:23617/2" value="2.2uf" x="-7.62" y="19.05" smashed="yes">
+<attribute name="NAME" x="-8.89" y="20.32" size="1.27" layer="25"/>
+<attribute name="POPULARITY" value="63" x="-7.62" y="19.05" size="1.778" layer="27" display="off"/>
+<attribute name="SPICEPREFIX" value="C" x="-7.62" y="19.05" size="1.778" layer="27" display="off"/>
+<attribute name="VALUE" x="-8.89" y="16.51" size="1.27" layer="27"/>
+</element>
+<element name="IC3" library="MAX5322EAI+" package="SOP65P778X199-28N" value="MAX5322EAI+" x="-15.24" y="21.59" smashed="yes">
+<attribute name="DESCRIPTION" value="Maxim MAX5322EAI+, 2-channel 12 bit Serial DAC, 28-Pin SSOP" x="-15.24" y="21.59" size="1.778" layer="27" display="off"/>
+<attribute name="HEIGHT" value="1.99mm" x="-15.24" y="21.59" size="1.778" layer="27" display="off"/>
+<attribute name="MANUFACTURER_NAME" value="Maxim Integrated" x="-15.24" y="21.59" size="1.778" layer="27" display="off"/>
+<attribute name="MANUFACTURER_PART_NUMBER" value="MAX5322EAI+" x="-15.24" y="21.59" size="1.778" layer="27" display="off"/>
+<attribute name="MOUSER_PART_NUMBER" value="700-MAX5322EAI" x="-15.24" y="21.59" size="1.778" layer="27" display="off"/>
+<attribute name="MOUSER_PRICE-STOCK" value="https://www.mouser.com/Search/Refine.aspx?Keyword=700-MAX5322EAI" x="-15.24" y="21.59" size="1.778" layer="27" display="off"/>
+<attribute name="NAME" x="-15.24" y="21.59" size="1.27" layer="25" align="center"/>
+<attribute name="RS_PART_NUMBER" value="7997645P" x="-15.24" y="21.59" size="1.778" layer="27" display="off"/>
+<attribute name="RS_PRICE-STOCK" value="http://uk.rs-online.com/web/p/products/7997645P" x="-15.24" y="21.59" size="1.778" layer="27" display="off"/>
+<attribute name="VALUE" x="-15.24" y="21.59" size="1.27" layer="27" align="center"/>
+</element>
 </elements>
 <signals>
@@
 <wire x1="17.6784" y1="33.0708" x2="17.46" y2="33.02" width="0.35" layer="1"/>
 <wire x1="24.0792" y1="33.0708" x2="24.13" y2="33.02" width="0.35" layer="1"/>
+<contactref element="C3" pad="2"/>
+<contactref element="C4" pad="2"/>
+<wire x1="25.4" y1="53.34" x2="26.67" y2="72.39" width="0" layer="19" extent="1-1"/>
+<wire x1="24.13" y1="40.64" x2="17.46" y2="45.72" width="0" layer="19" extent="1-1"/>
+<wire x1="18.415" y1="36.2966" x2="24.13" y2="40.64" width="0" layer="19" extent="1-1"/>
+<wire x1="7.874" y1="39.37" x2="18.415" y2="36.2966" width="0" layer="19" extent="1-1"/>
+<wire x1="-6.67" y1="25.4" x2="7.874" y2="39.37" width="0" layer="19" extent="1-1"/>
+<wire x1="-6.67" y1="19.05" x2="-6.67" y2="25.4" width="0" layer="19" extent="1-1"/>
+<wire x1="0" y1="66.04" x2="17.46" y2="45.72" width="0" layer="19" extent="1-1"/>
 </signal>
 <signal name="+12V" class="1">
@@
 <wire x1="15.9258" y1="36.4236" x2="15.875" y2="36.2966" width="0.35" layer="1"/>
 <wire x1="24.0792" y1="43.1292" x2="24.13" y2="43.18" width="0.35" layer="1"/>
+<contactref element="C4" pad="1"/>
+<wire x1="-8.57" y1="19.05" x2="15.56" y2="33.02" width="0" layer="19" extent="1-1"/>
 </signal>
 <signal name="N$2">
@@
 <wire x1="24.1554" y1="38.1" x2="24.13" y2="38.1" width="0.35" layer="1"/>
 <wire x1="17.2212" y1="43.2054" x2="17.145" y2="42.4434" width="0.35" layer="1"/>
+<contactref element="C3" pad="1"/>
+<wire x1="-8.57" y1="25.4" x2="6.35" y2="39.37" width="0" layer="19" extent="1-1"/>
 </signal>
 </signals>

Commit message: up
Parts:
- added C5, C7: 0.1, rcl:C0805
- added C6: 22uf, rcl:C0805
- added DAC_OUT, SPI_IN: 22-23-2101, con-molex:22-23-2101
- moved IC3 58.6 mm to (40.6, 39.4), turned to 90 degrees
- moved C4 22.9 mm to (11.4, 31.8), turned to 180 degrees
- moved C3 15.3 mm to (6.35, 31.8)
Connections:
- new net N$10: C5.1, C6.1, IC3.17, IC3.3, IC3.4, IC3.6, IC3.8, SPI_IN.7
- new net N$11: C5.2, C6.2, IC3.7, SPI_IN.8
- new net N$12: IC3.5, SPI_IN.4
- new net N$4: DAC_OUT.2, IC3.18
- new net N$5: DAC_OUT.3, IC3.25
- new net N$6: IC3.11, SPI_IN.2
- new net N$7: IC3.9, SPI_IN.1
- new net N$8: IC3.10, SPI_IN.3
- new net N$9: IC3.12, SPI_IN.9
- net +12V: now also C7.1, DAC_OUT.10, IC3.21
- net GND: now also C7.2, DAC_OUT.1, IC3.19, IC3.23, IC3.24, IC3.26
- net N$1: now also DAC_OUT.7, IC3.20, IC3.22
Routing:
- net +12V: track 14.9 -> 88.6 mm, vias 0 -> 2
- net N$1: track 62.2 -> 113.7 mm, vias 0 -> 1
- net N$10: track 0.00 -> 35.7 mm
- net GND: track 21.5 -> 50.7 mm
- net N$7: track 0.00 -> 28.4 mm, vias 0 -> 1
- net N$6: track 0.00 -> 26.9 mm, vias 0 -> 1
- net N$11: track 0.00 -> 26.2 mm
- net N$8: track 0.00 -> 24.8 mm, vias 0 -> 1
- net N$12: track 0.00 -> 17.2 mm
- net N$9: track 0.00 -> 12.2 mm
- net N$5: track 0.00 -> 11.9 mm
- net N$4: track 0.00 -> 8.98 mm
- net N$2: track 63.6 -> 55.3 mm
Other:
- board size 46.7 x 47 mm -> 59.4 x 55.9 mm
- board text added: "MBMC CURRENT and DAC BOARD 1.0"
- board text added: "fgb@mchp"

Commit message: up
Parts:
- added R1, R2, R3: 50, rcl:M0805
- added R4: 4.7k, rcl:M0805
Connections:
- new net N$13: IC3.10, R2.2
- new net N$14: IC3.12, R3.2
- new net N$3: IC3.11, R1.2
- net N$10: now also R4.2
- net N$12: now also R4.1
- net N$6: now also R1.1; no longer IC3.11
- net N$8: now also R2.1; no longer IC3.10
- net N$9: now also R3.1; no longer IC3.12
Routing:
- net N$10: track 35.7 -> 81.4 mm, vias 0 -> 1
- net N$12: track 17.2 -> 35.9 mm
- net N$14: track 0.00 -> 13.5 mm, vias 0 -> 2
- net N$8: track 24.8 -> 11.7 mm, vias 1 -> 0
- net N$13: track 0.00 -> 12.1 mm
- net N$3: track 0.00 -> 11.6 mm
- net N$6: track 26.9 -> 16.5 mm, vias 1 -> 0
- net +12V: track 88.6 -> 82.3 mm, vias 2 -> 1
- net N$1: track 113.7 -> 108.6 mm
- net N$9: track 12.2 -> 10.7 mm
- net GND: track 50.7 -> 49.5 mm
- net N$7: track 28.4 -> 29.0 mm
- net N$11: track 26.2 -> 25.9 mm, vias 0 -> 2

Commit message: up
Parts:
- added D1: btb1, diode:DO35-7
- added D2: btb2, diode:DO35-7
- added LED1: 12v_led, led:CHIPLED_1206
- added LED2: 5v_led, led:CHIPLED_1206
- added R5, R6: 4.7k, rcl:M0805
- moved R4 22.5 mm to (35.6, 31.8), turned to 270 degrees
- moved R2 2.84 mm to (33.0, 36.8), turned to 90 degrees
- moved C6 2.54 mm to (41.9, 31.8), turned to 90 degrees
- moved R1 1.80 mm to (30.5, 36.8), turned to 90 degrees
- moved R3 1.80 mm to (33.0, 31.8), turned to 90 degrees
- moved C5 1.27 mm to (45.7, 31.8), turned to 270 degrees
Connections:
- new net DGND: C5.2, C6.2, D1.C, D2.A, IC3.7, LED2.C, SPI_IN.8
- new net N$15: DAC_OUT.6, IC1.3
- new net N$16: LED2.A, R6.2
- net +12V: now also R5.1
- net GND: now also D1.A, D2.C, LED1.C
- net N$10: now also R6.1
- net N$11: now also LED1.A, R5.2; no longer C5.2, C6.2, IC3.7, SPI_IN.8
Routing:
- net N$15: track 0.00 -> 37.3 mm
- net DGND: track 0.00 -> 33.8 mm, vias 0 -> 2
- net N$10: track 81.4 -> 109.4 mm, vias 1 -> 2
- net N$2: track 55.6 -> 77.1 mm
- net N$12: track 35.9 -> 19.6 mm
- net GND: track 49.5 -> 58.7 mm, vias 0 -> 1
- net N$16: track 0.00 -> 7.78 mm
- net N$11: track 25.9 -> 19.2 mm, vias 2 -> 0
- net +12V: track 82.3 -> 75.7 mm, vias 1 -> 5
- net N$3: track 11.6 -> 14.5 mm
- net N$8: track 11.7 -> 14.2 mm
- net N$6: track 16.5 -> 14.2 mm
- net N$9: track 10.7 -> 8.58 mm
- net N$13: track 12.1 -> 10.6 mm
- net N$14: track 13.5 -> 13.1 mm, vias 2 -> 0
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- added copper zone on layer 16, net DGND

Commit message: up
Parts:
- added PAD3: DUD, wirepad:2,15/1,0
Connections:
- net GND: now also PAD3.1
Changed lines of the file:
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@@
 <wire x1="49.2" y1="76.19" x2="-10.16" y2="76.19" width="0" layer="20"/>
 <wire x1="-10.16" y1="76.19" x2="-10.16" y2="20.32" width="0" layer="20"/>
-<hole x="-7.62" y="73.66" drill="1"/>
-<hole x="-7.62" y="22.86" drill="1"/>
-<hole x="46.99" y="22.86" drill="1"/>
-<hole x="46.99" y="73.66" drill="1"/>
+<hole x="-7.62" y="73.66" drill="2.5"/>
+<hole x="-7.62" y="22.86" drill="2.5"/>
+<hole x="46.99" y="22.86" drill="2.5"/>
+<hole x="46.99" y="73.66" drill="2.5"/>
 <hole x="1.27" y="39.37" drill="6.858"/>
-<text x="-5.08" y="26.67" size="1.778" layer="1" font="vector" ratio="16" rot="R90">MBMC CURRENT and DAC BOARD 1.0</text>
+<text x="-6.35" y="26.67" size="1.778" layer="1" font="vector" ratio="16" rot="R90">MBMC CURRENT and DAC BOARD 1.0</text>
 <text x="3.81" y="71.12" size="1.27" layer="1" font="vector" ratio="15">fgb@mchp</text>
 </plain>
@@
 <attribute name="VALUE" x="5.08" y="24.13" size="1.27" layer="27" rot="R90"/>
 </element>
+<element name="PAD3" library="wirepad" library_urn="urn:adsk.eagle:library:412" package="2,15/1,0" package3d_urn="urn:adsk.eagle:package:30831/1" value="DUD" x="10.16" y="48.26" smashed="yes">
+<attribute name="NAME" x="9.017" y="49.657" size="1.27" layer="25" ratio="10"/>
+<attribute name="POPULARITY" value="11" x="10.16" y="48.26" size="1.778" layer="27" display="off"/>
+<attribute name="VALUE" x="10.16" y="49.26" size="0.0254" layer="27"/>
+</element>
 </elements>
 <signals>
@@
 <wire x1="36.4236" y1="45.72" x2="36.576" y2="45.72" width="0.35" layer="1"/>
 <via x="36.4236" y="45.72" extent="1-16" drill="0.35"/>
+<contactref element="PAD3" pad="1"/>
+<wire x1="25.4" y1="53.34" x2="26.67" y2="72.39" width="0" layer="19" extent="1-1"/>
+<wire x1="24.13" y1="40.64" x2="17.46" y2="45.72" width="0" layer="19" extent="1-1"/>
+<wire x1="18.415" y1="36.2966" x2="24.13" y2="40.64" width="0" layer="19" extent="1-1"/>
+<wire x1="10.48" y1="31.75" x2="17.46" y2="33.02" width="0" layer="19" extent="1-1"/>
+<wire x1="6.35" y1="22.86" x2="6.35" y2="26.67" width="0" layer="19" extent="1-1"/>
+<wire x1="7.874" y1="39.37" x2="7.3" y2="31.75" width="0" layer="19" extent="1-1"/>
+<wire x1="36.51" y1="48.26" x2="25.4" y2="53.34" width="0" layer="19" extent="1-1"/>
+<wire x1="42.265" y1="42.868" x2="39.665" y2="42.868" width="0" layer="19" extent="1-1"/>
+<wire x1="10.16" y1="48.26" x2="0" y2="27.15" width="0" layer="19" extent="1-1"/>
+<wire x1="0" y1="66.04" x2="17.46" y2="45.72" width="0" layer="19" extent="1-1"/>
 </signal>
 <signal name="+12V" class="1">

Commit message: up
Parts:
- added PAD4: DUD2, wirepad:2,15/1,0
- added SV1: MON1, con-lstb:MA04-1
- PAD3: value DUD -> DUD1
- moved C3 28.1 mm to (33.0, 22.9)
- moved C4 28.1 mm to (38.1, 22.9)
- moved C5 28.1 mm to (72.4, 22.9)
- moved C6 28.1 mm to (68.6, 22.9)
- moved DAC_OUT 28.1 mm to (68.6, 50.8)
- moved PAD2 28.1 mm to (52.1, 44.5)
- moved R6 28.1 mm to (27.9, 21.6)
- moved U$1 28.1 mm to (53.3, 50.8)
- moved C1 28.1 mm to (43.2, 36.8)
- moved C2 28.1 mm to (43.2, 24.1)
- moved D1 28.1 mm to (36.8, 17.8)
- moved D2 28.1 mm to (36.8, 14.0)
- moved IC1 28.1 mm to (43.2, 30.5)
- moved IC2 28.1 mm to (31.8, 30.5)
- moved IC3 28.1 mm to (67.3, 30.5)
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Connections:
- net DGND: now also PAD4.1
- net GND: now also SV1.1
- net N$1: now also SV1.2
- net N$15: now also SV1.3
- net N$2: now also SV1.4
Routing:
- net N$15: track 37.3 -> 62.0 mm
- net +12V: track 75.7 -> 93.3 mm, vias 5 -> 4
- net N$1: track 108.4 -> 121.4 mm
- net GND: track 58.7 -> 70.1 mm, vias 1 -> 0
- net N$10: track 109.4 -> 98.7 mm
- net DGND: track 33.8 -> 23.4 mm
- net N$2: track 77.1 -> 68.9 mm
- net N$11: track 19.2 -> 21.8 mm
Other:
- board size 59.4 x 55.9 mm -> 60.6 x 57.1 mm
- board text added: "MBMC CURRENT and DAC BOARD 1.1"
- board text removed: "MBMC CURRENT and DAC BOARD 1.0"

Commit message: up
Parts:
- moved D2 1.27 mm to (36.8, 12.7)
Routing:
- net +12V: track 93.3 -> 79.2 mm, vias 4 -> 5
- net N$2: track 68.9 -> 73.5 mm
- net N$10: track 98.7 -> 94.6 mm
- net N$1: track 121.4 -> 123.2 mm, vias 1 -> 2
- net N$5: track 12.0 -> 13.0 mm
- net GND: track 70.1 -> 70.9 mm
