File: touch_board/touch_board.brd (EAGLE design)
At the start: 46.7 x 31.7 mm, 10 parts, among them IC1 PIC18F47K42-I_PT

Commit message: update
Parts:
- added C7: 0.1, rcl:C0805
- added LED1: RUN, led:CHIPLED_1206
- added LED2: MODE, led:CHIPLED_1206
- added R3, R5, R7: 220, rcl:R0805
- added R4: 10k, rcl:R0805
- added SV1: ICSP, con-lstb:MA06-1
- added SV2: IO1, con-lstb:MA05-2
- added SV3: RESET, con-lstb:MA03-1
- moved C6 13.7 mm to (55.9, 73.7), turned to 180 degrees
- moved R1 3.59 mm to (67.3, 63.5), turned to 0 degrees
- moved C4 3.59 mm to (67.3, 58.4), turned to 180 degrees
- moved C2 2.84 mm to (36.8, 63.5), turned to 180 degrees
- moved C1 2.84 mm to (36.8, 58.4), turned to 180 degrees
- moved C5 2.84 mm to (41.9, 63.5), turned to 180 degrees
- moved R2 2.54 mm to (62.2, 63.5), turned to 0 degrees
- moved C3 2.54 mm to (62.2, 58.4), turned to 180 degrees
Connections:
- new net N$10: IC1.39, R7.2
- new net N$11: LED2.A, R7.1
- new net N$2: C7.1, R3.1, R4.1, SV1.1, SV2.4, SV3.1
- new net N$3: IC1.18, R3.2
- new net N$4: IC1.25, R5.2, SV2.1
- new net N$5: IC1.26, SV2.2
- new net N$6: IC1.17, SV1.4
- new net N$7: IC1.16, SV1.5
- new net N$8: IC1.27, SV2.3
- new net N$9: LED1.A, R5.1
- net VDD: now also R4.2, SV1.2, SV2.9
- net VSS: now also C7.2, LED1.C, LED2.C, SV1.3, SV2.10, SV3.2, SV3.3
Routing:
- net N$2: track 0.00 -> 53.4 mm
- net N$4: track 0.00 -> 46.1 mm, vias 0 -> 1
- net VDD: track 54.0 -> 96.5 mm
- net N$8: track 0.00 -> 40.9 mm, vias 0 -> 1
- net N$5: track 0.00 -> 36.9 mm, vias 0 -> 2
- net N$11: track 0.00 -> 20.5 mm
- net N$7: track 0.00 -> 19.0 mm, vias 0 -> 1
- net N$9: track 0.00 -> 17.6 mm
- net N$1: track 7.65 -> 24.7 mm
- net N$10: track 0.00 -> 15.7 mm, vias 0 -> 2
- net N$6: track 0.00 -> 15.0 mm, vias 0 -> 1
- net VCC: track 4.55 -> 11.3 mm
- net N$3: track 0.00 -> 5.41 mm
- net GND: track 34.1 -> 33.7 mm, vias 0 -> 2

Commit message: update
Parts:
- added C8: 0.1, rcl:C0805
- added C9: 10uf, rcl:C0805
- added IC2: MAX203EEWP, maxim-10:SO20L
- added JMP1, JMP2: 0R-JUMPA, jump-0r-smd:A0R-JMP
- added X1: RS-232-1, con-molex:22-23-2041
- added X2: RS-232-2, con-molex:22-23-2041
- added X3: POWER, con-molex:22-23-2021
- added X4: 22-23-2041, con-molex:22-23-2041
Connections:
- new net N$12: IC2.11, IC2.16
- new net N$13: IC2.10, IC2.17
- new net N$14: IC2.12, IC2.15
- new net N$15: IC2.5, X1.2
- new net N$16: IC2.18, X2.2
- new net N$17: IC2.4, X1.3
- new net N$18: IC2.19, X2.3
- new net N$19: IC1.44, IC2.2
- new net N$20: IC2.1, X4.1
- new net N$21: IC1.1, IC2.3
- new net N$22: IC2.20, X4.3
- net GND: now also C8.2, C9.2, IC2.6, IC2.9, JMP1.1, JMP1.3, JMP2.1, JMP2.3, X1.1, X2.1
- net N$6: now also X4.4
- net N$7: now also X4.2
- net VCC: now also C8.1, C9.1, IC2.7, X1.4, X2.4
- net VDD: now also X3.1
- net VSS: now also JMP1.2, JMP2.2, X3.2
Routing:
- net VCC: track 11.3 -> 112.4 mm, vias 0 -> 1
- net N$7: track 19.0 -> 68.2 mm
- net N$19: track 0.00 -> 46.7 mm, vias 0 -> 2
- net N$6: track 15.0 -> 59.7 mm
- net N$21: track 0.00 -> 34.1 mm, vias 0 -> 2
- net N$22: track 0.00 -> 28.6 mm
- net N$20: track 0.00 -> 20.2 mm, vias 0 -> 1
- net GND: track 33.7 -> 53.2 mm
- net N$18: track 0.00 -> 17.6 mm, vias 0 -> 1
- net N$16: track 0.00 -> 16.8 mm, vias 0 -> 1
- net VDD: track 96.5 -> 113.2 mm
- net N$15: track 0.00 -> 16.2 mm, vias 0 -> 1
- net N$17: track 0.00 -> 14.6 mm
- net N$13: track 0.00 -> 13.3 mm
- net N$12: track 0.00 -> 9.18 mm
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- added copper zone on layer 1, net GND
Other:
- board size 46.7 x 31.7 mm -> 68.2 x 39.4 mm

Commit message: update
Parts:
- removed X4: 22-23-2041, con-molex:22-23-2041
- added R6: 220, rcl:R0805
- added S1: ICD/SERIAL, JS202011SCQN:JS202011SCQN
- added S2: RESET_PB, switch-omron:B3F-10XX
- added SV4, SV5, SV6, SV7: IO1, con-lstb:MA05-2
- added XT1: HFBR-1521, fiber-optic-hp:HFBR-15X3
- moved SV1 25.4 mm to (41.9, 38.1)
- moved X3 17.8 mm to (54.6, 44.5)
- moved JMP2 6.35 mm to (33.0, 58.4)
- moved X2 6.35 mm to (14.0, 50.8)
- moved C5 6.35 mm to (36.8, 67.3)
- moved R7 6.35 mm to (41.9, 63.5)
- moved X1 5.08 mm to (14.0, 64.8)
- moved C7 4.02 mm to (54.6, 50.8), turned to 0 degrees
- moved C6 2.54 mm to (55.9, 76.2)
- moved LED1 2.54 mm to (49.5, 76.2)
- moved IC2 2.54 mm to (24.1, 59.7)
- moved C8 2.54 mm to (21.6, 69.8)
- moved C9 2.54 mm to (26.7, 69.8)
- moved OS1 1.80 mm to (63.5, 73.7)
Connections:
- new net N$23: S1.5, SV1.4
- new net N$24: S1.2, SV1.5
- new net N$25: R6.1, XT1.1
- new net N$26: IC1.19, SV4.1
- new net N$27: IC1.20, SV4.2
- new net N$28: IC1.21, SV4.3
- new net N$29: IC1.22, SV4.4
- new net N$30: IC1.23, SV4.5
- new net N$31: IC1.31, SV4.7
- new net N$32: IC1.24, SV4.6
- new net N$33: IC1.32, SV5.1
- new net N$34: IC1.35, SV5.2
- new net N$35: IC1.36, SV5.3
- new net N$36: IC1.37, SV5.4
- new net N$37: IC1.42, SV5.5
- new net N$38: IC1.43, SV5.6
- new net N$39: IC1.38, SV6.1
- new net N$40: IC1.40, SV6.3
- new net N$41: IC1.41, SV6.4
- new net N$42: IC1.2, SV6.5
- new net N$43: IC1.3, SV6.6
- new net N$44: IC1.4, SV6.7
- new net N$45: IC1.5, SV6.8
- new net N$46: IC1.8, SV7.1
- new net N$47: IC1.9, SV7.2
- new net N$48: IC1.10, SV7.3
- new net N$49: IC1.11, SV7.4
- new net N$50: IC1.14, SV7.5
- new net N$51: IC1.15, SV7.6
- net N$1: now also SV4.8
- net N$10: now also SV6.2
- net N$19: now also SV5.7
- net N$2: now also S2.2
- net N$20: now also R6.2, S1.1; no longer X4.1
- net N$21: now also SV5.8
- net N$22: now also S1.4; no longer X4.3
- net N$6: now also S1.6; no longer SV1.4, X4.4
- net N$7: now also S1.3; no longer SV1.5, X4.2
- net VDD: now also SV4.9, SV5.9, SV6.9, SV7.9
- net VSS: now also S2.4, SV4.10, SV5.10, SV6.10, SV7.10, XT1.2
Routing:
- net VSS: track 0.00 -> 242.2 mm, vias 0 -> 4
- net VDD: track 113.2 -> 215.2 mm, vias 0 -> 5
- net N$49: track 0.00 -> 96.1 mm
- net N$27: track 0.00 -> 95.1 mm, vias 0 -> 1
- net N$19: track 46.7 -> 127.5 mm, vias 2 -> 4
- net N$42: track 0.00 -> 75.1 mm, vias 0 -> 2
- net N$43: track 0.00 -> 70.4 mm, vias 0 -> 3
- net N$40: track 0.00 -> 66.2 mm, vias 0 -> 2
- net N$39: track 0.00 -> 63.9 mm, vias 0 -> 2
- net N$21: track 34.1 -> 95.3 mm, vias 2 -> 5
- net N$46: track 0.00 -> 55.1 mm, vias 0 -> 4
- net N$50: track 0.00 -> 51.5 mm, vias 0 -> 2
- net N$37: track 0.00 -> 50.7 mm, vias 0 -> 3
- net N$51: track 0.00 -> 47.6 mm, vias 0 -> 2
- net N$10: track 15.7 -> 62.5 mm, vias 2 -> 3
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- removed copper zone on layer 1, net VSS
Other:
- board size 68.2 x 39.4 mm -> 88.6 x 47 mm

Commit message: update
Parts:
- moved LED1 47.1 mm to (53.3, 29.2)
- moved R5 41.0 mm to (47.0, 26.7)
- moved SV4 40.4 mm to (64.8, 36.8), turned to 180 degrees
- moved C6 38.1 mm to (78.7, 45.7)
- moved OS1 37.5 mm to (78.7, 39.4)
- moved SV6 33.0 mm to (50.8, 64.8), turned to 90 degrees
- moved SV7 31.4 mm to (50.8, 49.5), turned to 90 degrees
- moved X1 31.4 mm to (25.4, 35.6), turned to 0 degrees
- moved R4 28.5 mm to (61.0, 29.2)
- moved X2 27.9 mm to (25.4, 25.4), turned to 0 degrees
- moved C7 27.2 mm to (71.1, 29.2)
- moved SV2 25.5 mm to (40.6, 49.5), turned to 90 degrees
- moved X3 25.4 mm to (39.4, 24.1)
- moved SV1 24.3 mm to (59.7, 21.6)
- moved XT1 22.5 mm to (81.3, 19.1)
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Connections:
- net N$6: now also SV7.8
- net N$7: now also SV7.7
Routing:
- net N$49: track 96.1 -> 11.5 mm
- net N$27: track 95.1 -> 14.0 mm, vias 1 -> 0
- net N$19: track 127.5 -> 55.4 mm, vias 4 -> 2
- net N$42: track 75.1 -> 14.8 mm, vias 2 -> 0
- net N$43: track 70.4 -> 16.6 mm, vias 3 -> 0
- net N$40: track 66.2 -> 14.5 mm, vias 2 -> 1
- net N$39: track 63.9 -> 15.0 mm, vias 2 -> 1
- net N$46: track 55.1 -> 10.4 mm, vias 4 -> 0
- net N$37: track 50.7 -> 8.48 mm, vias 3 -> 0
- net N$48: track 46.6 -> 6.05 mm, vias 2 -> 0
- net N$10: track 62.5 -> 23.3 mm, vias 3 -> 2
- net N$50: track 51.5 -> 12.6 mm, vias 2 -> 1
- net VDD: track 215.2 -> 181.8 mm, vias 5 -> 0
- net N$4: track 40.1 -> 71.1 mm, vias 4 -> 1
- net N$16: track 19.7 -> 48.0 mm, vias 1 -> 0
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Other:
- board size 88.6 x 47 mm -> 81 x 62.2 mm
- board text added: "FGB@MCHP 1.0"
- board text added: "These are the controllers you are looking for!"

Commit message: update
Parts:
- added K1: G6K-2P, relay:G6K-2P
- added L1, L2: 1000, inductor-neosid:SM-1206
- added X4: GLORY, con-molex:22-23-2021
- added X5: Relay conn, con-phoenix-254:8POL254
- moved R6 46.0 mm to (71.1, 22.9), turned to 180 degrees
- moved C9 8.89 mm to (21.6, 69.8)
- moved X3 3.81 mm to (35.6, 24.1)
- moved C8 2.54 mm to (26.7, 69.8)
- moved R5 1.80 mm to (48.3, 25.4)
- moved C6 1.27 mm to (80.0, 45.7)
Connections:
- new net N$52: IC1.38, K1.1, SV6.1, X5.1
- new net N$53: K1.3, X5.3
- new net N$54: K1.4, X5.4
- new net N$55: K1.5, X5.5
- new net N$56: K1.6, X5.6
- new net N$57: K1.7, X5.7
- new net N$58: C1.1, C2.1, C3.1, C5.1, IC1.28, IC1.7, L1.1, L2.2, R2.1
- net N$39: now also K1.2, X5.2; no longer IC1.38, SV6.1
- net VDD: now also L1.2, L2.1, X4.1; no longer C1.1, C2.1, C3.1, C5.1, IC1.28, IC1.7, R2.1
- net VSS: now also K1.8, X4.2, X5.8
Routing:
- net N$58: track 0.00 -> 73.1 mm, vias 0 -> 5
- net N$20: track 33.1 -> 97.7 mm, vias 2 -> 3
- net N$25: track 72.0 -> 15.4 mm
- net GND: track 76.5 -> 123.5 mm, vias 0 -> 2
- net N$52: track 0.00 -> 42.2 mm, vias 0 -> 1
- net VSS: track 257.0 -> 291.8 mm
- net N$57: track 0.00 -> 27.0 mm
- net N$2: track 97.1 -> 72.2 mm
- net N$56: track 0.00 -> 22.4 mm
- net VDD: track 181.8 -> 159.6 mm, vias 0 -> 2
- net N$17: track 31.3 -> 52.0 mm, vias 1 -> 0
- net N$23: track 55.5 -> 72.7 mm
- net N$55: track 0.00 -> 16.4 mm
- net N$22: track 19.3 -> 35.6 mm
- net N$8: track 50.5 -> 34.4 mm, vias 0 -> 1
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- added copper zone on layer 16, net GND
- added copper zone on layer 1, net VDD
- removed copper zone on layer 1, net GND

Commit message: update
Parts:
- added D1: 5.6V, diode:ZDIO-7.5
- added F1: 1206L050, polyfuse-smd_10:1206L
- moved C8 19.1 mm to (25.4, 50.8)
- moved C9 19.0 mm to (21.6, 50.8)
- moved S1 12.8 mm to (25.4, 34.3)
- moved X1 8.89 mm to (25.4, 44.5)
- moved SV3 4.58 mm to (49.5, 39.4), turned to 180 degrees
- moved R3 3.81 mm to (53.3, 34.3)
- moved S2 2.84 mm to (38.1, 38.1)
- moved C5 2.54 mm to (36.8, 68.6)
- turned X3 to 0 degrees
- turned X4 to 0 degrees
Connections:
- new net N$60: D1.C, F1.1, X3.1, X4.1
- net VDD: now also F1.2; no longer X3.1, X4.1
- net VSS: now also D1.A
Routing:
- net N$5: track 33.2 -> 78.0 mm
- net N$23: track 72.7 -> 47.4 mm
- net N$17: track 52.0 -> 30.9 mm
- net N$60: track 0.00 -> 20.5 mm
- net N$19: track 65.6 -> 85.8 mm, vias 2 -> 0
- net VCC: track 150.6 -> 131.9 mm, vias 0 -> 1
- net GND: track 123.5 -> 108.3 mm
- net VSS: track 291.8 -> 306.8 mm, vias 0 -> 1
- net N$30: track 9.62 -> 24.5 mm, vias 1 -> 0
- net N$24: track 58.0 -> 46.8 mm
- net N$21: track 75.8 -> 65.7 mm, vias 1 -> 0
- net N$15: track 28.5 -> 19.9 mm
- net N$4: track 62.6 -> 70.8 mm
- net N$7: track 44.4 -> 52.1 mm, vias 2 -> 4
- net N$3: track 15.6 -> 22.5 mm
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
Commit message: updatei# Please enter the commit message for your changes. Lines starting
Parts:
- removed LED1: RUN, led:CHIPLED_1206
- removed S2: RESET_PB, switch-omron:B3F-10XX
- added S3: RESETSW, SamacSys_Parts:B3W-9_1-LED
- moved R5 24.0 mm to (35.6, 45.7), turned to 270 degrees
- moved D1 13.3 mm to (50.8, 29.2)
Connections:
- net N$2: now also S3.1, S3.2; no longer S2.2
- net N$9: now also S3.5; no longer LED1.A
- net VSS: now also S3.3, S3.4, S3.6; no longer LED1.C, S2.4
Routing:
- net N$5: track 78.0 -> 34.0 mm, vias 1 -> 0
- net N$4: track 70.8 -> 41.9 mm
- net VSS: track 306.8 -> 287.8 mm
- net N$2: track 68.4 -> 86.1 mm
- net N$21: track 65.7 -> 76.3 mm, vias 0 -> 1
- net N$60: track 20.5 -> 30.2 mm
- net N$38: track 12.2 -> 18.1 mm
- net N$7: track 52.1 -> 57.6 mm, vias 4 -> 1
- net N$8: track 40.1 -> 45.5 mm, vias 3 -> 1
- net N$3: track 22.5 -> 17.4 mm
- net N$1: track 32.9 -> 37.7 mm, vias 2 -> 1
- net GND: track 108.3 -> 103.6 mm, vias 2 -> 1
- net N$23: track 47.4 -> 51.9 mm, vias 0 -> 1
- net VDD: track 155.3 -> 159.5 mm, vias 3 -> 2
- net N$22: track 30.5 -> 34.7 mm
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
Commit message: update
Parts:
- added D2: 1N4148, diode:SOD-123_MINI-SMA
- moved R4 2.84 mm to (63.5, 30.5)
Connections:
- new net N$59: C7.1, D2.A, R4.1
- net N$2: now also D2.C; no longer C7.1, R4.1
Routing:
- net N$2: track 86.1 -> 61.1 mm
- net VCC: track 129.8 -> 115.6 mm
- net N$59: track 0.00 -> 10.5 mm
- net N$23: track 51.9 -> 62.3 mm, vias 1 -> 0
- net VSS: track 287.8 -> 295.1 mm, vias 1 -> 0
- net VDD: track 159.5 -> 162.4 mm
- net N$7: track 57.6 -> 55.0 mm
- net N$58: track 69.7 -> 68.5 mm
- net N$50: track 11.8 -> 12.5 mm
- net N$51: track 16.0 -> 15.5 mm, vias 2 -> 3
- net N$24: track 48.3 -> 47.8 mm
