File: touch_board/touch_board.brd (EAGLE design)
At the start: 81 x 62.2 mm, 43 parts, among them IC1 PIC18F47K42-I_PT, IC2 MAX203EEWP, K1 G6K-2P, X1 RS-232-1, X2 RS-232-2, X3 POWER, X4 GLORY, X5 Relay conn

Commit message: update
Connections:
- removed net N$59: C7.1, D2.A, R4.1
- new net N$62: C7.1, D2.A, R4.1, S3.1, S3.2, SV3.1
- net N$2: no longer S3.1, S3.2, SV3.1
Routing:
- net N$62: track 0.00 -> 46.8 mm, vias 0 -> 1
- net VCC: track 115.6 -> 132.8 mm, vias 2 -> 1
- net N$1: track 37.7 -> 53.4 mm, vias 1 -> 0
- net N$4: track 41.9 -> 56.5 mm, vias 2 -> 1
- net VDD: track 162.4 -> 149.8 mm
- net N$30: track 20.4 -> 9.27 mm, vias 0 -> 1
- net N$59: track 10.5 -> 0.00 mm
- net N$2: track 61.1 -> 54.5 mm
- net N$38: track 18.1 -> 12.2 mm
- net N$8: track 45.5 -> 39.9 mm
- net VSS: track 295.1 -> 300.5 mm
- net N$31: track 18.7 -> 23.9 mm
- net N$34: track 15.0 -> 17.2 mm
- net N$6: track 52.7 -> 50.8 mm
- net N$58: track 68.5 -> 67.1 mm
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
Commit message: update
Parts:
- added C10: 0.1, rcl:C0805
- added LED1: PWR ON, led:CHIPLED_1206
- added PAD1: LCD9, wirepad:SMD1,27-2,54
- added PAD2: LCD10, wirepad:SMD1,27-2,54
- added R8: 220, rcl:R0805
- added SV8: LCD, con-lstb:MA10-1
Connections:
- new net N$63: IC1.42, SV5.5, SV8.1
- new net N$66: PAD1.1, SV8.9
- new net N$67: PAD2.1, SV8.10
- net N$33: now also SV8.6
- net N$34: now also SV8.4
- net N$35: now also SV8.5
- net N$36: now also SV8.3
- net N$37: now also LED1.A, R8.2; no longer IC1.42, SV5.5
- net N$38: now also SV8.2
- net VDD: now also C10.1, R8.1, SV8.7
- net VSS: now also C10.2, LED1.C, SV8.8
Routing:
- net VDD: track 149.8 -> 221.5 mm, vias 2 -> 1
- net N$63: track 0.00 -> 46.6 mm, vias 0 -> 1
- net N$36: track 10.7 -> 52.2 mm, vias 1 -> 0
- net N$33: track 19.2 -> 59.9 mm
- net GND: track 103.6 -> 136.5 mm, vias 1 -> 2
- net VSS: track 300.5 -> 329.3 mm, vias 0 -> 1
- net N$34: track 17.2 -> 45.5 mm
- net N$38: track 12.2 -> 39.9 mm, vias 0 -> 3
- net N$35: track 11.7 -> 38.1 mm
- net N$19: track 83.1 -> 59.1 mm, vias 1 -> 3
- net N$1: track 53.4 -> 32.7 mm
- net N$4: track 56.5 -> 36.9 mm, vias 1 -> 2
- net VCC: track 132.8 -> 150.0 mm, vias 1 -> 2
- net N$23: track 62.6 -> 49.6 mm
- net N$30: track 9.27 -> 20.4 mm, vias 1 -> 0
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
Commit message: update
Parts:
- added SV9: USBH, con-lstb:MA03-1
- added X6: MINI-USB-UX60A-MB-5ST, con-hirose:UX60A-MB-5ST
- moved K1 17.0 mm to (77.5, 64.8)
Connections:
- new net N$59: SV9.3, X6.2
- new net N$61: SV9.2, X6.3
- new net N$64: SV9.1, X6.4
- net N$60: now also X6.1
- net VSS: now also X6.5
Routing:
- net N$60: track 30.1 -> 104.3 mm, vias 0 -> 2
- net N$4: track 36.9 -> 84.1 mm, vias 2 -> 0
- net N$5: track 34.4 -> 64.8 mm
- net VDD: track 221.5 -> 243.9 mm
- net N$58: track 67.1 -> 88.1 mm, vias 3 -> 8
- net VCC: track 150.0 -> 130.4 mm, vias 2 -> 4
- net VSS: track 329.3 -> 348.4 mm, vias 1 -> 2
- net N$64: track 0.00 -> 18.1 mm, vias 0 -> 1
- net N$61: track 0.00 -> 16.3 mm, vias 0 -> 1
- net N$59: track 0.00 -> 15.2 mm
- net N$56: track 22.4 -> 7.42 mm
- net N$8: track 31.1 -> 45.2 mm
- net N$57: track 27.2 -> 13.2 mm
- net N$36: track 52.2 -> 39.4 mm
- net N$10: track 24.4 -> 37.1 mm, vias 1 -> 0
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
Commit message: update and fix switch pins on pcb
Parts:
- renumbered X3 to POWER, X4 to GLORY
Connections:
- removed net N$24: S1.2, SV1.5
- new net N$65: S1.3, SV1.5
- net N$23: now also S1.6; no longer S1.5
- net N$6: now also S1.5; no longer S1.6
- net N$7: now also S1.2; no longer S1.3
Routing:
- net N$24: track 48.1 -> 0.00 mm
- net N$4: track 84.1 -> 42.2 mm, vias 0 -> 1
- net N$65: track 0.00 -> 39.7 mm, vias 0 -> 1
- net VDD: track 243.9 -> 205.7 mm, vias 1 -> 2
- net N$5: track 64.8 -> 32.7 mm
- net N$58: track 88.1 -> 72.7 mm, vias 8 -> 5
- net N$8: track 45.2 -> 30.3 mm
- net N$6: track 52.4 -> 66.5 mm
- net VSS: track 348.4 -> 336.3 mm, vias 2 -> 0
- net VCC: track 130.4 -> 141.1 mm, vias 4 -> 2
- net N$2: track 54.2 -> 63.6 mm, vias 2 -> 0
- net N$20: track 93.6 -> 102.2 mm, vias 4 -> 2
- net N$23: track 45.7 -> 52.7 mm, vias 1 -> 0
- net N$17: track 25.6 -> 32.2 mm
- net N$63: track 40.4 -> 46.4 mm, vias 3 -> 2
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
Commit message: update
Parts:
- removed S1: ICD/SERIAL, JS202011SCQN:JS202011SCQN
- added ICSP/SERIAL: JS202011SCQN, JS202011SCQN_fixed:SW_JS202011SCQN
Connections:
- net N$20: now also ICSP/SERIAL.1, XT1.2; no longer R6.2, S1.1
- net N$22: now also ICSP/SERIAL.4; no longer S1.4
- net N$23: now also ICSP/SERIAL.6; no longer S1.6
- net N$6: now also ICSP/SERIAL.5; no longer S1.5
- net N$65: now also ICSP/SERIAL.3; no longer S1.3
- net N$7: now also ICSP/SERIAL.2; no longer S1.2
- net VDD: now also R6.2
- net VSS: no longer XT1.2
Routing:
- net VDD: track 205.7 -> 252.6 mm, vias 2 -> 1
- net N$4: track 42.2 -> 84.8 mm, vias 1 -> 0
- net N$2: track 63.6 -> 40.2 mm, vias 0 -> 2
- net N$7: track 58.2 -> 81.0 mm
- net N$22: track 30.8 -> 49.2 mm
- net N$63: track 46.4 -> 63.9 mm
- net N$10: track 36.8 -> 23.3 mm, vias 0 -> 1
- net N$51: track 15.3 -> 28.4 mm, vias 1 -> 0
- net N$23: track 52.7 -> 39.7 mm, vias 0 -> 1
- net N$30: track 9.27 -> 20.4 mm, vias 1 -> 0
- net N$36: track 39.4 -> 49.7 mm, vias 0 -> 2
- net N$16: track 51.7 -> 41.7 mm
- net N$32: track 30.2 -> 20.4 mm
- net N$20: track 102.2 -> 111.5 mm, vias 2 -> 0
- net N$58: track 72.7 -> 81.4 mm, vias 5 -> 8
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Other:
- board text added: "FGB@MCHP 1.1"
- board text removed: "FGB@MCHP 1.0"

Commit message: update
Parts:
- moved R7 19.4 mm to (26.7, 69.8)
- moved C2 16.1 mm to (21.6, 69.8)
- moved LED2 13.7 mm to (31.8, 73.7)
- moved C5 12.5 mm to (25.4, 73.7)
- moved C1 12.5 mm to (31.8, 69.8)
- moved SV2 11.4 mm to (45.7, 59.7), turned to 0 degrees
- moved L1 6.35 mm to (45.7, 43.2), turned to 180 degrees
- moved SV6 6.35 mm to (45.7, 68.6), turned to 0 degrees
- moved SV7 5.24 mm to (45.7, 50.8), turned to 0 degrees
- moved K1 2.54 mm to (80.0, 64.8)
- moved OS1 1.27 mm to (80.0, 39.4)
- moved R3 1.27 mm to (52.1, 34.3)
- moved R5 1.27 mm to (35.6, 44.5), turned to 0 degrees
- turned SV4 to 0 degrees
Routing:
- net VDD: track 252.6 -> 207.2 mm, vias 1 -> 2
- net GND: track 130.3 -> 173.8 mm, vias 3 -> 1
- net N$58: track 81.4 -> 123.8 mm, vias 8 -> 6
- net N$2: track 40.2 -> 76.7 mm, vias 2 -> 0
- net VCC: track 148.7 -> 116.7 mm
- net N$4: track 84.8 -> 59.0 mm, vias 0 -> 2
- net N$41: track 16.0 -> 40.2 mm, vias 2 -> 0
- net N$47: track 13.5 -> 37.3 mm, vias 0 -> 1
- net N$63: track 63.9 -> 41.4 mm
- net N$10: track 23.3 -> 44.8 mm, vias 1 -> 4
- net N$5: track 32.9 -> 54.1 mm
- net N$51: track 28.4 -> 48.6 mm, vias 0 -> 2
- net N$7: track 81.0 -> 63.3 mm, vias 2 -> 4
- net N$52: track 50.4 -> 66.7 mm
- net N$48: track 6.05 -> 22.0 mm, vias 0 -> 3
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Other:
- board text added: "FGB@MCHP 1.2"
- board text removed: "FGB@MCHP 1.1"

Commit message: update
Parts:
- removed D2: 1N4148, diode:SOD-123_MINI-SMA
- added C11: 10uf, rcl:C0805
- added R9: 197, rcl:R0805
- R3: value 220 -> 197
- moved K1 1.80 mm to (78.7, 63.5)
- renumbered ICSP/SERIAL to SERIAL/ICSP
Connections:
- net N$2: now also R9.1; no longer D2.C
- net N$58: now also C11.1
- net N$62: now also R9.2; no longer D2.A
- net VSS: now also C11.2
Routing:
- net N$21: track 81.4 -> 130.4 mm, vias 3 -> 2
- net N$51: track 48.6 -> 22.4 mm, vias 2 -> 1
- net VDD: track 207.2 -> 232.3 mm
- net N$10: track 44.8 -> 66.5 mm, vias 4 -> 3
- net N$5: track 54.1 -> 34.2 mm, vias 2 -> 3
- net GND: track 173.8 -> 159.5 mm, vias 1 -> 2
- net N$32: track 10.5 -> 24.5 mm
- net N$60: track 101.8 -> 114.8 mm, vias 3 -> 2
- net N$36: track 40.4 -> 52.8 mm, vias 2 -> 3
- net N$44: track 21.3 -> 33.6 mm
- net N$2: track 76.7 -> 65.3 mm, vias 0 -> 2
- net N$38: track 43.2 -> 54.5 mm
- net N$59: track 25.7 -> 15.1 mm
- net N$17: track 31.1 -> 20.6 mm, vias 0 -> 1
- net N$34: track 52.6 -> 42.5 mm, vias 1 -> 2
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Other:
- board text added: "FGB@MCHP 1.3"
- board text removed: "FGB@MCHP 1.2"

Commit message: up
Routing:
- net VCC: track 111.6 -> 112.6 mm
Changed lines of the file:
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@@
 <?xml version="1.0" encoding="utf-8"?>
 <!DOCTYPE eagle SYSTEM "eagle.dtd">
-<eagle version="9.4.1">
+<eagle version="9.5.0">
 <drawing>
 <settings>
@@
 <contactref element="C8" pad="1"/>
 <contactref element="C9" pad="1"/>
-<wire x1="25.2984" y1="51.816" x2="21.6408" y2="51.816" width="0.1524" layer="1"/>
-<wire x1="21.6408" y1="51.816" x2="21.59" y2="51.75" width="0.1524" layer="1"/>
-<wire x1="25.2984" y1="51.816" x2="25.4" y2="51.75" width="0.1524" layer="1"/>
+<wire x1="23.34336875" y1="53.086" x2="22.618315625" y2="53.086" width="0.1524" layer="1"/>
+<wire x1="22.618315625" y1="53.086" x2="21.59" y2="51.75" width="0.1524" layer="1"/>
+<wire x1="23.34336875" y1="53.086" x2="25.4" y2="51.75" width="0.1524" layer="1"/>
 <wire x1="19.6596" y1="57.7596" x2="19.2024" y2="57.7596" width="0.1524" layer="1"/>
 <wire x1="20.4216" y1="56.9976" x2="19.6596" y2="57.7596" width="0.1524" layer="1"/>
