File: touch_board/touch_board.brd (EAGLE design)
At the start: 81 x 62.2 mm, 52 parts, among them IC1 PIC18F47K42-I_PT, IC2 MAX203EEWP, K1 G6K-2P, X1 RS-232-1, X2 RS-232-2, X5 Relay conn, X6 MINI-USB-UX60A-MB-5ST

Commit message: up
Parts:
- added TP1: TPB1,27, testpad:B1,27
Connections:
- net VSS: now also TP1.TP
Routing:
- net VSS: track 344.2 -> 352.1 mm
Changed lines of the file:
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@@
 <attribute name="VALUE" x="88.9" y="26.67" size="1.27" layer="27"/>
+</element>
+<element name="TP1" library="testpad" library_urn="urn:adsk.eagle:library:385" package="B1,27" package3d_urn="urn:adsk.eagle:package:27944/2" value="TPB1,27" x="69.85" y="77.47" smashed="yes">
+<attribute name="NAME" x="69.215" y="78.486" size="1.27" layer="25" ratio="10"/>
+<attribute name="POPULARITY" value="19" x="69.85" y="77.47" size="1.778" layer="27" display="off"/>
+<attribute name="TP_SIGNAL_NAME" value="" x="69.85" y="77.47" size="1.778" layer="27" display="off"/>
+<attribute name="VALUE" x="69.215" y="76.708" size="0.0254" layer="27"/>
 </element>
 </elements>
@@
 <via x="61.1124" y="71.3232" extent="1-16" drill="0.35"/>
 <via x="35.9664" y="72.8472" extent="1-16" drill="0.35"/>
+<contactref element="TP1" pad="TP"/>
+<wire x1="72.5424" y1="77.4192" x2="69.9516" y2="77.4192" width="0.1524" layer="1"/>
+<wire x1="76.2" y1="73.7616" x2="72.5424" y2="77.4192" width="0.1524" layer="1"/>
+<wire x1="69.9516" y1="77.4192" x2="69.85" y2="77.47" width="0.1524" layer="1"/>
 </signal>
 <signal name="VDD">
@@
 <mfgpreviewcolor name="substratecolor" color="0xFF786E46"/>
 </mfgpreviewcolors>
-<errors>
-</errors>
 </board>
 </drawing>

Commit message: up
Parts:
- added D2: 5.6, diode:SMB
- moved D1 1.80 mm to (49.5, 30.5)
Connections:
- net N$60: now also D2.C
- net VSS: now also D2.A
Routing:
- net VSS: track 352.1 -> 371.2 mm
- net N$60: track 114.8 -> 118.5 mm
Other:
- board text added: "FGB@MCHP 1.4"
- board text removed: "FGB@MCHP 1.3"
Changed lines of the file:
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@@
 <?xml version="1.0" encoding="utf-8"?>
 <!DOCTYPE eagle SYSTEM "eagle.dtd">
-<eagle version="9.5.0">
+<eagle version="9.6.2">
 <drawing>
 <settings>
@@
 <layers>
 <layer number="1" name="Top" color="4" fill="1" visible="yes" active="yes"/>
+<layer number="2" name="Route2" color="1" fill="3" visible="no" active="no"/>
+<layer number="3" name="Route3" color="4" fill="3" visible="no" active="no"/>
+<layer number="4" name="Route4" color="1" fill="4" visible="no" active="no"/>
+<layer number="5" name="Route5" color="4" fill="4" visible="no" active="no"/>
+<layer number="6" name="Route6" color="1" fill="8" visible="no" active="no"/>
+<layer number="7" name="Route7" color="4" fill="8" visible="no" active="no"/>
+<layer number="8" name="Route8" color="1" fill="2" visible="no" active="no"/>
+<layer number="9" name="Route9" color="4" fill="2" visible="no" active="no"/>
+<layer number="10" name="Route10" color="1" fill="7" visible="no" active="no"/>
+<layer number="11" name="Route11" color="4" fill="7" visible="no" active="no"/>
+<layer number="12" name="Route12" color="1" fill="5" visible="no" active="no"/>
+<layer number="13" name="Route13" color="4" fill="5" visible="no" active="no"/>
+<layer number="14" name="Route14" color="1" fill="6" visible="no" active="no"/>
+<layer number="15" name="Route15" color="4" fill="6" visible="no" active="no"/>
 <layer number="16" name="Bottom" color="1" fill="1" visible="yes" active="yes"/>
 <layer number="17" name="Pads" color="2" fill="1" visible="yes" active="yes"/>
@@
 <hole x="93.98" y="77.47" drill="2.5"/>
 <hole x="17.78" y="77.47" drill="2.5"/>
-<text x="22.86" y="76.2" size="1.778" layer="1" font="vector" ratio="13">FGB@MCHP 1.3</text>
+<text x="22.86" y="76.2" size="1.778" layer="1" font="vector" ratio="13">FGB@MCHP 1.4</text>
 <text x="93.98" y="24.13" size="1.6764" layer="1" font="vector" ratio="14" rot="R90">These are the controllers you are looking for!</text>
 </plain>
@@
 <attribute name="VALUE" x="45.44" y="31.69" size="1.27" layer="27"/>
 </element>
-<element name="D1" library="diode" library_urn="urn:adsk.eagle:library:210" package="ZDIO-7.5" package3d_urn="urn:adsk.eagle:package:43411/1" value="5.6V" x="50.8" y="29.21" smashed="yes" rot="R180">
-<attribute name="NAME" x="54.5592" y="28.7782" size="1.27" layer="25" ratio="10" rot="R180"/>
-<attribute name="VALUE" x="50.8" y="28.448" size="1.27" layer="27" ratio="10" rot="R180"/>
+<element name="D1" library="diode" library_urn="urn:adsk.eagle:library:210" package="ZDIO-7.5" package3d_urn="urn:adsk.eagle:package:43411/1" value="5.6V" x="49.53" y="30.48" smashed="yes" rot="R180">
+<attribute name="NAME" x="53.2892" y="30.0482" size="1.27" layer="25" ratio="10" rot="R180"/>
+<attribute name="POPULARITY" value="6" x="49.53" y="30.48" size="1.778" layer="27" rot="R180" display="off"/>
+<attribute name="VALUE" x="49.53" y="29.718" size="1.27" layer="27" ratio="10" rot="R180"/>
 </element>
 <element name="S3" library="SamacSys_Parts" package="B3W-9_1-LED" value="RESETSW" x="38.1" y="35.56" smashed="yes">
@@
 <attribute name="TP_SIGNAL_NAME" value="" x="69.85" y="77.47" size="1.778" layer="27" display="off"/>
 <attribute name="VALUE" x="69.215" y="76.708" size="0.0254" layer="27"/>
+</element>
+<element name="D2" library="diode" library_urn="urn:adsk.eagle:library:210" package="SMB" package3d_urn="urn:adsk.eagle:package:43404/2" value="5.6" x="49.53" y="26.67" smashed="yes" rot="R180">
+<attribute name="NAME" x="51.689" y="24.511" size="1.27" layer="25" rot="R180"/>
+<attribute name="POPULARITY" value="3" x="49.53" y="26.67" size="1.778" layer="27" rot="R180" display="off"/>
+<attribute name="VALUE" x="51.689" y="30.099" size="1.27" layer="27" rot="R180"/>
 </element>
 </elements>
@@
 <wire x1="43.2816" y1="24.0792" x2="44.5008" y2="22.86" width="0.1524" layer="1"/>
 <wire x1="43.2816" y1="24.0792" x2="43.18" y2="24.13" width="0.1524" layer="1"/>
-<wire x1="46.9392" y1="23.1648" x2="46.9392" y2="29.1084" width="0.1524" layer="1"/>
 <wire x1="46.6344" y1="22.86" x2="46.9392" y2="23.1648" width="0.1524" layer="1"/>
-<wire x1="46.9392" y1="29.1084" x2="46.99" y2="29.21" width="0.1524" layer="1"/>
 <wire x1="46.6344" y1="22.86" x2="46.51" y2="22.86" width="0.1524" layer="1"/>
 <wire x1="38.5572" y1="24.2316" x2="36.8808" y2="24.2316" width="0.1524" layer="1"/>
@@
 <wire x1="46.9392" y1="23.1648" x2="50.292" y2="19.812" width="0.1524" layer="1"/>
 <wire x1="58.3692" y1="21.4884" x2="58.42" y2="21.59" width="0.1524" layer="1"/>
-<wire x1="46.9392" y1="23.1648" x2="46.51" y2="22.86" width="0.1524" layer="1"/>
 <wire x1="53.34" y1="49.53" x2="57.762" y2="49.53" width="0.1524" layer="1"/>
 <wire x1="50.8" y1="52.07" x2="53.34" y2="49.53" width="0.1524" layer="1"/>
@@
 <wire x1="50.9016" y1="51.9684" x2="50.8" y2="52.07" width="0.1524" layer="16"/>
 <wire x1="49.53" y1="39.4716" x2="49.53" y2="39.37" width="0.1524" layer="16"/>
-<wire x1="46.9392" y1="30.3276" x2="46.9392" y2="29.2608" width="0.1524" layer="16"/>
-<wire x1="41.7576" y1="35.5092" x2="46.9392" y2="30.3276" width="0.1524" layer="16"/>
-<wire x1="46.9392" y1="29.2608" x2="46.99" y2="29.21" width="0.1524" layer="16"/>
-<wire x1="41.7576" y1="35.5092" x2="41.7" y2="35.56" width="0.1524" layer="16"/>
 <wire x1="69.7992" y1="40.2336" x2="69.7992" y2="38.1" width="0.1524" layer="16"/>
 <wire x1="62.0268" y1="48.006" x2="69.7992" y2="40.2336" width="0.1524" layer="16"/>
@@
 <wire x1="76.2" y1="73.7616" x2="72.5424" y2="77.4192" width="0.1524" layer="1"/>
 <wire x1="69.9516" y1="77.4192" x2="69.85" y2="77.47" width="0.1524" layer="1"/>
+<contactref element="D2" pad="A"/>
+<wire x1="47.244" y1="23.4696" x2="47.244" y2="26.67" width="0.1524" layer="1"/>
+<wire x1="46.9392" y1="23.1648" x2="47.244" y2="23.4696" width="0.1524" layer="1"/>
+<wire x1="46.9392" y1="23.1648" x2="46.51" y2="22.86" width="0.1524" layer="1"/>
+<wire x1="47.244" y1="26.67" x2="47.33" y2="26.67" width="0.1524" layer="1"/>
+<wire x1="41.7576" y1="35.5092" x2="45.72" y2="31.5468" width="0.1524" layer="16"/>
+<wire x1="41.7576" y1="35.5092" x2="41.7" y2="35.56" width="0.1524" layer="16"/>
+<wire x1="53.6448" y1="31.5468" x2="45.72" y2="31.5468" width="0.1524" layer="16"/>
+<wire x1="54.2544" y1="30.9372" x2="53.6448" y2="31.5468" width="0.1524" layer="16"/>
+<wire x1="54.2544" y1="30.0228" x2="54.2544" y2="30.9372" width="0.1524" layer="16"/>
+<wire x1="48.4632" y1="24.2316" x2="54.2544" y2="30.0228" width="0.1524" layer="16"/>
+<wire x1="43.2816" y1="24.2316" x2="48.4632" y2="24.2316" width="0.1524" layer="16"/>
+<wire x1="43.2816" y1="24.2316" x2="43.18" y2="24.13" width="0.1524" layer="16"/>
+<wire x1="45.72" y1="31.5468" x2="45.72" y2="30.48" width="0.1524" layer="16"/>
 </signal>
 <signal name="VDD">
@@
 <contactref element="R9" pad="1"/>
 <wire x1="53.0352" y1="33.528" x2="53.0352" y2="34.29" width="0.1524" layer="1"/>
-<wire x1="59.8932" y1="26.67" x2="55.3212" y2="31.242" width="0.1524" layer="1"/>
-<wire x1="55.3212" y1="31.242" x2="53.0352" y2="33.528" width="0.1524" layer="1"/>
+<wire x1="59.8932" y1="26.67" x2="57.3024" y2="29.2608" width="0.1524" layer="1"/>
+<wire x1="57.3024" y1="29.2608" x2="53.0352" y2="33.528" width="0.1524" layer="1"/>
 <wire x1="59.8932" y1="26.67" x2="60.01" y2="26.67" width="0.1524" layer="1"/>
-<wire x1="49.3776" y1="21.6408" x2="53.34" y2="21.6408" width="0.1524" layer="1"/>
-<wire x1="48.9204" y1="22.098" x2="49.3776" y2="21.6408" width="0.1524" layer="1"/>
-<wire x1="48.9204" y1="24.8412" x2="48.9204" y2="22.098" width="0.1524" layer="1"/>
-<wire x1="55.3212" y1="31.242" x2="48.9204" y2="24.8412" width="0.1524" layer="1"/>
-<wire x1="53.34" y1="21.6408" x2="53.34" y2="21.59" width="0.1524" layer="1"/>
 <wire x1="43.1292" y1="59.8932" x2="43.1292" y2="60.96" width="0.1524" layer="1"/>
 <wire x1="41.7576" y1="58.5216" x2="43.1292" y2="59.8932" width="0.1524" layer="1"/>
@@
 <via x="38.4048" y="48.768" extent="1-16" drill="0.35"/>
 <via x="52.2732" y="36.8808" extent="1-16" drill="0.35"/>
+<wire x1="49.3776" y1="21.6408" x2="53.34" y2="21.6408" width="0.1524" layer="1"/>
+<wire x1="48.9204" y1="22.098" x2="49.3776" y2="21.6408" width="0.1524" layer="1"/>
+<wire x1="48.9204" y1="23.622" x2="48.9204" y2="22.098" width="0.1524" layer="1"/>
+<wire x1="50.4444" y1="25.146" x2="48.9204" y2="23.622" width="0.1524" layer="1"/>
+<wire x1="53.1876" y1="25.146" x2="50.4444" y2="25.146" width="0.1524" layer="1"/>
+<wire x1="57.3024" y1="29.2608" x2="53.1876" y2="25.146" width="0.1524" layer="1"/>
+<wire x1="53.34" y1="21.6408" x2="53.34" y2="21.59" width="0.1524" layer="1"/>
 </signal>
 <signal name="N$3">
@@
 <contactref element="D1" pad="C"/>
 <contactref element="X6" pad="1"/>
-<wire x1="48.1584" y1="29.1084" x2="54.5592" y2="29.1084" width="0.1524" layer="16"/>
-<wire x1="44.958" y1="25.908" x2="48.1584" y2="29.1084" width="0.1524" layer="16"/>
 <wire x1="42.3672" y1="25.908" x2="44.958" y2="25.908" width="0.1524" layer="16"/>
 <wire x1="40.6908" y1="24.2316" x2="42.3672" y2="25.908" width="0.1524" layer="16"/>
-<wire x1="54.5592" y1="29.1084" x2="54.61" y2="29.21" width="0.1524" layer="16"/>
 <wire x1="40.6908" y1="24.2316" x2="40.64" y2="24.13" width="0.1524" layer="16"/>
 <wire x1="41.91" y1="34.29" x2="45.59" y2="34.29" width="0.1524" layer="1"/>
@@
 <via x="34.8996" y="65.532" extent="1-16" drill="0.35"/>
 <via x="33.6804" y="42.0624" extent="1-16" drill="0.35"/>
+<contactref element="D2" pad="C"/>
+<wire x1="51.816" y1="28.956" x2="51.816" y2="26.67" width="0.1524" layer="1"/>
+<wire x1="51.816" y1="26.67" x2="51.73" y2="26.67" width="0.1524" layer="1"/>
+<wire x1="44.958" y1="25.908" x2="49.53" y2="30.48" width="0.1524" layer="16"/>
+<wire x1="53.34" y1="30.48" x2="51.816" y2="28.956" width="0.1524" layer="1"/>
+<wire x1="49.53" y1="30.48" x2="53.34" y2="30.48" width="0.1524" layer="16"/>
 </signal>
 <signal name="N$62">
