File: touch_board/touch_board.sch (EAGLE design)
At the start: 10 parts, among them IC1 PIC18F47K42-I_PT

Commit message: update
Parts:
- added C7: 0.1, rcl:C-USC0805
- added LED1: RUN, led:LEDCHIPLED_1206
- added LED2: MODE, led:LEDCHIPLED_1206
- added R3, R5, R7: 220, rcl:R-US_R0805
- added R4: 10k, rcl:R-US_R0805
- added SV1: ICSP, con-lstb:MA06-1
- added SV2: IO1, con-lstb:MA05-2
- added SV3: RESET, con-lstb:MA03-1
Connections:
- new net N$10: IC1.RD1, R7.2
- new net N$11: LED2.A, R7.1
- new net N$2: C7.1, R3.1, R4.1, SV1.1, SV2.4, SV3.1
- new net N$3: IC1.VPP/!MCLR!/RE3, R3.2
- new net N$4: IC1.RE0, R5.2, SV2.1
- new net N$5: IC1.RE1, SV2.2
- new net N$6: IC1.ICSPDAT/RB7, SV1.4
- new net N$7: IC1.ICSPCLK/RB6, SV1.5
- new net N$8: IC1.RE2, SV2.3
- new net N$9: LED1.A, R5.1
- net VDD: now also R4.2, SV1.2, SV2.9
- net VSS: now also C7.2, LED1.C, LED2.C, SV1.3, SV2.10, SV3.2, SV3.3
Other:
- moved on the sheet: C3

Commit message: update
Parts:
- added C8: 0.1, rcl:C-USC0805
- added C9: 10uf, rcl:C-USC0805
- added IC2: MAX203EEWP, maxim-10:MAX203EEWP
- added JMP1, JMP2: 0R-JUMPA, jump-0r-smd:0R-JUMPA
- added X1: RS-232-1, con-molex:22-23-2041
- added X2: RS-232-2, con-molex:22-23-2041
- added X3: POWER, con-molex:22-23-2021
- added X4: 22-23-2041, con-molex:22-23-2041
Connections:
- new net N$12: IC2G$1.C2-/1, IC2G$1.C2-/2
- new net N$13: IC2G$1.V-/1, IC2G$1.V-/2
- new net N$14: IC2G$1.C2+/1, IC2G$1.C2+/2
- new net N$15: IC2G$1.T1OUT, X1-2.S
- new net N$16: IC2G$1.T2OUT, X2-2.S
- new net N$17: IC2G$1.R1IN, X1-3.S
- new net N$18: IC2G$1.R2IN, X2-3.S
- new net N$19: IC1.RC6, IC2G$1.T1IN
- new net N$20: IC2G$1.T2IN, X4-1.S
- new net N$21: IC1.RC7, IC2G$1.R1OUT
- new net N$22: IC2G$1.R2OUT, X4-3.S
- net GND: now also C8.2, C9.2, JMP1-0R.1, JMP1-0R.3, JMP2-0R.1, JMP2-0R.3, X1-1.S, X2-1.S
- net N$6: now also X4-4.S
- net N$7: now also X4-2.S
- net VCC: now also C8.1, C9.1, X1-4.S, X2-4.S
- net VDD: now also X3-1.S
- net VSS: now also JMP1-0R.2, JMP2-0R.2, X3-2.S

Commit message: update
Parts:
- removed X4: 22-23-2041, con-molex:22-23-2041
- added R6: 220, rcl:R-US_R0805
- added S1: ICD/SERIAL, JS202011SCQN:JS202011SCQN
- added S2: RESET_PB, switch-omron:10-XX
- added SV4, SV5, SV6, SV7: IO1, con-lstb:MA05-2
- added XT1: HFBR-1521, fiber-optic-hp:HFBR-1521
Connections:
- new net N$23: S1.5, SV1.4
- new net N$24: S1.2, SV1.5
- new net N$25: R6.1, XT1.A
- new net N$26: IC1.RA0, SV4.1
- new net N$27: IC1.RA1, SV4.2
- new net N$28: IC1.RA2, SV4.3
- new net N$29: IC1.RA3, SV4.4
- new net N$30: IC1.RA4, SV4.5
- new net N$31: IC1.RA6, SV4.7
- new net N$32: IC1.RA5, SV4.6
- new net N$33: IC1.RC0, SV5.1
- new net N$34: IC1.RC1, SV5.2
- new net N$35: IC1.RC2, SV5.3
- new net N$36: IC1.RC3, SV5.4
- new net N$37: IC1.RC4, SV5.5
- new net N$38: IC1.RC5, SV5.6
- new net N$39: IC1.RD0, SV6.1
- new net N$40: IC1.RD2, SV6.3
- new net N$41: IC1.RD3, SV6.4
- new net N$42: IC1.RD4, SV6.5
- new net N$43: IC1.RD5, SV6.6
- new net N$44: IC1.RD6, SV6.7
- new net N$45: IC1.RD7, SV6.8
- new net N$46: IC1.RB0, SV7.1
- new net N$47: IC1.RB1, SV7.2
- new net N$48: IC1.RB2, SV7.3
- new net N$49: IC1.RB3, SV7.4
- new net N$50: IC1.RB4, SV7.5
- new net N$51: IC1.RB5, SV7.6
- net N$1: now also SV4.8
- net N$10: now also SV6.2
- net N$19: now also SV5.7
- net N$2: now also S2.S1
- net N$20: now also R6.2, S1.1; no longer X4-1.S
- net N$21: now also SV5.8
- net N$22: now also S1.4; no longer X4-3.S
- net N$6: now also S1.6; no longer SV1.4, X4-4.S
- net N$7: now also S1.3; no longer SV1.5, X4-2.S
- net VDD: now also SV4.9, SV5.9, SV6.9, SV7.9
- net VSS: now also S2.P1, SV4.10, SV5.10, SV6.10, SV7.10, XT1.C

Commit message: update
Connections:
- net N$6: now also SV7.8
- net N$7: now also SV7.7
Changed lines of the file:
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@@
 <wire x1="73.66" y1="-12.7" x2="60.96" y2="-12.7" width="0.1524" layer="91"/>
 <junction x="73.66" y="-2.54"/>
-<wire x1="60.96" y1="-12.7" x2="60.96" y2="-40.64" width="0.1524" layer="91"/>
 <pinref part="S1" gate="G$1" pin="6"/>
+<wire x1="60.96" y1="-15.24" x2="60.96" y2="-40.64" width="0.1524" layer="91"/>
 <wire x1="60.96" y1="-40.64" x2="45.72" y2="-40.64" width="0.1524" layer="91"/>
 <junction x="45.72" y="-40.64"/>
+<pinref part="SV7" gate="G$1" pin="8"/>
+<wire x1="30.48" y1="12.7" x2="2.54" y2="12.7" width="0.1524" layer="91"/>
+<wire x1="2.54" y1="12.7" x2="2.54" y2="-12.7" width="0.1524" layer="91"/>
+<wire x1="2.54" y1="-12.7" x2="60.96" y2="-12.7" width="0.1524" layer="91"/>
+<wire x1="60.96" y1="-12.7" x2="60.96" y2="-15.24" width="0.1524" layer="91"/>
+<junction x="60.96" y="-12.7"/>
+<junction x="30.48" y="12.7"/>
 </segment>
 </net>
@@
 <pinref part="S1" gate="G$1" pin="3"/>
 <junction x="25.4" y="-40.64"/>
+<pinref part="SV7" gate="G$1" pin="7"/>
+<wire x1="45.72" y1="12.7" x2="55.88" y2="12.7" width="0.1524" layer="91"/>
+<wire x1="55.88" y1="12.7" x2="55.88" y2="20.32" width="0.1524" layer="91"/>
+<wire x1="55.88" y1="20.32" x2="17.78" y2="20.32" width="0.1524" layer="91"/>
+<wire x1="17.78" y1="20.32" x2="17.78" y2="-10.16" width="0.1524" layer="91"/>
+<wire x1="17.78" y1="-10.16" x2="55.88" y2="-10.16" width="0.1524" layer="91"/>
+<junction x="45.72" y="12.7"/>
+<junction x="55.88" y="-10.16"/>
 </segment>
 </net>

Commit message: update
Parts:
- added K1: G6K-2P, relay:G6K-2P
- added L1, L2: 1000, inductor-neosid:SM-1206
- added X4: GLORY, con-molex:22-23-2021
- added X5: Relay conn, con-phoenix-254:MPT8
Connections:
- new net N$52: IC1.RD0, K11.+, SV6.1, X5-1.1
- new net N$53: K12.P, X5-3.1
- new net N$54: K12.S, X5-4.1
- new net N$55: K13.S, X5-5.1
- new net N$56: K13.P, X5-6.1
- new net N$57: K13.O, X5-7.1
- new net N$58: C1.1, C2.1, C3.1, C5.1, IC1.VDD_1, IC1.VDD_2, L1.1, L2.2, R2.1
- net N$39: now also K12.O, X5-2.1; no longer IC1.RD0, SV6.1
- net VDD: now also L1.2, L2.1, X4-1.S; no longer C1.1, C2.1, C3.1, C5.1, IC1.VDD_1, IC1.VDD_2, R2.1
- net VSS: now also K11.-, X4-2.S, X5-8.1
Other:
- moved on the sheet: C5

Commit message: update
Parts:
- added D1: 5.6V, diode:ZENER-DIODEZD-7.5
- added F1: 1206L050, polyfuse-smd_10:1206L050
Connections:
- new net N$60: D1.C, F1.1, X3-1.S, X4-1.S
- net VDD: now also F1.2; no longer X3-1.S, X4-1.S
- net VSS: now also D1.A
Changed lines of the file:
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@@
 <layer number="97" name="Info" color="7" fill="1" visible="yes" active="yes"/>
 <layer number="98" name="Guide" color="6" fill="1" visible="yes" active="yes"/>
+<layer number="99" name="SpiceOrder" color="5" fill="1" visible="yes" active="yes"/>
 <layer number="250" name="Descript" color="3" fill="1" visible="no" active="no"/>
 <layer number="251" name="SMDround" color="12" fill="11" visible="no" active="no"/>
@@
 <part name="X3" library="con-molex" library_urn="urn:adsk.eagle:library:165" deviceset="22-23-2021" device="" package3d_urn="urn:adsk.eagle:package:8078633/1" value="POWER"/>
 <part name="VSS13" library="supply1" library_urn="urn:adsk.eagle:library:371" deviceset="VSS" device=""/>
-<part name="VDD8" library="supply1" library_urn="urn:adsk.eagle:library:371" deviceset="VDD" device=""/>
 <part name="C8" library="rcl" library_urn="urn:adsk.eagle:library:334" deviceset="C-US" device="C0805" package3d_urn="urn:adsk.eagle:package:23617/2" value="0.1"/>
 <part name="C9" library="rcl" library_urn="urn:adsk.eagle:library:334" deviceset="C-US" device="C0805" package3d_urn="urn:adsk.eagle:package:23617/2" value="10uf"/>
@@
 <part name="S2" library="switch-omron" library_urn="urn:adsk.eagle:library:377" deviceset="10-XX" device="" package3d_urn="urn:adsk.eagle:package:27496/1" value="RESET_PB"/>
 <part name="X4" library="con-molex" library_urn="urn:adsk.eagle:library:165" deviceset="22-23-2021" device="" package3d_urn="urn:adsk.eagle:package:8078633/1" value="GLORY"/>
-<part name="VDD13" library="supply1" library_urn="urn:adsk.eagle:library:371" deviceset="VDD" device=""/>
 <part name="VSS20" library="supply1" library_urn="urn:adsk.eagle:library:371" deviceset="VSS" device=""/>
 <part name="K1" library="relay" library_urn="urn:adsk.eagle:library:339" deviceset="G6K" device="-2P" package3d_urn="urn:adsk.eagle:package:24346/1"/>
@@
 <part name="VDD14" library="supply1" library_urn="urn:adsk.eagle:library:371" deviceset="VDD" device=""/>
 <part name="VDD15" library="supply1" library_urn="urn:adsk.eagle:library:371" deviceset="VDD" device=""/>
+<part name="VDD1" library="supply1" library_urn="urn:adsk.eagle:library:371" deviceset="VDD" device=""/>
+<part name="F1" library="polyfuse-smd_10" deviceset="?" device="1206L" technology="050"/>
+<part name="D1" library="diode" library_urn="urn:adsk.eagle:library:210" deviceset="ZENER-DIODE" device="ZD-7.5" package3d_urn="urn:adsk.eagle:package:43411/1" value="5.6V"/>
+<part name="VSS23" library="supply1" library_urn="urn:adsk.eagle:library:371" deviceset="VSS" device=""/>
 </parts>
 <sheets>
@@
 <attribute name="VALUE" x="111.76" y="-53.34" size="1.778" layer="96" rot="R90"/>
 </instance>
-<instance part="VDD8" gate="G$1" x="114.3" y="-40.64" smashed="yes">
-<attribute name="VALUE" x="111.76" y="-43.18" size="1.778" layer="96" rot="R90"/>
-</instance>
 <instance part="C8" gate="G$1" x="12.7" y="50.8" smashed="yes">
 <attribute name="NAME" x="13.716" y="51.435" size="1.778" layer="95"/>
@@
 <attribute name="NAME" x="101.6" y="-56.642" size="1.524" layer="95"/>
 </instance>
-<instance part="VDD13" gate="G$1" x="96.52" y="-50.8" smashed="yes">
-<attribute name="VALUE" x="93.98" y="-53.34" size="1.778" layer="96" rot="R90"/>
-</instance>
 <instance part="VSS20" gate="G$1" x="96.52" y="-58.42" smashed="yes">
 <attribute name="VALUE" x="93.98" y="-63.5" size="1.778" layer="96" rot="R90"/>
@@
 <instance part="VDD15" gate="G$1" x="5.08" y="27.94" smashed="yes" rot="R180">
 <attribute name="VALUE" x="7.62" y="30.48" size="1.778" layer="96" rot="R270"/>
+</instance>
+<instance part="VDD1" gate="G$1" x="111.76" y="-60.96" smashed="yes" rot="R180">
+<attribute name="VALUE" x="114.3" y="-58.42" size="1.778" layer="96" rot="R270"/>
+</instance>
+<instance part="F1" gate="G$1" x="121.92" y="-58.42" smashed="yes">
+<attribute name="NAME" x="118.11" y="-55.88" size="1.778" layer="95"/>
+<attribute name="VALUE" x="118.11" y="-62.23" size="1.778" layer="96"/>
+</instance>
+<instance part="D1" gate="G$1" x="129.54" y="-55.88" smashed="yes" rot="R180">
+<attribute name="NAME" x="131.318" y="-57.785" size="1.778" layer="95" rot="R180"/>
+<attribute name="VALUE" x="131.318" y="-52.451" size="1.778" layer="96" rot="R180"/>
+</instance>
+<instance part="VSS23" gate="G$1" x="137.16" y="-55.88" smashed="yes" rot="R90">
+<attribute name="VALUE" x="142.24" y="-58.42" size="1.778" layer="96" rot="R180"/>
 </instance>
 </instances>
@@
 <junction x="-15.24" y="66.04"/>
 </segment>
+<segment>
+<pinref part="D1" gate="G$1" pin="A"/>
+<pinref part="VSS23" gate="G$1" pin="VSS"/>
+<wire x1="134.62" y1="-55.88" x2="132.08" y2="-55.88" width="0.1524" layer="91"/>
+<junction x="134.62" y="-55.88"/>
+</segment>
 </net>
 <net name="VDD" class="0">
@@
 </segment>
 <segment>
-<pinref part="X3" gate="-1" pin="S"/>
-<pinref part="VDD8" gate="G$1" pin="VDD"/>
-<junction x="114.3" y="-43.18"/>
-</segment>
-<segment>
 <pinref part="SV4" gate="G$1" pin="9"/>
 <pinref part="VDD9" gate="G$1" pin="VDD"/>
@@
 </segment>
 <segment>
-<pinref part="X4" gate="-1" pin="S"/>
-<pinref part="VDD13" gate="G$1" pin="VDD"/>
-<junction x="96.52" y="-53.34"/>
-</segment>
-<segment>
 <pinref part="L1" gate="G$1" pin="2"/>
 <pinref part="VDD14" gate="G$1" pin="VDD"/>
@@
 <pinref part="VDD15" gate="G$1" pin="VDD"/>
 <junction x="5.08" y="30.48"/>
+</segment>
+<segment>
+<pinref part="VDD1" gate="G$1" pin="VDD"/>
+<wire x1="116.84" y1="-58.42" x2="111.76" y2="-58.42" width="0.1524" layer="91"/>
+<junction x="111.76" y="-58.42"/>
+<pinref part="F1" gate="G$1" pin="2"/>
 </segment>
 </net>
@@
 </segment>
 </net>
+<net name="N$60" class="0">
+<segment>
+<wire x1="127" y1="-58.42" x2="127" y2="-55.88" width="0.1524" layer="91"/>
+<wire x1="127" y1="-55.88" x2="127" y2="-50.8" width="0.1524" layer="91"/>
+<wire x1="127" y1="-50.8" x2="109.22" y2="-50.8" width="0.1524" layer="91"/>
+<pinref part="X4" gate="-1" pin="S"/>
+<wire x1="96.52" y1="-53.34" x2="96.52" y2="-43.18" width="0.1524" layer="91"/>
+<pinref part="X3" gate="-1" pin="S"/>
+<wire x1="96.52" y1="-43.18" x2="109.22" y2="-43.18" width="0.1524" layer="91"/>
+<wire x1="109.22" y1="-43.18" x2="114.3" y2="-43.18" width="0.1524" layer="91"/>
+<wire x1="109.22" y1="-50.8" x2="109.22" y2="-43.18" width="0.1524" layer="91"/>
+<junction x="96.52" y="-53.34"/>
+<junction x="109.22" y="-43.18"/>
+<junction x="114.3" y="-43.18"/>
+<pinref part="F1" gate="G$1" pin="1"/>
+<pinref part="D1" gate="G$1" pin="C"/>
+<junction x="127" y="-55.88"/>
+</segment>
+</net>

Commit message: updatei# Please enter the commit message for your changes. Lines starting
Parts:
- removed LED1: RUN, led:LEDCHIPLED_1206
- removed S2: RESET_PB, switch-omron:10-XX
- added S3: RESETSW, SamacSys_Parts:B3W-9000-Y1N
Connections:
- net N$2: now also S3.1, S3.2; no longer S2.S1
- net N$9: now also S3.+; no longer LED1.A
- net VSS: now also S3.-, S3.3, S3.4; no longer LED1.C, S2.P1
Changed lines of the file:
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@@
 <part name="VSS9" library="supply1" library_urn="urn:adsk.eagle:library:371" deviceset="VSS" device=""/>
 <part name="R5" library="rcl" library_urn="urn:adsk.eagle:library:334" deviceset="R-US_" device="R0805" package3d_urn="urn:adsk.eagle:package:23553/2" value="220"/>
-<part name="LED1" library="led" library_urn="urn:adsk.eagle:library:259" deviceset="LED" device="CHIPLED_1206" package3d_urn="urn:adsk.eagle:package:15823/2" value="RUN"/>
-<part name="VSS10" library="supply1" library_urn="urn:adsk.eagle:library:371" deviceset="VSS" device=""/>
 <part name="LED2" library="led" library_urn="urn:adsk.eagle:library:259" deviceset="LED" device="CHIPLED_1206" package3d_urn="urn:adsk.eagle:package:15823/2" value="MODE"/>
 <part name="VSS11" library="supply1" library_urn="urn:adsk.eagle:library:371" deviceset="VSS" device=""/>
@@
 <part name="VSS19" library="supply1" library_urn="urn:adsk.eagle:library:371" deviceset="VSS" device=""/>
 <part name="VDD12" library="supply1" library_urn="urn:adsk.eagle:library:371" deviceset="VDD" device=""/>
-<part name="S2" library="switch-omron" library_urn="urn:adsk.eagle:library:377" deviceset="10-XX" device="" package3d_urn="urn:adsk.eagle:package:27496/1" value="RESET_PB"/>
 <part name="X4" library="con-molex" library_urn="urn:adsk.eagle:library:165" deviceset="22-23-2021" device="" package3d_urn="urn:adsk.eagle:package:8078633/1" value="GLORY"/>
 <part name="VSS20" library="supply1" library_urn="urn:adsk.eagle:library:371" deviceset="VSS" device=""/>
@@
 <part name="D1" library="diode" library_urn="urn:adsk.eagle:library:210" deviceset="ZENER-DIODE" device="ZD-7.5" package3d_urn="urn:adsk.eagle:package:43411/1" value="5.6V"/>
 <part name="VSS23" library="supply1" library_urn="urn:adsk.eagle:library:371" deviceset="VSS" device=""/>
+<part name="S3" library="SamacSys_Parts" deviceset="B3W-9000-Y1N" device="" value="RESETSW"/>
+<part name="VSS24" library="supply1" library_urn="urn:adsk.eagle:library:371" deviceset="VSS" device=""/>
+<part name="VSS25" library="supply1" library_urn="urn:adsk.eagle:library:371" deviceset="VSS" device=""/>
 </parts>
 <sheets>
@@
 <attribute name="VALUE" x="168.402" y="-31.75" size="1.778" layer="96" rot="R90"/>
 </instance>
-<instance part="LED1" gate="G$1" x="165.1" y="-35.56" smashed="yes">
-<attribute name="NAME" x="168.656" y="-40.132" size="1.778" layer="95" rot="R90"/>
-<attribute name="VALUE" x="170.815" y="-40.132" size="1.778" layer="96" rot="R90"/>
-</instance>
-<instance part="VSS10" gate="G$1" x="165.1" y="-43.18" smashed="yes">
-<attribute name="VALUE" x="162.56" y="-48.26" size="1.778" layer="96" rot="R90"/>
-</instance>
 <instance part="LED2" gate="G$1" x="78.74" y="86.36" smashed="yes">
 <attribute name="NAME" x="82.296" y="81.788" size="1.778" layer="95" rot="R90"/>
@@
 <attribute name="VALUE" x="43.18" y="15.24" size="1.778" layer="96" rot="R90"/>
 </instance>
-<instance part="S2" gate="1" x="129.54" y="-40.64" smashed="yes">
-<attribute name="NAME" x="123.19" y="-43.18" size="1.778" layer="95" rot="R90"/>
-<attribute name="VALUE" x="125.73" y="-37.465" size="1.778" layer="96" rot="R90"/>
-</instance>
 <instance part="X4" gate="-1" x="99.06" y="-53.34" smashed="yes">
 <attribute name="NAME" x="101.6" y="-54.102" size="1.524" layer="95"/>
@@
 <instance part="VSS23" gate="G$1" x="137.16" y="-55.88" smashed="yes" rot="R90">
 <attribute name="VALUE" x="142.24" y="-58.42" size="1.778" layer="96" rot="R180"/>
+</instance>
+<instance part="S3" gate="G$1" x="165.1" y="-53.34" smashed="yes">
+<attribute name="NAME" x="181.61" y="-45.72" size="1.778" layer="95" align="center-left"/>
+<attribute name="VALUE" x="181.61" y="-48.26" size="1.778" layer="96" align="center-left"/>
+</instance>
+<instance part="VSS24" gate="G$1" x="165.1" y="-60.96" smashed="yes">
+<attribute name="VALUE" x="162.56" y="-66.04" size="1.778" layer="96" rot="R90"/>
+</instance>
+<instance part="VSS25" gate="G$1" x="185.42" y="-60.96" smashed="yes">
+<attribute name="VALUE" x="182.88" y="-66.04" size="1.778" layer="96" rot="R90"/>
 </instance>
 </instances>
@@
 </segment>
 <segment>
-<pinref part="LED1" gate="G$1" pin="C"/>
-<pinref part="VSS10" gate="G$1" pin="VSS"/>
-<junction x="165.1" y="-40.64"/>
-</segment>
-<segment>
 <pinref part="LED2" gate="G$1" pin="C"/>
 <pinref part="VSS11" gate="G$1" pin="VSS"/>
@@
 <pinref part="SV3" gate="G$1" pin="3"/>
 <junction x="137.16" y="-40.64"/>
-<wire x1="137.16" y1="-40.64" x2="137.16" y2="-45.72" width="0.1524" layer="91"/>
+<wire x1="137.16" y1="-40.64" x2="137.16" y2="-48.26" width="0.1524" layer="91"/>
 <junction x="137.16" y="-38.1"/>
-<pinref part="S2" gate="1" pin="P1"/>
-<wire x1="137.16" y1="-45.72" x2="137.16" y2="-48.26" width="0.1524" layer="91"/>
-<wire x1="132.08" y1="-45.72" x2="137.16" y2="-45.72" width="0.1524" layer="91"/>
-<junction x="132.08" y="-45.72"/>
-<junction x="137.16" y="-45.72"/>
 </segment>
 <segment>
@@
 <wire x1="134.62" y1="-55.88" x2="132.08" y2="-55.88" width="0.1524" layer="91"/>
 <junction x="134.62" y="-55.88"/>
+</segment>
+<segment>
+<pinref part="S3" gate="G$1" pin="3"/>
+<pinref part="VSS24" gate="G$1" pin="VSS"/>
+<junction x="165.1" y="-58.42"/>
+</segment>
+<segment>
+<pinref part="S3" gate="G$1" pin="-"/>
+<pinref part="VSS25" gate="G$1" pin="VSS"/>
+<junction x="185.42" y="-58.42"/>
+<pinref part="S3" gate="G$1" pin="4"/>
+<wire x1="185.42" y1="-53.34" x2="187.96" y2="-53.34" width="0.1524" layer="91"/>
+<wire x1="187.96" y1="-53.34" x2="187.96" y2="-58.42" width="0.1524" layer="91"/>
+<wire x1="187.96" y1="-58.42" x2="185.42" y2="-58.42" width="0.1524" layer="91"/>
+<junction x="185.42" y="-53.34"/>
 </segment>
 </net>
@@
 <junction x="137.16" y="-20.32"/>
 <wire x1="132.08" y1="-20.32" x2="137.16" y2="-20.32" width="0.1524" layer="91"/>
-<wire x1="132.08" y1="-20.32" x2="132.08" y2="-35.56" width="0.1524" layer="91"/>
+<wire x1="132.08" y1="-20.32" x2="132.08" y2="-30.48" width="0.1524" layer="91"/>
 <pinref part="SV3" gate="G$1" pin="1"/>
+<wire x1="132.08" y1="-30.48" x2="132.08" y2="-35.56" width="0.1524" layer="91"/>
 <wire x1="132.08" y1="-35.56" x2="137.16" y2="-35.56" width="0.1524" layer="91"/>
 <junction x="137.16" y="-35.56"/>
 <junction x="132.08" y="-20.32"/>
-<pinref part="S2" gate="1" pin="S1"/>
-<junction x="132.08" y="-35.56"/>
+<pinref part="S3" gate="G$1" pin="2"/>
+<pinref part="S3" gate="G$1" pin="1"/>
+<wire x1="165.1" y1="-55.88" x2="165.1" y2="-53.34" width="0.1524" layer="91"/>
+<wire x1="165.1" y1="-53.34" x2="165.1" y2="-50.8" width="0.1524" layer="91"/>
+<wire x1="165.1" y1="-50.8" x2="152.4" y2="-50.8" width="0.1524" layer="91"/>
+<wire x1="152.4" y1="-50.8" x2="152.4" y2="-30.48" width="0.1524" layer="91"/>
+<wire x1="152.4" y1="-30.48" x2="132.08" y2="-30.48" width="0.1524" layer="91"/>
+<junction x="132.08" y="-30.48"/>
+<junction x="165.1" y="-53.34"/>
+<junction x="165.1" y="-55.88"/>
 </segment>
 </net>
@@
 <segment>
 <pinref part="R5" gate="G$1" pin="1"/>
-<pinref part="LED1" gate="G$1" pin="A"/>
+<wire x1="165.1" y1="-33.02" x2="190.5" y2="-33.02" width="0.1524" layer="91"/>
+<wire x1="190.5" y1="-33.02" x2="190.5" y2="-55.88" width="0.1524" layer="91"/>
+<pinref part="S3" gate="G$1" pin="+"/>
+<wire x1="190.5" y1="-55.88" x2="185.42" y2="-55.88" width="0.1524" layer="91"/>
+<junction x="185.42" y="-55.88"/>
 <junction x="165.1" y="-33.02"/>
 </segment>
