File: touch_board/touch_board.sch (EAGLE design)
At the start: 42 parts, among them IC1 PIC18F47K42-I_PT, IC2 MAX203EEWP, K1 G6K-2P, X1 RS-232-1, X2 RS-232-2, X3 POWER, X4 GLORY, X5 Relay conn

Commit message: update
Parts:
- added D2: 1N4148, diode:CGRM4001-G
Connections:
- new net N$59: C7.1, D2.A, R4.1
- net N$2: now also D2.C; no longer C7.1, R4.1
Other:
- moved on the sheet: C7, R4
Changed lines of the file:
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@@
 <part name="VSS24" library="supply1" library_urn="urn:adsk.eagle:library:371" deviceset="VSS" device=""/>
 <part name="VSS25" library="supply1" library_urn="urn:adsk.eagle:library:371" deviceset="VSS" device=""/>
+<part name="D2" library="diode" library_urn="urn:adsk.eagle:library:210" deviceset="CGRM400*-G" device="" package3d_urn="urn:adsk.eagle:package:43457/2" technology="1" value="1N4148"/>
 </parts>
 <sheets>
@@
 <attribute name="VALUE" x="110.236" y="84.709" size="1.778" layer="96"/>
 </instance>
-<instance part="C7" gate="G$1" x="76.2" y="-22.86" smashed="yes">
-<attribute name="NAME" x="77.216" y="-22.225" size="1.778" layer="95"/>
-<attribute name="VALUE" x="77.216" y="-27.051" size="1.778" layer="96"/>
+<instance part="C7" gate="G$1" x="66.04" y="-22.86" smashed="yes">
+<attribute name="NAME" x="67.056" y="-22.225" size="1.778" layer="95"/>
+<attribute name="VALUE" x="67.056" y="-27.051" size="1.778" layer="96"/>
 </instance>
 <instance part="VSS7" gate="G$1" x="76.2" y="-30.48" smashed="yes">
@@
 <attribute name="VALUE" x="79.502" y="-19.05" size="1.778" layer="96" rot="R90"/>
 </instance>
-<instance part="R4" gate="G$1" x="71.12" y="-20.32" smashed="yes" rot="R180">
-<attribute name="NAME" x="74.93" y="-21.8186" size="1.778" layer="95" rot="R180"/>
-<attribute name="VALUE" x="74.93" y="-17.018" size="1.778" layer="96" rot="R180"/>
-</instance>
-<instance part="VDD5" gate="G$1" x="63.5" y="-20.32" smashed="yes" rot="R90">
-<attribute name="VALUE" x="66.04" y="-22.86" size="1.778" layer="96" rot="R180"/>
+<instance part="R4" gate="G$1" x="48.26" y="-20.32" smashed="yes" rot="R180">
+<attribute name="NAME" x="52.07" y="-21.8186" size="1.778" layer="95" rot="R180"/>
+<attribute name="VALUE" x="52.07" y="-17.018" size="1.778" layer="96" rot="R180"/>
+</instance>
+<instance part="VDD5" gate="G$1" x="40.64" y="-20.32" smashed="yes" rot="R90">
+<attribute name="VALUE" x="43.18" y="-22.86" size="1.778" layer="96" rot="R180"/>
 </instance>
 <instance part="SV1" gate="1" x="76.2" y="-48.26" smashed="yes" rot="R90">
@@
 <instance part="VSS25" gate="G$1" x="185.42" y="-60.96" smashed="yes">
 <attribute name="VALUE" x="182.88" y="-66.04" size="1.778" layer="96" rot="R90"/>
+</instance>
+<instance part="D2" gate="G$1" x="68.58" y="-20.32" smashed="yes">
+<attribute name="NAME" x="71.12" y="-19.8374" size="1.778" layer="95"/>
+<attribute name="VALUE" x="71.12" y="-22.6314" size="1.778" layer="96"/>
 </instance>
 </instances>
@@
 <pinref part="C7" gate="G$1" pin="2"/>
 <pinref part="VSS7" gate="G$1" pin="VSS"/>
+<wire x1="66.04" y1="-27.94" x2="76.2" y2="-27.94" width="0.1524" layer="91"/>
+<junction x="66.04" y="-27.94"/>
 <junction x="76.2" y="-27.94"/>
 </segment>
@@
 <pinref part="R4" gate="G$1" pin="2"/>
 <pinref part="VDD5" gate="G$1" pin="VDD"/>
-<junction x="66.04" y="-20.32"/>
+<junction x="43.18" y="-20.32"/>
 </segment>
 <segment>
@@
 <net name="N$2" class="0">
 <segment>
-<pinref part="C7" gate="G$1" pin="1"/>
 <pinref part="R3" gate="G$1" pin="1"/>
-<pinref part="R4" gate="G$1" pin="1"/>
-<junction x="76.2" y="-20.32"/>
 <wire x1="76.2" y1="-20.32" x2="83.82" y2="-20.32" width="0.1524" layer="91"/>
 <wire x1="83.82" y1="-20.32" x2="83.82" y2="-40.64" width="0.1524" layer="91"/>
@@
 <junction x="165.1" y="-53.34"/>
 <junction x="165.1" y="-55.88"/>
+<pinref part="D2" gate="G$1" pin="C"/>
+<wire x1="71.12" y1="-20.32" x2="76.2" y2="-20.32" width="0.1524" layer="91"/>
+<junction x="71.12" y="-20.32"/>
+<junction x="76.2" y="-20.32"/>
 </segment>
 </net>
@@
 </segment>
 </net>
+<net name="N$59" class="0">
+<segment>
+<pinref part="C7" gate="G$1" pin="1"/>
+<pinref part="R4" gate="G$1" pin="1"/>
+<junction x="53.34" y="-20.32"/>
+<wire x1="53.34" y1="-20.32" x2="66.04" y2="-20.32" width="0.1524" layer="91"/>
+<pinref part="D2" gate="G$1" pin="A"/>
+<junction x="66.04" y="-20.32"/>
+</segment>
+</net>
