File: touch_board/d232_board.sch (EAGLE design)
At the start: 11 parts, among them IC3 7805TV, IC4 7805TV

Commit message: update
Parts:
- added SG1, SG2, SG3: EB2209A, buzzer:EB2209A
Connections:
- new net N$1: IC1.O1, JP1.1
- new net N$10: IC1.I2, JP4.2
- new net N$11: IC1.I3, JP4.3
- new net N$12: IC1.I4, JP4.4
- new net N$13: IC1.I5, JP4.5
- new net N$14: IC1.I6, JP4.6
- new net N$15: IC1.I7, JP4.7
- new net N$16: IC1.I8, JP4.8
- new net N$17: IC2.I1, JP5.1
- new net N$18: IC2.I2, JP5.2
- new net N$19: IC2.I3, JP5.3
- new net N$2: IC1.O2, JP1.2
- new net N$20: IC2.I4, JP5.4
- new net N$21: IC2.I5, JP5.5
- new net N$22: IC2.I6, JP5.6
- new net N$23: IC2.I7, JP5.7
- new net N$24: IC2.I8, JP5.8
- new net N$25: IC2.O1, SG1.-
- new net N$26: IC2.O2, SG2.-
- new net N$27: IC2.O3, SG3.-
- new net N$3: IC1.O3, JP1.3
- new net N$4: IC1.O4, JP1.4
- new net N$5: IC1.O5, JP1.5
- new net N$6: IC1.O6, JP1.6
- new net N$7: IC1.O7, JP1.7
- new net N$8: IC1.O8, JP1.8
- new net N$9: IC1.I1, JP4.1
- net +10V: now also SG1.+
- net +24V: now also SG2.+, SG3.+
- net +5V: now also IC1.CD+
- net GND: now also JP4.10, JP5.10
Other:
- moved on the sheet: JP1, JP2, JP4, JP5

Commit message: board cons
Connections:
- net +10V: now also JP7.7; no longer JP7.4
- net +5V: now also JP7.5; no longer JP7.3
- net GND: now also JP7.3, JP7.4
Changed lines of the file:
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@@
 <junction x="53.34" y="-10.16"/>
 <junction x="48.26" y="-22.86"/>
+<wire x1="55.88" y1="-10.16" x2="58.42" y2="-10.16" width="0.1524" layer="91"/>
+<pinref part="JP7" gate="A" pin="4"/>
+<wire x1="58.42" y1="-10.16" x2="60.96" y2="-10.16" width="0.1524" layer="91"/>
+<wire x1="60.96" y1="-10.16" x2="60.96" y2="-2.54" width="0.1524" layer="91"/>
+<pinref part="JP7" gate="A" pin="3"/>
+<wire x1="58.42" y1="-2.54" x2="58.42" y2="-10.16" width="0.1524" layer="91"/>
+<junction x="55.88" y="-10.16"/>
+<junction x="58.42" y="-10.16"/>
 </segment>
 <segment>
@@
 </segment>
 <segment>
-<pinref part="JP7" gate="A" pin="3"/>
-<pinref part="SUPPLY11" gate="+5V" pin="+5V"/>
-<wire x1="58.42" y1="-2.54" x2="58.42" y2="-22.86" width="0.1524" layer="91"/>
-<junction x="58.42" y="-22.86"/>
+<pinref part="IC1" gate="G$1" pin="CD+"/>
+<pinref part="SUPPLY13" gate="+5V" pin="+5V"/>
 </segment>
 <segment>
-<pinref part="IC1" gate="G$1" pin="CD+"/>
-<pinref part="SUPPLY13" gate="+5V" pin="+5V"/>
+<pinref part="JP7" gate="A" pin="5"/>
+<wire x1="63.5" y1="-2.54" x2="63.5" y2="-20.32" width="0.1524" layer="91"/>
+<wire x1="63.5" y1="-20.32" x2="58.42" y2="-20.32" width="0.1524" layer="91"/>
+<pinref part="SUPPLY11" gate="+5V" pin="+5V"/>
+<wire x1="58.42" y1="-20.32" x2="58.42" y2="-22.86" width="0.1524" layer="91"/>
+<junction x="58.42" y="-22.86"/>
 </segment>
 </net>
@@
 </segment>
 <segment>
-<pinref part="JP7" gate="A" pin="4"/>
-<wire x1="60.96" y1="-2.54" x2="60.96" y2="-22.86" width="0.1524" layer="91"/>
-<pinref part="SUPPLY12" gate="G$1" pin="+10V"/>
-<wire x1="60.96" y1="-22.86" x2="63.5" y2="-22.86" width="0.1524" layer="91"/>
-<junction x="63.5" y="-22.86"/>
-</segment>
-<segment>
 <pinref part="SG1" gate="G$1" pin="+"/>
 <pinref part="SUPPLY16" gate="G$1" pin="+10V"/>
 <junction x="73.66" y="43.18"/>
 </segment>
+<segment>
+<pinref part="JP7" gate="A" pin="7"/>
+<wire x1="68.58" y1="-2.54" x2="68.58" y2="-22.86" width="0.1524" layer="91"/>
+<pinref part="SUPPLY12" gate="G$1" pin="+10V"/>
+<wire x1="68.58" y1="-22.86" x2="63.5" y2="-22.86" width="0.1524" layer="91"/>
+<junction x="63.5" y="-22.86"/>
+</segment>
 </net>

Commit message: update board
Parts:
- added C1, C3: 0.47, rcl:C-USC1206K
- added C2, C4, C5: 22uf, rcl:C-USC1206K
- added R1, R2, R3, R4, R5, R6, R7, R8: 91, rcl:R-US_0204/2V
- added X1: 057-050-1, con-panduit:057-050-1
- IC1, IC2: value (none) -> uln2803
Connections:
- new net N$28: JP6.1, X1-1.S
- new net N$29: JP6.2, X1-2.S
- new net N$30: JP6.3, X1-3.S
- new net N$31: JP6.4, X1-4.S
- new net N$32: JP2.1, R1.1
- new net N$33: JP2.2, R2.1
- new net N$34: JP2.3, R3.1
- new net N$35: JP2.4, R4.1
- new net N$36: JP2.5, R5.1
- new net N$37: JP2.6, R6.1
- new net N$38: JP2.7, R7.1
- new net N$39: JP2.8, R8.1
- net +10V: now also C4.1
- net +24V: now also C1.1, C3.1
- net +5V: now also C2.1, C5.1, R1.2, R2.2, R3.2, R4.2, R5.2, R6.2, R7.2, R8.2
- net GND: now also C1.2, C2.2, C3.2, C4.2, C5.2, JP6.10, X1-50.S
- net N$10: now also X1-10.S
- net N$11: now also X1-11.S
- net N$14: now also X1-14.S
- net N$16: now also X1-16.S
- net N$17: now also X1-17.S
- net N$18: now also X1-18.S
- net N$20: now also X1-20.S
- net N$21: now also X1-21.S
- net N$9: now also X1-9.S
Other:
- moved on the sheet: JP6

Commit message: up
Parts:
- added IC5: 7805TV, linear:7805TV
- added R9: 91, rcl:R-US_0204/2V
Connections:
- new net +12V: C3.1, IC4.VI, IC5.VO
- net +24V: now also IC5.VI; no longer C3.1, IC4.VI
- net +5V: now also R9.2
- net GND: now also IC5.GND
- net N$29: now also R9.1
Changed lines of the file:
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@@
 <part name="SUPPLY5" library="supply2" library_urn="urn:adsk.eagle:library:372" deviceset="+5V" device=""/>
 <part name="SUPPLY6" library="supply2" library_urn="urn:adsk.eagle:library:372" deviceset="+10V" device=""/>
-<part name="SUPPLY7" library="supply2" library_urn="urn:adsk.eagle:library:372" deviceset="+24V" device=""/>
 <part name="SUPPLY8" library="supply2" library_urn="urn:adsk.eagle:library:372" deviceset="+24V" device=""/>
 <part name="SUPPLY9" library="supply2" library_urn="urn:adsk.eagle:library:372" deviceset="+24V" device=""/>
@@
 <part name="C5" library="rcl" library_urn="urn:adsk.eagle:library:334" deviceset="C-US" device="C1206K" package3d_urn="urn:adsk.eagle:package:23682/2" value="22uf"/>
 <part name="SUPPLY26" library="supply2" library_urn="urn:adsk.eagle:library:372" deviceset="GND" device=""/>
+<part name="IC5" library="linear" library_urn="urn:adsk.eagle:library:262" deviceset="78*" device="TV" package3d_urn="urn:adsk.eagle:package:16417/2" technology="05"/>
+<part name="SUPPLY27" library="supply2" library_urn="urn:adsk.eagle:library:372" deviceset="+24V" device=""/>
+<part name="SUPPLY28" library="supply2" library_urn="urn:adsk.eagle:library:372" deviceset="GND" device=""/>
+<part name="SUPPLY29" library="supply2" library_urn="urn:adsk.eagle:library:372" deviceset="+12V" device=""/>
+<part name="SUPPLY7" library="supply2" library_urn="urn:adsk.eagle:library:372" deviceset="+12V" device=""/>
+<part name="R9" library="rcl" library_urn="urn:adsk.eagle:library:334" deviceset="R-US_" device="0204/2V" package3d_urn="urn:adsk.eagle:package:23495/1" value="91"/>
+<part name="SUPPLY30" library="supply2" library_urn="urn:adsk.eagle:library:372" deviceset="+5V" device=""/>
 </parts>
 <sheets>
@@
 <attribute name="VALUE" x="38.1" y="-12.065" size="1.778" layer="96"/>
 </instance>
-<instance part="SUPPLY7" gate="+24V" x="20.32" y="-15.24" smashed="yes">
-<attribute name="VALUE" x="17.78" y="-12.065" size="1.778" layer="96"/>
-</instance>
 <instance part="SUPPLY8" gate="+24V" x="-7.62" y="-15.24" smashed="yes">
 <attribute name="VALUE" x="-10.16" y="-12.065" size="1.778" layer="96"/>
@@
 <instance part="SUPPLY26" gate="GND" x="111.76" y="55.88" smashed="yes">
 <attribute name="VALUE" x="109.855" y="52.705" size="1.778" layer="96"/>
+</instance>
+<instance part="IC5" gate="A1" x="104.14" y="-27.94" smashed="yes">
+<attribute name="NAME" x="96.52" y="-22.225" size="1.778" layer="95"/>
+<attribute name="VALUE" x="96.52" y="-24.765" size="1.778" layer="96"/>
+</instance>
+<instance part="SUPPLY27" gate="+24V" x="93.98" y="-25.4" smashed="yes">
+<attribute name="VALUE" x="91.44" y="-22.225" size="1.778" layer="96"/>
+</instance>
+<instance part="SUPPLY28" gate="GND" x="104.14" y="-38.1" smashed="yes">
+<attribute name="VALUE" x="102.235" y="-41.275" size="1.778" layer="96"/>
+</instance>
+<instance part="SUPPLY29" gate="+12V" x="114.3" y="-25.4" smashed="yes">
+<attribute name="VALUE" x="111.76" y="-22.225" size="1.778" layer="96"/>
+</instance>
+<instance part="SUPPLY7" gate="+12V" x="20.32" y="-15.24" smashed="yes">
+<attribute name="VALUE" x="17.78" y="-12.065" size="1.778" layer="96"/>
+</instance>
+<instance part="R9" gate="G$1" x="40.64" y="91.44" smashed="yes">
+<attribute name="NAME" x="36.83" y="92.9386" size="1.778" layer="95"/>
+<attribute name="VALUE" x="36.83" y="88.138" size="1.778" layer="96"/>
+</instance>
+<instance part="SUPPLY30" gate="+5V" x="45.72" y="93.98" smashed="yes">
+<attribute name="VALUE" x="43.815" y="97.155" size="1.778" layer="96"/>
 </instance>
 </instances>
@@
 <pinref part="SUPPLY26" gate="GND" pin="GND"/>
 </segment>
+<segment>
+<pinref part="IC5" gate="A1" pin="GND"/>
+<pinref part="SUPPLY28" gate="GND" pin="GND"/>
+</segment>
 </net>
 <net name="+5V" class="0">
@@
 <pinref part="C2" gate="G$1" pin="1"/>
 <junction x="12.7" y="-17.78"/>
-<pinref part="C2" gate="G$1" pin="1"/>
 </segment>
 <segment>
@@
 <wire x1="111.76" y1="66.04" x2="101.6" y2="66.04" width="0.1524" layer="91"/>
 </segment>
+<segment>
+<pinref part="R9" gate="G$1" pin="2"/>
+<pinref part="SUPPLY30" gate="+5V" pin="+5V"/>
+</segment>
 </net>
 <net name="+10V" class="0">
@@
 <pinref part="C4" gate="G$1" pin="1"/>
 <junction x="40.64" y="-17.78"/>
-<pinref part="C4" gate="G$1" pin="1"/>
 </segment>
 <segment>
@@
 <net name="+24V" class="0">
 <segment>
-<pinref part="IC4" gate="A1" pin="VI"/>
-<pinref part="SUPPLY7" gate="+24V" pin="+24V"/>
-<pinref part="C3" gate="G$1" pin="1"/>
-<junction x="20.32" y="-17.78"/>
-<pinref part="C3" gate="G$1" pin="1"/>
-</segment>
-<segment>
 <pinref part="IC3" gate="A1" pin="VI"/>
 <pinref part="SUPPLY8" gate="+24V" pin="+24V"/>
 <pinref part="C1" gate="G$1" pin="1"/>
 <junction x="-7.62" y="-17.78"/>
-<pinref part="C1" gate="G$1" pin="1"/>
 </segment>
 <segment>
@@
 <pinref part="SUPPLY18" gate="+24V" pin="+24V"/>
 <junction x="111.76" y="22.86"/>
+</segment>
+<segment>
+<pinref part="IC5" gate="A1" pin="VI"/>
+<pinref part="SUPPLY27" gate="+24V" pin="+24V"/>
 </segment>
 </net>
@@
 <wire x1="-22.86" y1="78.74" x2="-15.24" y2="78.74" width="0.1524" layer="91"/>
 <junction x="-15.24" y="78.74"/>
+<wire x1="-22.86" y1="88.9" x2="-7.62" y2="88.9" width="0.1524" layer="91"/>
+<wire x1="-7.62" y1="88.9" x2="-7.62" y2="91.44" width="0.1524" layer="91"/>
+<pinref part="R9" gate="G$1" pin="1"/>
+<wire x1="35.56" y1="91.44" x2="-7.62" y2="91.44" width="0.1524" layer="91"/>
+<junction x="-22.86" y="88.9"/>
 </segment>
 </net>
@@
 </segment>
 </net>
+<net name="+12V" class="0">
+<segment>
+<pinref part="IC5" gate="A1" pin="VO"/>
+<pinref part="SUPPLY29" gate="+12V" pin="+12V"/>
+</segment>
+<segment>
+<pinref part="IC4" gate="A1" pin="VI"/>
+<pinref part="C3" gate="G$1" pin="1"/>
+<junction x="20.32" y="-17.78"/>
+<pinref part="SUPPLY7" gate="+12V" pin="+12V"/>
+</segment>
+</net>

Commit message: up
Parts:
- added C6, C7: 0.47, rcl:C-USC1206K
- added C8: 22uf, rcl:C-USC1206K
- added LED1: PWR, led:LEDCHIPLED_1206
- added R10: 91, rcl:R-US_0204/2V
- added R11: 1k, rcl:R-US_0204/2V
- JP1: value (none) -> LEDC
- JP2: value (none) -> LEDP
- JP3: value (none) -> PORTIO
- JP4: value (none) -> PORT2
- JP5: value (none) -> PORT3
- JP6: value (none) -> PORT1
- JP7: value (none) -> DC POWER
- renumbered IC3 to IC3_5V, IC4 to IC4_10V, IC5 to IC5_12V
Connections:
- new net N$40: IC2.O4, JP3.2
- new net N$41: IC2.O5, JP3.3
- new net N$42: IC2.O6, JP3.4
- new net N$43: IC2.O7, JP3.5
- new net N$44: IC2.O8, JP3.6
- new net N$45: IC2.CD+, JP3.7
- new net N$46: LED1.A, R11.1
- net +12V: now also C8.1, JP7.8
- net +24V: now also C7.1, JP3.1
- net +5V: now also C6.1, R10.2, R11.2
- net GND: now also C6.2, C7.2, C8.2, JP1.9, JP2.9, JP3.8, LED1.C
- net N$30: now also R10.1

Commit message: add board design files
Parts:
- added TP1, TP2, TP3, TP4, TP5, TP6: TPB2,54, testpad:TPB2,54
Connections:
- net +5V: now also TP3.TP, TP5.TP
- net GND: now also TP4.TP, TP6.TP
- net N$28: now also TP1.TP
- net N$31: now also TP2.TP
Changed lines of the file:
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@@
 <?xml version="1.0" encoding="utf-8"?>
 <!DOCTYPE eagle SYSTEM "eagle.dtd">
-<eagle version="9.4.2">
+<eagle version="9.5.0">
 <drawing>
 <settings>
@@
 <part name="R11" library="rcl" library_urn="urn:adsk.eagle:library:334" deviceset="R-US_" device="0204/2V" package3d_urn="urn:adsk.eagle:package:23495/1" value="1k"/>
 <part name="SUPPLY41" library="supply2" library_urn="urn:adsk.eagle:library:372" deviceset="+5V" device=""/>
+<part name="TP1" library="testpad" library_urn="urn:adsk.eagle:library:385" deviceset="TP" device="B2,54" package3d_urn="urn:adsk.eagle:package:27948/1"/>
+<part name="TP2" library="testpad" library_urn="urn:adsk.eagle:library:385" deviceset="TP" device="B2,54" package3d_urn="urn:adsk.eagle:package:27948/1"/>
+<part name="TP3" library="testpad" library_urn="urn:adsk.eagle:library:385" deviceset="TP" device="B2,54" package3d_urn="urn:adsk.eagle:package:27948/1"/>
+<part name="TP4" library="testpad" library_urn="urn:adsk.eagle:library:385" deviceset="TP" device="B2,54" package3d_urn="urn:adsk.eagle:package:27948/1"/>
+<part name="TP5" library="testpad" library_urn="urn:adsk.eagle:library:385" deviceset="TP" device="B2,54" package3d_urn="urn:adsk.eagle:package:27948/1"/>
+<part name="TP6" library="testpad" library_urn="urn:adsk.eagle:library:385" deviceset="TP" device="B2,54" package3d_urn="urn:adsk.eagle:package:27948/1"/>
+<part name="SUPPLY42" library="supply2" library_urn="urn:adsk.eagle:library:372" deviceset="GND" device=""/>
+<part name="SUPPLY43" library="supply2" library_urn="urn:adsk.eagle:library:372" deviceset="GND" device=""/>
+<part name="SUPPLY44" library="supply2" library_urn="urn:adsk.eagle:library:372" deviceset="+5V" device=""/>
+<part name="SUPPLY45" library="supply2" library_urn="urn:adsk.eagle:library:372" deviceset="+5V" device=""/>
 </parts>
 <sheets>
@@
 <instance part="SUPPLY41" gate="+5V" x="-22.86" y="-2.54" smashed="yes">
 <attribute name="VALUE" x="-24.765" y="0.635" size="1.778" layer="96"/>
+</instance>
+<instance part="TP1" gate="G$1" x="-63.5" y="109.22" smashed="yes">
+<attribute name="NAME" x="-64.77" y="110.49" size="1.778" layer="95"/>
+<attribute name="TP_SIGNAL_NAME" x="-62.23" y="107.95" size="1.778" layer="97"/>
+</instance>
+<instance part="TP2" gate="G$1" x="-55.88" y="109.22" smashed="yes">
+<attribute name="NAME" x="-57.15" y="110.49" size="1.778" layer="95"/>
+<attribute name="TP_SIGNAL_NAME" x="-54.61" y="107.95" size="1.778" layer="97"/>
+</instance>
+<instance part="TP3" gate="G$1" x="66.04" y="109.22" smashed="yes">
+<attribute name="NAME" x="64.77" y="110.49" size="1.778" layer="95"/>
+<attribute name="TP_SIGNAL_NAME" x="67.31" y="107.95" size="1.778" layer="97"/>
+</instance>
+<instance part="TP4" gate="G$1" x="66.04" y="96.52" smashed="yes">
+<attribute name="NAME" x="64.77" y="97.79" size="1.778" layer="95"/>
+<attribute name="TP_SIGNAL_NAME" x="67.31" y="95.25" size="1.778" layer="97"/>
+</instance>
+<instance part="TP5" gate="G$1" x="78.74" y="109.22" smashed="yes">
+<attribute name="NAME" x="77.47" y="110.49" size="1.778" layer="95"/>
+<attribute name="TP_SIGNAL_NAME" x="80.01" y="107.95" size="1.778" layer="97"/>
+</instance>
+<instance part="TP6" gate="G$1" x="78.74" y="96.52" smashed="yes">
+<attribute name="NAME" x="77.47" y="97.79" size="1.778" layer="95"/>
+<attribute name="TP_SIGNAL_NAME" x="80.01" y="95.25" size="1.778" layer="97"/>
+</instance>
+<instance part="SUPPLY42" gate="GND" x="66.04" y="91.44" smashed="yes">
+<attribute name="VALUE" x="64.135" y="88.265" size="1.778" layer="96"/>
+</instance>
+<instance part="SUPPLY43" gate="GND" x="78.74" y="91.44" smashed="yes">
+<attribute name="VALUE" x="76.835" y="88.265" size="1.778" layer="96"/>
+</instance>
+<instance part="SUPPLY44" gate="+5V" x="63.5" y="106.68" smashed="yes" rot="R90">
+<attribute name="VALUE" x="60.325" y="104.775" size="1.778" layer="96" rot="R90"/>
+</instance>
+<instance part="SUPPLY45" gate="+5V" x="76.2" y="106.68" smashed="yes" rot="R90">
+<attribute name="VALUE" x="73.025" y="104.775" size="1.778" layer="96" rot="R90"/>
 </instance>
 </instances>
@@
 <pinref part="LED1" gate="G$1" pin="C"/>
 <pinref part="SUPPLY40" gate="GND" pin="GND"/>
+</segment>
+<segment>
+<pinref part="TP4" gate="G$1" pin="TP"/>
+<pinref part="SUPPLY42" gate="GND" pin="GND"/>
+</segment>
+<segment>
+<pinref part="TP6" gate="G$1" pin="TP"/>
+<pinref part="SUPPLY43" gate="GND" pin="GND"/>
 </segment>
 </net>
@@
 <pinref part="SUPPLY41" gate="+5V" pin="+5V"/>
 </segment>
+<segment>
+<pinref part="TP3" gate="G$1" pin="TP"/>
+<pinref part="SUPPLY44" gate="+5V" pin="+5V"/>
+</segment>
+<segment>
+<pinref part="TP5" gate="G$1" pin="TP"/>
+<pinref part="SUPPLY45" gate="+5V" pin="+5V"/>
+</segment>
 </net>
 <net name="+10V" class="0">
@@
 <pinref part="C7" gate="G$1" pin="1"/>
 <junction x="93.98" y="-27.94"/>
-<pinref part="C7" gate="G$1" pin="1"/>
 </segment>
 <segment>
@@
 <pinref part="X1" gate="-1" pin="S"/>
 <wire x1="-66.04" y1="86.36" x2="-66.04" y2="91.44" width="0.1524" layer="91"/>
-<wire x1="-66.04" y1="91.44" x2="-20.32" y2="91.44" width="0.1524" layer="91"/>
+<wire x1="-66.04" y1="91.44" x2="-63.5" y2="91.44" width="0.1524" layer="91"/>
 <pinref part="JP6" gate="A" pin="1"/>
+<wire x1="-63.5" y1="91.44" x2="-20.32" y2="91.44" width="0.1524" layer="91"/>
 <wire x1="-20.32" y1="91.44" x2="-20.32" y2="81.28" width="0.1524" layer="91"/>
 <wire x1="-20.32" y1="81.28" x2="-15.24" y2="81.28" width="0.1524" layer="91"/>
 <junction x="-15.24" y="81.28"/>
+<pinref part="TP1" gate="G$1" pin="TP"/>
+<wire x1="-63.5" y1="91.44" x2="-63.5" y2="106.68" width="0.1524" layer="91"/>
+<junction x="-63.5" y="91.44"/>
+<junction x="-63.5" y="106.68"/>
 </segment>
 </net>
@@
 <pinref part="X1" gate="-4" pin="S"/>
 <wire x1="-43.18" y1="81.28" x2="-43.18" y2="78.74" width="0.1524" layer="91"/>
-<wire x1="-43.18" y1="78.74" x2="-27.94" y2="78.74" width="0.1524" layer="91"/>
+<wire x1="-43.18" y1="78.74" x2="-30.48" y2="78.74" width="0.1524" layer="91"/>
+<wire x1="-30.48" y1="78.74" x2="-27.94" y2="78.74" width="0.1524" layer="91"/>
 <wire x1="-27.94" y1="78.74" x2="-27.94" y2="73.66" width="0.1524" layer="91"/>
 <pinref part="JP6" gate="A" pin="4"/>
 <wire x1="-27.94" y1="73.66" x2="-15.24" y2="73.66" width="0.1524" layer="91"/>
 <junction x="-15.24" y="73.66"/>
+<wire x1="-30.48" y1="78.74" x2="-30.48" y2="104.14" width="0.1524" layer="91"/>
+<wire x1="-30.48" y1="104.14" x2="-55.88" y2="104.14" width="0.1524" layer="91"/>
+<pinref part="TP2" gate="G$1" pin="TP"/>
+<wire x1="-55.88" y1="104.14" x2="-55.88" y2="106.68" width="0.1524" layer="91"/>
+<junction x="-30.48" y="78.74"/>
+<junction x="-55.88" y="106.68"/>
 </segment>
 </net>
@@
 <pinref part="C8" gate="G$1" pin="1"/>
 <junction x="114.3" y="-27.94"/>
-<pinref part="C8" gate="G$1" pin="1"/>
-</segment>
-<segment>
+</segment>
+<segment>

Commit message: up
Other:
- moved on the sheet: R1
Changed lines of the file:
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@@
 <attribute name="VALUE" x="-45.085" y="-41.275" size="1.778" layer="96"/>
 </instance>
-<instance part="R1" gate="G$1" x="96.52" y="83.82" smashed="yes">
-<attribute name="NAME" x="92.71" y="85.3186" size="1.778" layer="95"/>
-<attribute name="VALUE" x="92.71" y="80.518" size="1.778" layer="96"/>
+<instance part="R1" gate="G$1" x="96.52" y="93.98" smashed="yes">
+<attribute name="NAME" x="92.71" y="95.4786" size="1.778" layer="95"/>
+<attribute name="VALUE" x="92.71" y="90.678" size="1.778" layer="96"/>
 </instance>
 <instance part="R2" gate="G$1" x="96.52" y="81.28" smashed="yes">
@@
 <pinref part="R2" gate="G$1" pin="2"/>
 <junction x="101.6" y="81.28"/>
-<wire x1="101.6" y1="81.28" x2="101.6" y2="83.82" width="0.1524" layer="91"/>
-<junction x="101.6" y="83.82"/>
+<wire x1="101.6" y1="81.28" x2="101.6" y2="93.98" width="0.1524" layer="91"/>
+<junction x="101.6" y="93.98"/>
 <wire x1="101.6" y1="66.04" x2="101.6" y2="63.5" width="0.1524" layer="91"/>
 <pinref part="C5" gate="G$1" pin="1"/>
@@
 <pinref part="JP2" gate="A" pin="1"/>
 <pinref part="R1" gate="G$1" pin="1"/>
-<wire x1="91.44" y1="83.82" x2="83.82" y2="81.28" width="0.1524" layer="91"/>
+<wire x1="91.44" y1="93.98" x2="83.82" y2="81.28" width="0.1524" layer="91"/>
 <junction x="83.82" y="81.28"/>
 </segment>
