File: touch_board/d232_board.sch (EAGLE design)
At the start: 42 parts, among them IC1 uln2803, IC2 uln2803, IC3_5V 7805TV, IC4_10V 7805TV, IC5_12V 7805TV, X1 057-050-1

Commit message: up
Parts:
- added TP10, TP11, TP7, TP8: TPB2,54, testpad:TPB2,54
Connections:
- net +10V: now also TP8.TP
- net +12V: now also TP10.TP
- net +24V: now also TP11.TP
- net +5V: now also TP7.TP
Changed lines of the file:
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@@
 <part name="SUPPLY44" library="supply2" library_urn="urn:adsk.eagle:library:372" deviceset="+5V" device=""/>
 <part name="SUPPLY45" library="supply2" library_urn="urn:adsk.eagle:library:372" deviceset="+5V" device=""/>
+<part name="TP7" library="testpad" library_urn="urn:adsk.eagle:library:385" deviceset="TP" device="B2,54" package3d_urn="urn:adsk.eagle:package:27948/1"/>
+<part name="TP8" library="testpad" library_urn="urn:adsk.eagle:library:385" deviceset="TP" device="B2,54" package3d_urn="urn:adsk.eagle:package:27948/1"/>
+<part name="TP10" library="testpad" library_urn="urn:adsk.eagle:library:385" deviceset="TP" device="B2,54" package3d_urn="urn:adsk.eagle:package:27948/1"/>
+<part name="SUPPLY46" library="supply2" library_urn="urn:adsk.eagle:library:372" deviceset="+5V" device=""/>
+<part name="SUPPLY47" library="supply2" library_urn="urn:adsk.eagle:library:372" deviceset="+10V" device=""/>
+<part name="SUPPLY48" library="supply2" library_urn="urn:adsk.eagle:library:372" deviceset="+12V" device=""/>
+<part name="TP11" library="testpad" library_urn="urn:adsk.eagle:library:385" deviceset="TP" device="B2,54" package3d_urn="urn:adsk.eagle:package:27948/1"/>
+<part name="SUPPLY49" library="supply2" library_urn="urn:adsk.eagle:library:372" deviceset="+24V" device=""/>
 </parts>
 <sheets>
@@
 <instance part="SUPPLY45" gate="+5V" x="76.2" y="106.68" smashed="yes" rot="R90">
 <attribute name="VALUE" x="73.025" y="104.775" size="1.778" layer="96" rot="R90"/>
+</instance>
+<instance part="TP7" gate="G$1" x="58.42" y="-43.18" smashed="yes">
+<attribute name="NAME" x="57.15" y="-41.91" size="1.778" layer="95"/>
+<attribute name="TP_SIGNAL_NAME" x="59.69" y="-44.45" size="1.778" layer="97"/>
+</instance>
+<instance part="TP8" gate="G$1" x="66.04" y="-43.18" smashed="yes">
+<attribute name="NAME" x="64.77" y="-41.91" size="1.778" layer="95"/>
+<attribute name="TP_SIGNAL_NAME" x="67.31" y="-44.45" size="1.778" layer="97"/>
+</instance>
+<instance part="TP10" gate="G$1" x="73.66" y="-43.18" smashed="yes">
+<attribute name="NAME" x="72.39" y="-41.91" size="1.778" layer="95"/>
+<attribute name="TP_SIGNAL_NAME" x="74.93" y="-44.45" size="1.778" layer="97"/>
+</instance>
+<instance part="SUPPLY46" gate="+5V" x="58.42" y="-48.26" smashed="yes" rot="R180">
+<attribute name="VALUE" x="60.325" y="-51.435" size="1.778" layer="96" rot="R180"/>
+</instance>
+<instance part="SUPPLY47" gate="G$1" x="66.04" y="-48.26" smashed="yes" rot="R180">
+<attribute name="VALUE" x="68.58" y="-51.435" size="1.778" layer="96" rot="R180"/>
+</instance>
+<instance part="SUPPLY48" gate="+12V" x="73.66" y="-48.26" smashed="yes" rot="R180">
+<attribute name="VALUE" x="76.2" y="-51.435" size="1.778" layer="96" rot="R180"/>
+</instance>
+<instance part="TP11" gate="G$1" x="81.28" y="-43.18" smashed="yes">
+<attribute name="NAME" x="80.01" y="-41.91" size="1.778" layer="95"/>
+<attribute name="TP_SIGNAL_NAME" x="82.55" y="-44.45" size="1.778" layer="97"/>
+</instance>
+<instance part="SUPPLY49" gate="+24V" x="81.28" y="-48.26" smashed="yes" rot="R180">
+<attribute name="VALUE" x="83.82" y="-51.435" size="1.778" layer="96" rot="R180"/>
 </instance>
 </instances>
@@
 <pinref part="X1" gate="-50" pin="S"/>
 <pinref part="SUPPLY20" gate="GND" pin="GND"/>
+<junction x="-43.18" y="-35.56"/>
 </segment>
 <segment>
@@
 <pinref part="SUPPLY45" gate="+5V" pin="+5V"/>
 </segment>
+<segment>
+<pinref part="TP7" gate="G$1" pin="TP"/>
+<pinref part="SUPPLY46" gate="+5V" pin="+5V"/>
+<junction x="58.42" y="-45.72"/>
+</segment>
 </net>
 <net name="+10V" class="0">
@@
 <junction x="63.5" y="-22.86"/>
 </segment>
+<segment>
+<pinref part="SUPPLY47" gate="G$1" pin="+10V"/>
+<pinref part="SUPPLY47" gate="G$1" pin="+10V"/>
+<pinref part="TP8" gate="G$1" pin="TP"/>
+<junction x="66.04" y="-45.72"/>
+</segment>
 </net>
 <net name="+24V" class="0">
@@
 <wire x1="129.54" y1="12.7" x2="129.54" y2="7.62" width="0.1524" layer="91"/>
 <junction x="129.54" y="7.62"/>
+</segment>
+<segment>
+<pinref part="TP11" gate="G$1" pin="TP"/>
+<pinref part="SUPPLY49" gate="+24V" pin="+24V"/>
+<junction x="81.28" y="-45.72"/>
 </segment>
 </net>
@@
 <junction x="71.12" y="-22.86"/>
 </segment>
-</net>
+<segment>
+<pinref part="TP10" gate="G$1" pin="TP"/>
+<pinref part="SUPPLY48" gate="+12V" pin="+12V"/>
+<junction x="73.66" y="-45.72"/>
+</segment>
+</net>

Commit message: up
Parts:
- renumbered SG1 to MSE14LCH2, SG2 to MSE28LWH1, SG3 to MSE28LDD7
Other:
- note added: "chirp"
- note added: "siren"
- note added: "warp"
Changed lines of the file:
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@@
 <part name="SUPPLY14" library="supply2" library_urn="urn:adsk.eagle:library:372" deviceset="GND" device=""/>
 <part name="SUPPLY15" library="supply2" library_urn="urn:adsk.eagle:library:372" deviceset="GND" device=""/>
-<part name="SG1" library="buzzer" library_urn="urn:adsk.eagle:library:113" deviceset="EB2209A" device="" package3d_urn="urn:adsk.eagle:package:5276/1"/>
-<part name="SG2" library="buzzer" library_urn="urn:adsk.eagle:library:113" deviceset="EB2209A" device="" package3d_urn="urn:adsk.eagle:package:5276/1"/>
-<part name="SG3" library="buzzer" library_urn="urn:adsk.eagle:library:113" deviceset="EB2209A" device="" package3d_urn="urn:adsk.eagle:package:5276/1"/>
+<part name="MSE14LCH2" library="buzzer" library_urn="urn:adsk.eagle:library:113" deviceset="EB2209A" device="" package3d_urn="urn:adsk.eagle:package:5276/1"/>
+<part name="MSE28LWH1" library="buzzer" library_urn="urn:adsk.eagle:library:113" deviceset="EB2209A" device="" package3d_urn="urn:adsk.eagle:package:5276/1"/>
+<part name="MSE28LDD7" library="buzzer" library_urn="urn:adsk.eagle:library:113" deviceset="EB2209A" device="" package3d_urn="urn:adsk.eagle:package:5276/1"/>
 <part name="SUPPLY16" library="supply2" library_urn="urn:adsk.eagle:library:372" deviceset="+10V" device=""/>
 <part name="SUPPLY17" library="supply2" library_urn="urn:adsk.eagle:library:372" deviceset="+24V" device=""/>
@@
 <sheet>
 <plain>
+<text x="76.2" y="38.1" size="1.778" layer="91">chirp</text>
+<text x="96.52" y="27.94" size="1.778" layer="91">siren</text>
+<text x="114.3" y="17.78" size="1.778" layer="91">warp</text>
 </plain>
 <instances>
@@
 <attribute name="VALUE" x="8.255" y="4.445" size="1.778" layer="96"/>
 </instance>
-<instance part="SG1" gate="G$1" x="71.12" y="40.64" smashed="yes" rot="R180">
+<instance part="MSE14LCH2" gate="G$1" x="71.12" y="40.64" smashed="yes" rot="R180">
 <attribute name="NAME" x="73.66" y="34.29" size="1.778" layer="95" rot="R180"/>
 <attribute name="VALUE" x="66.04" y="40.64" size="1.778" layer="96" rot="R180"/>
 </instance>
-<instance part="SG2" gate="G$1" x="91.44" y="30.48" smashed="yes" rot="R180">
+<instance part="MSE28LWH1" gate="G$1" x="91.44" y="30.48" smashed="yes" rot="R180">
 <attribute name="NAME" x="93.98" y="24.13" size="1.778" layer="95" rot="R180"/>
 <attribute name="VALUE" x="86.36" y="30.48" size="1.778" layer="96" rot="R180"/>
 </instance>
-<instance part="SG3" gate="G$1" x="109.22" y="20.32" smashed="yes" rot="R180">
+<instance part="MSE28LDD7" gate="G$1" x="109.22" y="20.32" smashed="yes" rot="R180">
 <attribute name="NAME" x="111.76" y="13.97" size="1.778" layer="95" rot="R180"/>
 <attribute name="VALUE" x="104.14" y="20.32" size="1.778" layer="96" rot="R180"/>
@@
 </segment>
 <segment>
-<pinref part="SG1" gate="G$1" pin="+"/>
+<pinref part="MSE14LCH2" gate="G$1" pin="+"/>
 <pinref part="SUPPLY16" gate="G$1" pin="+10V"/>
 <junction x="73.66" y="43.18"/>
@@
 <segment>
 <pinref part="SUPPLY47" gate="G$1" pin="+10V"/>
-<pinref part="SUPPLY47" gate="G$1" pin="+10V"/>
 <pinref part="TP8" gate="G$1" pin="TP"/>
 <junction x="66.04" y="-45.72"/>
@@
 </segment>
 <segment>
-<pinref part="SG2" gate="G$1" pin="+"/>
+<pinref part="MSE28LWH1" gate="G$1" pin="+"/>
 <pinref part="SUPPLY17" gate="+24V" pin="+24V"/>
 <junction x="93.98" y="33.02"/>
 </segment>
 <segment>
-<pinref part="SG3" gate="G$1" pin="+"/>
+<pinref part="MSE28LDD7" gate="G$1" pin="+"/>
 <pinref part="SUPPLY18" gate="+24V" pin="+24V"/>
 <junction x="111.76" y="22.86"/>
@@
 <pinref part="IC2" gate="G$1" pin="O1"/>
 <wire x1="53.34" y1="33.02" x2="53.34" y2="43.18" width="0.1524" layer="91"/>
-<pinref part="SG1" gate="G$1" pin="-"/>
+<pinref part="MSE14LCH2" gate="G$1" pin="-"/>
 <wire x1="53.34" y1="43.18" x2="66.04" y2="43.18" width="0.1524" layer="91"/>
 <junction x="53.34" y="33.02"/>
@@
 <wire x1="53.34" y1="30.48" x2="81.28" y2="30.48" width="0.1524" layer="91"/>
 <wire x1="81.28" y1="30.48" x2="81.28" y2="33.02" width="0.1524" layer="91"/>
-<pinref part="SG2" gate="G$1" pin="-"/>
+<pinref part="MSE28LWH1" gate="G$1" pin="-"/>
 <wire x1="81.28" y1="33.02" x2="86.36" y2="33.02" width="0.1524" layer="91"/>
 <junction x="53.34" y="30.48"/>
@@
 <wire x1="53.34" y1="27.94" x2="81.28" y2="27.94" width="0.1524" layer="91"/>
 <wire x1="81.28" y1="27.94" x2="81.28" y2="22.86" width="0.1524" layer="91"/>
-<pinref part="SG3" gate="G$1" pin="-"/>
+<pinref part="MSE28LDD7" gate="G$1" pin="-"/>
 <wire x1="81.28" y1="22.86" x2="104.14" y2="22.86" width="0.1524" layer="91"/>
 <junction x="53.34" y="27.94"/>
