File: display_board/display_spi.brd (EAGLE design)
At the start: 97.5 x 54.6 mm, 18 parts

Commit message: update
Parts:
- added IC1: LCD_DIP, ic-package:SOCKET-08
- R1, R2, R3, R4, R5, R6, R7, R8: device rcl:R1206 -> rcl:R0805
- moved R1 35.6 mm to (94.0, 29.2), turned to 180 degrees
- moved R2 27.9 mm to (83.8, 35.6)
- moved R3 20.1 mm to (83.8, 40.6)
- moved R6 15.3 mm to (83.8, 55.9)
- moved R4 13.7 mm to (83.8, 45.7)
- moved SV1 11.7 mm to (94.0, 22.9), turned to 0 degrees
- moved R5 11.5 mm to (83.8, 50.8)
- moved R7 8.98 mm to (88.9, 29.2), turned to 180 degrees
- moved C2 8.03 mm to (97.8, 34.3), turned to 270 degrees
- moved LCD 7.73 mm to (106.7, 39.4)
- moved C1 7.18 mm to (90.2, 34.3), turned to 270 degrees
- moved R8 4.58 mm to (99.1, 29.2), turned to 180 degrees
Connections:
- net GND: now also IC1.8
- net N$1: now also IC1.1, R7.2; no longer R1.2
- net N$10: now also R5.1; no longer R3.1
- net N$12: now also R3.1; no longer R5.1
- net N$13: now also R7.1; no longer R1.1
- net N$14: now also R2.1; no longer R6.1
- net N$15: now also R1.1; no longer R7.1
- net N$2: now also IC1.2, R6.2; no longer R2.2
- net N$3: now also IC1.3, R5.2; no longer R3.2
- net N$4: now also IC1.4
- net N$5: now also IC1.5, R3.2; no longer R5.2
- net N$6: now also IC1.6, R2.2; no longer R6.2
- net N$7: now also R1.2; no longer R7.2
- net N$9: now also R6.1; no longer R2.1
- net VDD: now also IC1.7
Routing:
- net GND: track 131.8 -> 28.2 mm
- net N$12: track 0.00 -> 64.9 mm
- net N$11: track 0.00 -> 60.5 mm
- net N$1: track 15.2 -> 72.2 mm
- net N$13: track 43.4 -> 6.53 mm
- net N$10: track 0.00 -> 33.0 mm
- net N$6: track 8.89 -> 40.6 mm, vias 1 -> 0
- net N$9: track 0.00 -> 28.4 mm
- net N$2: track 11.0 -> 30.1 mm, vias 1 -> 0
- net N$3: track 10.5 -> 27.5 mm, vias 1 -> 0
- net N$8: track 25.4 -> 10.1 mm
- net N$4: track 9.94 -> 25.2 mm, vias 1 -> 0
- net VDD: track 173.9 -> 188.0 mm, vias 1 -> 0
- net N$5: track 9.42 -> 22.8 mm, vias 1 -> 0
- net N$15: track 18.5 -> 6.48 mm
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- added copper zone on layer 16, net GND

Commit message: up mod display board
Parts:
- added C5: 0.1, rcl:C1206
- added GROUND, POWER: TPB1,27, testpad:B1,27
- added PWM_LCD: PWM, testpad:B1,27
- added R11: 133, rcl:R1206
- added R12: 4.7k, rcl:R1206
- added R13: 1k, rcl:R1206
- added SV2: PWM, con-lstb:MA06-1
- added U$1: IRLML2502TRPBF, IRLML2502TRPBF:SOT23
- moved SV1 7.73 mm to (92.7, 30.5)
- moved C1 6.35 mm to (90.2, 40.6), turned to 0 degrees
- moved C2 6.35 mm to (97.8, 40.6), turned to 0 degrees
- moved R1 6.35 mm to (94.0, 35.6)
- moved R7 6.35 mm to (88.9, 35.6)
- moved R8 6.35 mm to (99.1, 35.6)
- moved IC1 5.08 mm to (94.0, 49.5)
Connections:
- new net N$19: LED1.19, LED1.2, U$1.3
- new net N$20: C5.1, LCD1.40, R13.1, SV2.5
- new net N$21: R11.1, U$1.1
- new net N$22: PWM_LCD.TP, R11.2, R12.1, SV2.6
- net GND: now also C5.2, GROUND.TP, SV2.1, U$1.2; no longer LED1.19, LED1.2
- net VDD: now also POWER.TP, R12.2, R13.2, SV2.2; no longer LCD1.40
Routing:
- net N$20: track 0.00 -> 131.4 mm
- net N$22: track 0.00 -> 87.6 mm
- net GND: track 28.2 -> 86.8 mm, vias 0 -> 1
- net N$19: track 0.00 -> 46.5 mm
- net VDD: track 188.0 -> 233.7 mm, vias 0 -> 3
- net N$1: track 72.2 -> 51.8 mm
- net N$5: track 22.8 -> 36.0 mm
- net N$21: track 0.00 -> 7.36 mm
- net N$14: track 18.4 -> 12.8 mm
- net N$2: track 30.1 -> 25.1 mm
- net N$12: track 64.9 -> 60.1 mm
- net N$8: track 10.1 -> 14.1 mm
- net N$3: track 27.5 -> 24.0 mm
- net N$7: track 14.3 -> 17.2 mm
- net N$4: track 25.2 -> 23.0 mm
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
Commit message: up
Connections:
- removed net N$22: PWM_LCD.TP, R11.2, R12.1, SV2.6
- net N$14: now also PWM_LCD.TP, R11.2, R12.1, SV2.6
Routing:
- net N$22: track 87.6 -> 0.00 mm
- net N$14: track 12.8 -> 92.3 mm
- net VDD: track 233.7 -> 224.2 mm
- net N$20: track 131.4 -> 130.8 mm
Changed lines of the file:
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@@
 <?xml version="1.0" encoding="utf-8"?>
 <!DOCTYPE eagle SYSTEM "eagle.dtd">
-<eagle version="9.5.1">
+<eagle version="9.6.2">
 <drawing>
 <settings>
@@
 <wire x1="106.68" y1="35.5854" x2="106.68" y2="35.56" width="0.5" layer="16"/>
 <wire x1="95.9358" y1="43.9674" x2="95.7072" y2="44.0436" width="0.5" layer="16"/>
-<wire x1="89.0778" y1="25.4508" x2="88.9254" y2="25.4508" width="0.5" layer="1"/>
-<wire x1="91.3638" y1="27.7368" x2="89.0778" y2="25.4508" width="0.5" layer="1"/>
-<wire x1="104.4702" y1="27.7368" x2="91.3638" y2="27.7368" width="0.5" layer="1"/>
-<wire x1="105.4608" y1="26.7462" x2="104.4702" y2="27.7368" width="0.5" layer="1"/>
-<wire x1="107.8992" y1="26.7462" x2="105.4608" y2="26.7462" width="0.5" layer="1"/>
-<wire x1="108.6612" y1="27.5082" x2="107.8992" y2="26.7462" width="0.5" layer="1"/>
-<wire x1="108.6612" y1="33.528" x2="108.6612" y2="27.5082" width="0.5" layer="1"/>
-<wire x1="106.68" y1="35.5092" x2="108.6612" y2="33.528" width="0.5" layer="1"/>
-<wire x1="88.9254" y1="25.4508" x2="88.9" y2="25.4" width="0.5" layer="1"/>
-<wire x1="106.68" y1="35.5092" x2="106.68" y2="35.56" width="0.5" layer="1"/>
+<wire x1="88.9254" y1="26.289" x2="88.9254" y2="25.4508" width="0.5" layer="16"/>
+<wire x1="90.8304" y1="28.194" x2="88.9254" y2="26.289" width="0.5" layer="16"/>
+<wire x1="97.155" y1="28.194" x2="90.8304" y2="28.194" width="0.5" layer="16"/>
+<wire x1="103.251" y1="34.29" x2="97.155" y2="28.194" width="0.5" layer="16"/>
+<wire x1="103.251" y1="36.3474" x2="103.251" y2="34.29" width="0.5" layer="16"/>
+<wire x1="88.9254" y1="25.4508" x2="88.9" y2="25.4" width="0.5" layer="16"/>
+<wire x1="103.251" y1="36.3474" x2="103.3272" y2="36.576" width="0.5" layer="16"/>
 <wire x1="72.3138" y1="32.3088" x2="72.3138" y2="29.4894" width="0.5" layer="1"/>
 <wire x1="73.8378" y1="33.8328" x2="72.3138" y2="32.3088" width="0.5" layer="1"/>
@@
 <contactref element="SV1" pad="2"/>
 <contactref element="R2" pad="1"/>
+<contactref element="SV2" pad="6"/>
+<contactref element="R11" pad="2"/>
+<contactref element="R12" pad="1"/>
+<contactref element="PWM_LCD" pad="TP"/>
 <wire x1="82.9056" y1="34.29" x2="82.9056" y2="35.5092" width="0.1524" layer="1"/>
-<wire x1="88.4682" y1="28.7274" x2="82.9056" y2="34.29" width="0.1524" layer="1"/>
+<wire x1="88.4682" y1="28.7274" x2="83.0199" y2="34.1757" width="0.1524" layer="1"/>
+<wire x1="83.0199" y1="34.1757" x2="82.9056" y2="34.29" width="0.1524" layer="1"/>
 <wire x1="89.6874" y1="28.7274" x2="88.4682" y2="28.7274" width="0.1524" layer="1"/>
 <wire x1="91.44" y1="30.48" x2="89.6874" y2="28.7274" width="0.1524" layer="1"/>
 <wire x1="82.9056" y1="35.5092" x2="82.87" y2="35.56" width="0.1524" layer="1"/>
+<wire x1="98.679" y1="25.4508" x2="99.06" y2="25.4508" width="0.1524" layer="1"/>
+<wire x1="95.4024" y1="28.7274" x2="98.679" y2="25.4508" width="0.1524" layer="1"/>
+<wire x1="93.1164" y1="28.7274" x2="95.4024" y2="28.7274" width="0.1524" layer="1"/>
+<wire x1="91.44" y1="30.4038" x2="93.1164" y2="28.7274" width="0.1524" layer="1"/>
+<wire x1="99.06" y1="25.4508" x2="99.06" y2="25.4" width="0.1524" layer="1"/>
+<wire x1="91.44" y1="30.4038" x2="91.44" y2="30.48" width="0.1524" layer="1"/>
+<wire x1="40.9956" y1="29.2608" x2="33.0708" y2="29.2608" width="0.1524" layer="1"/>
+<wire x1="42.1386" y1="30.4038" x2="40.9956" y2="29.2608" width="0.1524" layer="1"/>
+<wire x1="44.6532" y1="30.4038" x2="42.1386" y2="30.4038" width="0.1524" layer="1"/>
+<wire x1="45.7962" y1="29.2608" x2="44.6532" y2="30.4038" width="0.1524" layer="1"/>
+<wire x1="33.0708" y1="29.2608" x2="33.02" y2="29.21" width="0.1524" layer="1"/>
+<wire x1="45.7962" y1="29.2608" x2="45.872" y2="29.21" width="0.1524" layer="1"/>
+<wire x1="45.8724" y1="29.2608" x2="50.9778" y2="29.2608" width="0.1524" layer="1"/>
+<wire x1="50.9778" y1="29.2608" x2="64.6176" y2="29.2608" width="0.1524" layer="1"/>
+<wire x1="64.6176" y1="29.2608" x2="64.618" y2="29.21" width="0.1524" layer="1"/>
+<wire x1="45.8724" y1="29.2608" x2="45.872" y2="29.21" width="0.1524" layer="1"/>
+<wire x1="75.9714" y1="27.1272" x2="83.0199" y2="34.1757" width="0.1524" layer="1"/>
+<wire x1="51.2064" y1="27.1272" x2="75.9714" y2="27.1272" width="0.1524" layer="1"/>
+<wire x1="50.9778" y1="27.3558" x2="51.2064" y2="27.1272" width="0.1524" layer="1"/>
+<wire x1="50.9778" y1="29.2608" x2="50.9778" y2="27.3558" width="0.1524" layer="1"/>
 </signal>
 <signal name="N$15">
@@
 <wire x1="49.8348" y1="28.0416" x2="49.85" y2="28.11" width="0.1524" layer="1"/>
 <wire x1="43.053" y1="29.1846" x2="43.028" y2="29.21" width="0.1524" layer="1"/>
-</signal>
-<signal name="N$22">
-<contactref element="SV2" pad="6"/>
-<contactref element="R11" pad="2"/>
-<contactref element="R12" pad="1"/>
-<contactref element="PWM_LCD" pad="TP"/>
-<wire x1="40.9956" y1="29.2608" x2="33.0708" y2="29.2608" width="0.1524" layer="1"/>
-<wire x1="42.1386" y1="30.4038" x2="40.9956" y2="29.2608" width="0.1524" layer="1"/>
-<wire x1="44.6532" y1="30.4038" x2="42.1386" y2="30.4038" width="0.1524" layer="1"/>
-<wire x1="45.7962" y1="29.2608" x2="44.6532" y2="30.4038" width="0.1524" layer="1"/>
-<wire x1="33.0708" y1="29.2608" x2="33.02" y2="29.21" width="0.1524" layer="1"/>
-<wire x1="45.7962" y1="29.2608" x2="45.872" y2="29.21" width="0.1524" layer="1"/>
-<wire x1="45.8724" y1="29.2608" x2="50.9778" y2="29.2608" width="0.1524" layer="1"/>
-<wire x1="50.9778" y1="29.2608" x2="64.6176" y2="29.2608" width="0.1524" layer="1"/>
-<wire x1="64.6176" y1="29.2608" x2="64.618" y2="29.21" width="0.1524" layer="1"/>
-<wire x1="45.8724" y1="29.2608" x2="45.872" y2="29.21" width="0.1524" layer="1"/>
-<wire x1="98.679" y1="25.4508" x2="99.06" y2="25.4508" width="0.1524" layer="1"/>
-<wire x1="96.9264" y1="27.2034" x2="98.679" y2="25.4508" width="0.1524" layer="1"/>
-<wire x1="93.5736" y1="27.2034" x2="96.9264" y2="27.2034" width="0.1524" layer="1"/>
-<wire x1="92.4306" y1="26.0604" x2="93.5736" y2="27.2034" width="0.1524" layer="1"/>
-<wire x1="92.4306" y1="24.1554" x2="92.4306" y2="26.0604" width="0.1524" layer="1"/>
-<wire x1="91.8972" y1="23.622" x2="92.4306" y2="24.1554" width="0.1524" layer="1"/>
-<wire x1="54.7116" y1="23.622" x2="91.8972" y2="23.622" width="0.1524" layer="1"/>
-<wire x1="50.9778" y1="27.3558" x2="54.7116" y2="23.622" width="0.1524" layer="1"/>
-<wire x1="50.9778" y1="29.2608" x2="50.9778" y2="27.3558" width="0.1524" layer="1"/>
-<wire x1="99.06" y1="25.4508" x2="99.06" y2="25.4" width="0.1524" layer="1"/>
 </signal>
 <signal name="N$20">
@@
 <wire x1="96.8502" y1="25.3746" x2="96.5454" y2="25.3746" width="0.1524" layer="1"/>
 <wire x1="98.6028" y1="23.622" x2="96.8502" y2="25.3746" width="0.1524" layer="1"/>
-<wire x1="105.4608" y1="23.622" x2="98.6028" y2="23.622" width="0.1524" layer="1"/>
-<wire x1="109.1946" y1="27.3558" x2="105.4608" y2="23.622" width="0.1524" layer="1"/>
-<wire x1="109.1946" y1="50.4444" x2="109.1946" y2="27.3558" width="0.1524" layer="1"/>
-<wire x1="104.8512" y1="54.7878" x2="109.1946" y2="50.4444" width="0.1524" layer="1"/>
+<wire x1="104.5464" y1="23.622" x2="98.6028" y2="23.622" width="0.1524" layer="1"/>
+<wire x1="109.0422" y1="28.1178" x2="104.5464" y2="23.622" width="0.1524" layer="1"/>
+<wire x1="109.0422" y1="50.5968" x2="109.0422" y2="28.1178" width="0.1524" layer="1"/>
+<wire x1="104.8512" y1="54.7878" x2="109.0422" y2="50.5968" width="0.1524" layer="1"/>
 <wire x1="88.6968" y1="54.7878" x2="104.8512" y2="54.7878" width="0.1524" layer="1"/>
 <wire x1="75.5904" y1="67.8942" x2="88.6968" y2="54.7878" width="0.1524" layer="1"/>
