File: secs_q84.X/rs232_mon.sch (EAGLE design)
At the start: 10 parts, among them X1 RS232 LINES, X2 ADC POWER

Commit message: up
Parts:
- added C1: 0.1uf, rcl:C-USC0805
- added C2: 10uf, rcl:C-USC0805
- added IC1: MAX203ECWP, maxim:MAX203ECWP
- added LED1: POWER, led:LEDCHIP-LED0603
- added R7, R8: 0ohm, rcl:R-US_R0805
- added R9: 1k, rcl:R-US_R0805
- added SV1: SERIAL BUS, con-lstb:MA10-1
Connections:
- removed net N$4: R6.2, X1-3.S
- new net EQRX: IC1G$1.R2OUT, SV1.4
- new net EQTX: IC1G$1.T2IN, SV1.5
- new net GND: C1.2, C2.2, LED1.C, R8.2
- new net MCURX: IC1G$1.R1OUT, SV1.2
- new net MCUTX: IC1G$1.T1IN, SV1.3
- new net N$5: IC1G$1.V-/1, IC1G$1.V-/2
- new net N$6: IC1G$1.C2-/1, IC1G$1.C2-/2
- new net N$7: IC1G$1.C2+/1, IC1G$1.C2+/2
- new net RS232EQRX: IC1G$1.R2IN, SV1.9
- new net RS232EQTX: IC1G$1.T2OUT, SV1.10
- new net RS232RX: IC1G$1.R1IN, R6.2, SV1.7, X1-3.S
- new net RS232TX: IC1G$1.T1OUT, R3.1, SV1.8, X1-2.S
- new net VCC: C1.1, C2.1, R7.2, R9.1
- net N$3: now also LED1.A, R9.2; no longer R3.1, X1-2.S
- net VDD: now also R7.1
- net VSS: now also R8.1, SV1.1, SV1.6
