File: secs_q84.X/secs_q84 v2.sch (EAGLE design)
At the start: 56 parts, among them IC1 MAX203ECWP, IC4 PIC18F47Q84-I_PT

Commit message: up
Parts:
- removed D1, D2: 5.6V, diode:ZENER-DIODESMB
- added Z1, Z2: BZT52B5V6-TP, BZT52B5V6-TP:BZT52B5V6-TP
- R13, R16: value 86.6k -> 82.5k
Connections:
- net AN1: now also Z1.K; no longer D1.C
- net AN2: now also Z2.K; no longer D2.C
- net VSS: now also Z1.A, Z2.A; no longer D1.A, D2.A
Changed lines of the file:
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@@
 <part name="R3" library="rcl" library_urn="urn:adsk.eagle:library:334" deviceset="R-US_" device="R0805" package3d_urn="urn:adsk.eagle:package:23553/2" value="12.1k"/>
 <part name="R4" library="rcl" library_urn="urn:adsk.eagle:library:334" deviceset="R-US_" device="R0805" package3d_urn="urn:adsk.eagle:package:23553/2" value="12.1k"/>
-<part name="R13" library="rcl" library_urn="urn:adsk.eagle:library:334" deviceset="R-US_" device="R0805" package3d_urn="urn:adsk.eagle:package:23553/2" value="86.6k"/>
+<part name="R13" library="rcl" library_urn="urn:adsk.eagle:library:334" deviceset="R-US_" device="R0805" package3d_urn="urn:adsk.eagle:package:23553/2" value="82.5k"/>
 <part name="R14" library="rcl" library_urn="urn:adsk.eagle:library:334" deviceset="R-US_" device="R0805" package3d_urn="urn:adsk.eagle:package:23553/2" value="12.1k"/>
 <part name="R15" library="rcl" library_urn="urn:adsk.eagle:library:334" deviceset="R-US_" device="R0805" package3d_urn="urn:adsk.eagle:package:23553/2" value="12.1k"/>
-<part name="R16" library="rcl" library_urn="urn:adsk.eagle:library:334" deviceset="R-US_" device="R0805" package3d_urn="urn:adsk.eagle:package:23553/2" value="86.6k"/>
+<part name="R16" library="rcl" library_urn="urn:adsk.eagle:library:334" deviceset="R-US_" device="R0805" package3d_urn="urn:adsk.eagle:package:23553/2" value="82.5k"/>
 <part name="VSS3" library="supply1" library_urn="urn:adsk.eagle:library:371" deviceset="VSS" device=""/>
 <part name="VSS5" library="supply1" library_urn="urn:adsk.eagle:library:371" deviceset="VSS" device=""/>
@@
 <part name="SV2" library="con-lstb" library_urn="urn:adsk.eagle:library:162" deviceset="MA06-1" device="" package3d_urn="urn:adsk.eagle:package:8340/1" value="CANBUS"/>
 <part name="P+4" library="supply1" library_urn="urn:adsk.eagle:library:371" deviceset="VCC" device=""/>
-<part name="D1" library="diode" library_urn="urn:adsk.eagle:library:210" deviceset="ZENER-DIODE" device="SMB" package3d_urn="urn:adsk.eagle:package:43404/2" value="5.6V"/>
-<part name="D2" library="diode" library_urn="urn:adsk.eagle:library:210" deviceset="ZENER-DIODE" device="SMB" package3d_urn="urn:adsk.eagle:package:43404/2" value="5.6V"/>
-<part name="VSS15" library="supply1" library_urn="urn:adsk.eagle:library:371" deviceset="VSS" device=""/>
-<part name="VSS16" library="supply1" library_urn="urn:adsk.eagle:library:371" deviceset="VSS" device=""/>
 <part name="GLORY" library="pinhead" library_urn="urn:adsk.eagle:library:325" deviceset="PINHD-1X2" device="" package3d_urn="urn:adsk.eagle:package:22435/2" value="GLORY"/>
 <part name="VSS17" library="supply1" library_urn="urn:adsk.eagle:library:371" deviceset="VSS" device=""/>
 <part name="VDD10" library="supply1" library_urn="urn:adsk.eagle:library:371" deviceset="VDD" device=""/>
 <part name="F1" library="0805L075WR" deviceset="0805L075WR" device=""/>
+<part name="Z1" library="BZT52B5V6-TP" deviceset="BZT52B5V6-TP" device=""/>
+<part name="Z2" library="BZT52B5V6-TP" deviceset="BZT52B5V6-TP" device=""/>
+<part name="VSS19" library="supply1" library_urn="urn:adsk.eagle:library:371" deviceset="VSS" device=""/>
+<part name="VSS20" library="supply1" library_urn="urn:adsk.eagle:library:371" deviceset="VSS" device=""/>
 </parts>
 <sheets>
@@
 <attribute name="VALUE" x="91.44" y="-2.54" size="1.778" layer="96" rot="R90"/>
 </instance>
-<instance part="D1" gate="G$1" x="218.44" y="101.6" smashed="yes" rot="R90">
-<attribute name="NAME" x="216.535" y="99.822" size="1.778" layer="95" rot="R90"/>
-<attribute name="VALUE" x="221.869" y="99.822" size="1.778" layer="96" rot="R90"/>
-</instance>
-<instance part="D2" gate="G$1" x="256.54" y="101.6" smashed="yes" rot="R90">
-<attribute name="NAME" x="254.635" y="99.822" size="1.778" layer="95" rot="R90"/>
-<attribute name="VALUE" x="259.969" y="99.822" size="1.778" layer="96" rot="R90"/>
-</instance>
-<instance part="VSS15" gate="G$1" x="218.44" y="96.52" smashed="yes">
-<attribute name="VALUE" x="215.9" y="91.44" size="1.778" layer="96" rot="R90"/>
-</instance>
-<instance part="VSS16" gate="G$1" x="256.54" y="96.52" smashed="yes">
-<attribute name="VALUE" x="254" y="91.44" size="1.778" layer="96" rot="R90"/>
-</instance>
 <instance part="GLORY" gate="G$1" x="83.82" y="88.9" smashed="yes" rot="R180">
 <attribute name="NAME" x="90.17" y="83.185" size="1.778" layer="95" rot="R180"/>
@@
 <attribute name="NAME" x="90.17" y="95.25" size="1.778" layer="95" align="center-left"/>
 <attribute name="VALUE" x="95.25" y="95.25" size="1.778" layer="96" align="center-left"/>
+</instance>
+<instance part="Z1" gate="G$1" x="200.66" y="104.14" smashed="yes" rot="R270">
+<attribute name="NAME" x="209.55" y="93.98" size="1.778" layer="95" rot="R270" align="center-left"/>
+<attribute name="VALUE" x="207.01" y="93.98" size="1.778" layer="96" rot="R270" align="center-left"/>
+</instance>
+<instance part="Z2" gate="G$1" x="246.38" y="104.14" smashed="yes" rot="R270">
+<attribute name="NAME" x="255.27" y="93.98" size="1.778" layer="95" rot="R270" align="center-left"/>
+<attribute name="VALUE" x="252.73" y="93.98" size="1.778" layer="96" rot="R270" align="center-left"/>
+</instance>
+<instance part="VSS19" gate="G$1" x="200.66" y="86.36" smashed="yes">
+<attribute name="VALUE" x="198.12" y="81.28" size="1.778" layer="96" rot="R90"/>
+</instance>
+<instance part="VSS20" gate="G$1" x="246.38" y="86.36" smashed="yes">
+<attribute name="VALUE" x="243.84" y="81.28" size="1.778" layer="96" rot="R90"/>
 </instance>
 </instances>
@@
 </segment>
 <segment>
-<pinref part="D1" gate="G$1" pin="A"/>
-<pinref part="VSS15" gate="G$1" pin="VSS"/>
-<junction x="218.44" y="99.06"/>
-</segment>
-<segment>
-<pinref part="D2" gate="G$1" pin="A"/>
-<pinref part="VSS16" gate="G$1" pin="VSS"/>
-<junction x="256.54" y="99.06"/>
-</segment>
-<segment>
 <pinref part="GLORY" gate="G$1" pin="1"/>
 <wire x1="86.36" y1="86.36" x2="101.6" y2="86.36" width="0.1524" layer="91"/>
@@
 <junction x="86.36" y="86.36"/>
 <junction x="101.6" y="86.36"/>
+</segment>
+<segment>
+<pinref part="Z1" gate="G$1" pin="A"/>
+<pinref part="VSS19" gate="G$1" pin="VSS"/>
+<junction x="200.66" y="88.9"/>
+</segment>
+<segment>
+<pinref part="Z2" gate="G$1" pin="A"/>
+<pinref part="VSS20" gate="G$1" pin="VSS"/>
+<junction x="246.38" y="88.9"/>
 </segment>
 </net>
@@
 <wire x1="228.6" y1="104.14" x2="223.52" y2="104.14" width="0.1524" layer="91"/>
 <junction x="223.52" y="104.14"/>
-<wire x1="223.52" y1="104.14" x2="218.44" y2="104.14" width="0.1524" layer="91"/>
 <junction x="228.6" y="104.14"/>
-<junction x="215.9" y="104.14"/>
+<junction x="200.66" y="104.14"/>
 <junction x="223.52" y="99.06"/>
 <junction x="223.52" y="109.22"/>
 <label x="210.82" y="101.6" size="1.778" layer="95"/>
-<pinref part="D1" gate="G$1" pin="C"/>
-<wire x1="218.44" y1="104.14" x2="215.9" y2="104.14" width="0.1524" layer="91"/>
-<junction x="218.44" y="104.14"/>
+<wire x1="223.52" y1="104.14" x2="200.66" y2="104.14" width="0.1524" layer="91"/>
+<pinref part="Z1" gate="G$1" pin="K"/>
 </segment>
 </net>
@@
 <wire x1="266.7" y1="104.14" x2="261.62" y2="104.14" width="0.1524" layer="91"/>
 <junction x="261.62" y="104.14"/>
-<wire x1="261.62" y1="104.14" x2="256.54" y2="104.14" width="0.1524" layer="91"/>
 <junction x="266.7" y="104.14"/>
-<junction x="254" y="104.14"/>
+<junction x="246.38" y="104.14"/>
 <junction x="261.62" y="109.22"/>
 <junction x="261.62" y="96.52"/>
 <label x="248.92" y="101.6" size="1.778" layer="95"/>
-<pinref part="D2" gate="G$1" pin="C"/>
-<wire x1="256.54" y1="104.14" x2="254" y2="104.14" width="0.1524" layer="91"/>
-<junction x="256.54" y="104.14"/>
+<wire x1="261.62" y1="104.14" x2="246.38" y2="104.14" width="0.1524" layer="91"/>
+<pinref part="Z2" gate="G$1" pin="K"/>
 </segment>
 </net>
